File: pcb/HalfBridge_SiC/HalfBridge_SiC.kicad_pcb (KiCad board)
At the start: 2 copper layers, 100 x 100 mm, 96 parts, among them J1 Screw_Terminal_01x02, J10 Conn_01x02, J11 Conn_01x02, J12 Conn_01x02, J14 Conn_01x02_Shielded, J3 AFBR-2624Z, J4 AFBR-2624Z, J5 AFBR-2624Z, J7 Conn_01x02, J8 Conn_01x02, J9 Conn_01x02, Q1 C3M0075120K, Q2 C3M0075120K, SW1 CAS-D20X1, SW2 CAS-D20X1, U1 74AHC1G86, U2 74AHC1G86, U3 74AHC1G86, U4 RKD-052005D, U5 NCD57252, U6 RKD-052005D, U7 MAX3284E, U8 MAX3284E, U9 MAX3284E

Commit message: cap
Parts:
- added J2: 413638-E, My_Connector:TEConnectivity_413638E, B.Cu at (126.7, 117.3)
- C34: footprint My_Capacitor_THT:C4AQNBU4550M1EJ -> My_Capacitor_THT:C_Rect_L42.0mm_W33.0mm_PW37.50mm_PL20.30mm_2port_C4AU
- moved C4 48.9 mm to (68.6, 46.6)
- moved U1 43.2 mm to (67.8, 49.2), turned to 0 degrees
- moved C5 41.3 mm to (68.6, 57.0)
- moved U2 35.9 mm to (67.8, 59.6), turned to 0 degrees
- moved C6 35.6 mm to (68.6, 68.0)
- moved U3 31.1 mm to (67.8, 70.7), turned to 0 degrees
- moved C34 14.8 mm to (106.0, 109.2)
- moved C2 6.99 mm to (91.8, 112.0)
- moved C1 5.26 mm to (97.8, 112.0)
- moved C24 3.73 mm to (48.5, 72.3)
- moved C27 3.73 mm to (46.5, 75.8)
- moved C30 3.73 mm to (45.5, 69.8)
- moved J14 3.73 mm to (60.2, 64.7)
- moved J5 3.73 mm to (50.0, 68.7)
- moved L4 3.73 mm to (44.0, 73.3)
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Routing:
- net /HalfBridge_GateDriver/inga: track 20.9 -> 78.8 mm
- net /HalfBridge_GateDriver/ingb: track 21.1 -> 69.1 mm
- net /HalfBridge_GateDriver/dis_x: track 20.2 -> 64.2 mm
- net /HalfBridge_Diff/ina_d: track 52.9 -> 13.5 mm
- net /HalfBridge_Diff/vcc: track 96.4 -> 58.6 mm
- net /HalfBridge_Diff/inb_d: track 47.0 -> 12.2 mm
- net /HalfBridge_Diff/inen_d: track 38.1 -> 12.6 mm

Commit message: pcb + horizontal of
Parts:
- C7, C8, R1, R9: moved to B.Cu
- J3, J4, J5: footprint OptoDevice:Broadcom_AFBR-16xxZ_Vertical -> OptoDevice:Broadcom_AFBR-16xxZ_Horizontal
- moved J1 31.7 mm to (45.0, 98.5)
- moved R25 13.2 mm to (58.2, 62.2)
- moved R26 13.2 mm to (58.2, 72.7)
- moved J10 13.1 mm to (61.7, 60.5)
- moved J11 13.1 mm to (61.7, 71.0)
- moved J12 13.1 mm to (61.7, 82.0)
- moved J7 13.0 mm to (55.0, 65.0)
- moved J8 13.0 mm to (55.0, 76.0)
- moved J9 13.0 mm to (55.0, 86.5)
- moved C32 13.0 mm to (63.7, 77.7)
- moved C33 13.0 mm to (63.7, 88.2)
- moved R23 13.0 mm to (57.8, 77.7)
- moved C24 13.0 mm to (49.2, 85.3)
- moved C27 13.0 mm to (47.2, 88.8)
- moved C30 13.0 mm to (46.2, 82.8)
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Connections:
- C1 pad 1: /HalfBridge_Power/dcp -> /dcp
- C1 pad 2: /HalfBridge_Power/dcn -> /dcn
- C2 pad 1: /HalfBridge_Power/dcp -> /dcp
- C2 pad 2: /HalfBridge_Power/dcn -> /dcn
- C3 pad 1: /HalfBridge_Power/dcp -> /dcp
- C3 pad 2: /HalfBridge_Power/dcn -> /dcn
- C34 pad 1: /HalfBridge_Power/dcp -> /dcp
- C34 pad 2: /HalfBridge_Power/dcn -> /dcn
- J2 pad D10: unconnected-(J2-PadD10) -> /dcn
- J2 pad D14: unconnected-(J2-PadD14) -> /dcp
- J2 pad D18: unconnected-(J2-PadD18) -> /dcp
- J2 pad D6: unconnected-(J2-PadD6) -> /dcn
- J2 pad Z12: unconnected-(J2-PadZ12) -> /dcp
- J2 pad Z16: unconnected-(J2-PadZ16) -> /dcp
- J2 pad Z4: unconnected-(J2-PadZ4) -> /dcn
- J2 pad Z8: unconnected-(J2-PadZ8) -> /dcn
- Q1 pad 1: /HalfBridge_Power/dcp -> /dcp
- Q2 pad 2: /HalfBridge_Power/dcn -> /dcn
Routing:
- net /HalfBridge_GateDriver/ingb: track 69.1 -> 0.00 mm
- net /HalfBridge_Diff/vcc: track 58.6 -> 82.2 mm
- net /HalfBridge_GateDriver/inga: track 78.8 -> 92.0 mm
- net /HalfBridge_Diff/ina_d: track 13.5 -> 0.58 mm
- net /HalfBridge_Diff/inen_d: track 12.6 -> 0.58 mm
- net /HalfBridge_GateDriver/anb: track 11.8 -> 0.00 mm
- net /HalfBridge_Diff/inb_d: track 12.2 -> 0.58 mm
- net /HalfBridge_GateDriver/dt: track 11.0 -> 0.00 mm
- net /HalfBridge_GateDriver/dis_x: track 64.2 -> 54.4 mm
- net /HalfBridge_GateDriver/dis: track 11.0 -> 6.71 mm
- net /HalfBridge_Diff/inb_nd: track 3.78 -> 0.00 mm
- net /HalfBridge_Diff/gnd: vias 9 -> 8
- added copper zone on F.Cu, net /dcn
- added copper zone on F.Cu, net /dcp
- removed copper zone on F.Cu, net /HalfBridge_Power/dcn
- removed copper zone on F.Cu, net /HalfBridge_Power/dcp
Other:
- outline, holes or cut-outs redrawn

Commit message: vgatereg + route + hsink
Parts:
- removed the J10 at (61.7, 60.5)
- removed J12: Conn_01x02, Connector_PinHeader_2.54mm:PinHeader_1x02_P2.54mm_Vertical
- added C16: 1 u, Capacitor_SMD:C_0805_2012Metric_Pad1.18x1.45mm_HandSolder, F.Cu at (64.8, 106.8)
- added C17: 1 u, Capacitor_SMD:C_0805_2012Metric_Pad1.18x1.45mm_HandSolder, F.Cu at (63.8, 132.4)
- added C18: 100n, Capacitor_SMD:C_0603_1608Metric_Pad1.08x0.95mm_HandSolder, F.Cu at (63.2, 101.5)
- added C19: 100n, Capacitor_SMD:C_0603_1608Metric_Pad1.08x0.95mm_HandSolder, F.Cu at (63.1, 124.4)
- added C5: C, Capacitor_SMD:C_2220_5750Metric_Pad1.97x5.40mm_HandSolder, F.Cu at (109.0, 116.6)
- added J11: Conn_01x02, Connector_PinHeader_2.54mm:PinHeader_1x02_P2.54mm_Horizontal, B.Cu at (64.3, 83.0)
- added R11: 0, Resistor_SMD:R_0805_2012Metric_Pad1.20x1.40mm_HandSolder, B.Cu at (62.4, 112.7)
- added R12: 0, Resistor_SMD:R_0805_2012Metric_Pad1.20x1.40mm_HandSolder, B.Cu at (64.4, 132.4)
- added R13: R, Resistor_SMD:R_0603_1608Metric_Pad0.98x0.95mm_HandSolder, F.Cu at (69.2, 104.0)
- added R14: R, Resistor_SMD:R_0603_1608Metric_Pad0.98x0.95mm_HandSolder, F.Cu at (67.6, 104.0)
- added R15: R, Resistor_SMD:R_0603_1608Metric_Pad0.98x0.95mm_HandSolder, F.Cu at (62.1, 104.4)
- added R16: R, Resistor_SMD:R_0603_1608Metric_Pad0.98x0.95mm_HandSolder, F.Cu at (69.2, 127.2)
- added R17: R, Resistor_SMD:R_0603_1608Metric_Pad0.98x0.95mm_HandSolder, F.Cu at (67.6, 127.2)
- added R18: R, Resistor_SMD:R_0603_1608Metric_Pad0.98x0.95mm_HandSolder, F.Cu at (62.2, 126.8)
- added SW1: SW_Nidec_CAS-120A1, Button_Switch_SMD:Nidec_Copal_CAS-120A, F.Cu at (68.3, 64.2)
- added SW2: SW_Nidec_CAS-120A1, Button_Switch_SMD:Nidec_Copal_CAS-120A, F.Cu at (68.3, 74.4)
- added SW3: SW_Nidec_CAS-120A1, Button_Switch_SMD:Nidec_Copal_CAS-120A, F.Cu at (68.3, 84.0)
- added TP1: TestPoint, TestPoint:TestPoint_Keystone_5015_Micro-Minature, F.Cu at (69.7, 114.8)
- added TP10: TestPoint, TestPoint:TestPoint_Keystone_5015_Micro-Minature, F.Cu at (55.0, 87.0)
- added TP2: TestPoint, TestPoint:TestPoint_Keystone_5015_Micro-Minature, F.Cu at (69.7, 119.4)
- added TP3: TestPoint, TestPoint:TestPoint_Keystone_5015_Micro-Minature, F.Cu at (68.3, 110.8)
- added TP4: TestPoint, TestPoint:TestPoint_Keystone_5015_Micro-Minature, F.Cu at (68.3, 123.4)
- added TP5: TestPoint, TestPoint:TestPoint_Keystone_5015_Micro-Minature, F.Cu at (55.0, 69.6)
- added TP6: TestPoint, TestPoint:TestPoint_Keystone_5015_Micro-Minature, F.Cu at (55.0, 66.6)
- added TP7: TestPoint, TestPoint:TestPoint_Keystone_5015_Micro-Minature, F.Cu at (55.0, 79.8)
- added TP8: TestPoint, TestPoint:TestPoint_Keystone_5015_Micro-Minature, F.Cu at (55.0, 76.8)
- added TP9: TestPoint, TestPoint:TestPoint_Keystone_5015_Micro-Minature, F.Cu at (55.0, 90.0)
- added U7: TL432DBZ, Package_TO_SOT_SMD:SOT-23, F.Cu at (64.9, 104.0)
- added U8: TL432DBZ, Package_TO_SOT_SMD:SOT-23, F.Cu at (64.9, 126.9)
- HS1: footprint My_Heatsink:Heatsink_Fischer_SK125_50 -> My_Heatsink:Heatsink_Fischer_SK687_50
- J1: value Screw_Terminal_01x02 -> Conn_01x02; footprint TerminalBlock_Phoenix:TerminalBlock_Phoenix_PT-1,5-2-3.5-H_1x02_P3.50mm_Horizontal -> Connector_Phoenix_SPT:PhoenixContact_SPT_1.5_2-H-3.5_1x02_P3.5mm_Horizontal
- J10: renamed from J11; footprint Connector_PinHeader_2.54mm:PinHeader_1x02_P2.54mm_Vertical -> Connector_PinHeader_2.54mm:PinHeader_1x02_P2.54mm_Horizontal; moved to B.Cu
- J6: renamed from J14; footprint My_Connector:SAMTEC_T1M-02-F-SV-L-P -> My_Connector:SAMTEC_T1M-02-F-SH-L-K
- J7, J8: value Conn_01x02 -> Conn_01x02_Shielded; footprint Connector_PinHeader_2.54mm:PinHeader_1x02_P2.54mm_Vertical -> My_Connector:SAMTEC_T1M-02-F-SH-L-K; moved to B.Cu
- J9: footprint Connector_PinHeader_2.54mm:PinHeader_1x02_P2.54mm_Vertical -> Connector_PinHeader_2.54mm:PinHeader_1x02_P2.54mm_Horizontal; moved to B.Cu
- R33: renamed from R25; footprint Resistor_SMD:R_0603_1608Metric -> Resistor_SMD:R_0603_1608Metric_Pad0.98x0.95mm_HandSolder
- R34: renamed from R27; footprint Resistor_SMD:R_0603_1608Metric -> Resistor_SMD:R_0603_1608Metric_Pad0.98x0.95mm_HandSolder
- R35: renamed from R26; footprint Resistor_SMD:R_0603_1608Metric -> Resistor_SMD:R_0603_1608Metric_Pad0.98x0.95mm_HandSolder
- moved J9 25.6 mm to (64.3, 62.6), turned to 180 degrees
- moved J8 16.7 mm to (64.8, 89.5), turned to 90 degrees
- moved J7 10.7 mm to (64.9, 69.0), turned to 90 degrees
- moved J1 7.02 mm to (51.9, 99.8)
- moved C2 6.80 mm to (91.0, 116.6)
- moved C3 5.20 mm to (97.0, 116.6)
- moved U1 4.64 mm to (73.0, 63.9)
- moved U2 4.54 mm to (73.0, 74.0)
- moved R33 4.20 mm to (62.2, 63.5)
- moved R35 4.20 mm to (62.2, 74.0)
- moved J6 4.18 mm to (64.8, 79.2)
- moved R34 4.01 mm to (62.2, 83.8)
- moved C7 3.79 mm to (72.6, 71.4)
- moved U3 3.68 mm to (73.0, 82.2)
- moved C6 3.59 mm to (72.2, 61.2)
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- renumbered C34 to C1, C8 to C10, C9 to C11, C13 to C12, C10 to C13, C11 to C14, C12 to C15, C1 to C2, C16 to C20, C17 to C21, C14 to C22, C15 to C23, C20 to C24, C21 to C25, C18 to C26, C19 to C27, C22 to C28, C23 to C29, C2 to C3, C24 to C30, C25 to C31, C26 to C32, C27 to C33, C28 to C34, C29 to C35, C30 to C36, C31 to C37, C32 to C38, C33 to C39, C3 to C4, C4 to C6, C5 to C7, C6 to C8, C7 to C9, R9 to R10, R11 to R19, R12 to R20, R13 to R21, R14 to R22, R15 to R23, R16 to R24, R17 to R25, R18 to R26, R19 to R27, R20 to R28, R21 to R29, R22 to R30, R23 to R31, R24 to R32, R10 to R9, SW1 to SW4, SW2 to SW5, U8 to U10, U9 to U11, U7 to U9
Connections:
- net Net-(D1-K) renamed /lvcc
- net Net-(D2-K) renamed /HalfBridge_GateDriver/lringa
- net Net-(D3-K) renamed /HalfBridge_GateDriver/lringb
- net Net-(D4-K) renamed /HalfBridge_GateDriver/lrdis
- J2 pad D22: unconnected-(J2-PadD22) -> /ph
- J2 pad D26: unconnected-(J2-PadD26) -> /ph
- J2 pad Z20: unconnected-(J2-PadZ20) -> /ph
- J2 pad Z24: unconnected-(J2-PadZ24) -> /ph
- J7 pad 1: /HalfBridge_Diff/ina_db -> /HalfBridge_Diff/ina_da
- J7 pad 2: /HalfBridge_Diff/ina_da -> /HalfBridge_Diff/ina_db
- J8 pad 1: /HalfBridge_Diff/inb_db -> /HalfBridge_Diff/inen_da
- J8 pad 2: /HalfBridge_Diff/inb_da -> /HalfBridge_Diff/inen_db
- J9 pad 1: /HalfBridge_Diff/inen_db -> /HalfBridge_Diff/ina_d
- J9 pad 2: /HalfBridge_Diff/inen_da -> /HalfBridge_Diff/gnd
- Q1 pad 2: /HalfBridge_Power/ph -> /ph
- Q2 pad 1: /HalfBridge_Power/ph -> /ph
- U1 pad 2: unconnected-(U1-Pad2) -> /HalfBridge_GateDriver/xorina
- U2 pad 2: unconnected-(U2-Pad2) -> /HalfBridge_GateDriver/xorinb
- U3 pad 2: unconnected-(U3-Pad2) -> /HalfBridge_GateDriver/xorinen
- U4 pad 1: Net-(U4-VIN+) -> /HalfBridge_GateDriver/vindc+
- U4 pad 2: Net-(U4-VIN-) -> /HalfBridge_GateDriver/vindc-
- U4 pad 6: unconnected-(U4-COM-Pad6) -> /HalfBridge_GateDriver/comh
- U6 pad 1: Net-(U6-VIN+) -> /HalfBridge_GateDriver/vindc+
- U6 pad 2: Net-(U6-VIN-) -> /HalfBridge_GateDriver/vindc-
- U6 pad 6: unconnected-(U6-COM-Pad6) -> /HalfBridge_GateDriver/coml
Routing:
- net /HalfBridge_Diff/vcc: track 82.2 -> 241.8 mm, vias 0 -> 1
- net /HalfBridge_GateDriver/ingb: track 0.00 -> 68.5 mm
- net /HalfBridge_GateDriver/vssh: track 1.55 -> 30.4 mm, vias 0 -> 2
- net /HalfBridge_GateDriver/vcci: track 0.00 -> 25.2 mm, vias 2 -> 5
- net /HalfBridge_Diff/inb_d: track 0.58 -> 21.6 mm
- net /HalfBridge_Diff/ina_d: track 0.58 -> 20.7 mm
- net /HalfBridge_Diff/inen_d: track 0.58 -> 20.7 mm
- net /HalfBridge_GateDriver/inga: track 92.0 -> 72.6 mm
- net /HalfBridge_GateDriver/vssl: track 2.16 -> 21.1 mm
- net /HalfBridge_GateDriver/gonl: track 0.00 -> 16.2 mm
- net /HalfBridge_Diff/inb_db: track 0.00 -> 14.2 mm, vias 0 -> 1
- net /HalfBridge_GateDriver/vddh: track 2.16 -> 16.3 mm, vias 0 -> 2
- net /HalfBridge_GateDriver/anb: track 0.00 -> 12.7 mm
- net /HalfBridge_Diff/inb_da: track 0.00 -> 12.7 mm, vias 0 -> 1
- net /HalfBridge_GateDriver/vddl: track 16.4 -> 28.9 mm
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- added copper zone on B.Cu, net /HalfBridge_Diff/gnd
- added copper zone on F.Cu, net /HalfBridge_Diff/gnd
- added copper zone on F.Cu, net /HalfBridge_GateDriver/gonh
- added copper zone on F.Cu, net /HalfBridge_GateDriver/gonl
- added copper zone on B.Cu, net /HalfBridge_GateDriver/kh
- added copper zone on F.Cu, net /HalfBridge_GateDriver/kh
- added copper zone on B.Cu, net /HalfBridge_GateDriver/kl
- added copper zone on F.Cu, net /HalfBridge_GateDriver/kl
- added copper zone on B.Cu, net /ph
- removed copper zone on B.Cu, net /HalfBridge_Power/ph
Other:
- outline, holes or cut-outs redrawn
- board text added: "* VCC"
- board text added: "AHWV 2024"
- board text added: "EN INB INA DIS PWM"
- board text added: "H"
- board text added: "INA/PWM INB EN/DIS"
- board text added: "S-END DIFF"
- board text added: "o"
- board text added: "x"

Commit message: comment + gdriver + logo
Parts:
- added C16: 10 u, Capacitor_SMD:C_0805_2012Metric_Pad1.18x1.45mm_HandSolder, F.Cu at (52.0, 106.8)
- added C17: 10 u, Capacitor_SMD:C_0805_2012Metric_Pad1.18x1.45mm_HandSolder, F.Cu at (51.6, 132.4)
- added C19: 10 u, Capacitor_SMD:C_0805_2012Metric_Pad1.18x1.45mm_HandSolder, F.Cu at (61.4, 107.4)
- added C25: 10 u, Capacitor_SMD:C_0805_2012Metric_Pad1.18x1.45mm_HandSolder, F.Cu at (61.4, 131.8)
- added L2: 4.7 u, Inductor_SMD:L_0603_1608Metric_Pad1.05x0.95mm_HandSolder, F.Cu at (48.8, 107.4)
- added L3: 4.7 u, Inductor_SMD:L_0603_1608Metric_Pad1.05x0.95mm_HandSolder, F.Cu at (48.8, 131.8)
- added Link:: LOGO, LOGO, F.Cu at (107.2, 79.8)
- C18: renamed from C16; value 1 u -> 10 u
- C20: renamed from C22; value C -> 100 n
- C21: renamed from C23; value C -> 100 n
- C24: renamed from C17; value 1 u -> 10 u
- C30: renamed from C26; value C -> 10 u
- C31: renamed from C27; value C -> 10 u
- U5: value NCD57252 -> NCV51563
- moved C24 1.52 mm to (65.2, 131.8)
- moved C37 1.02 mm to (47.0, 89.2), turned to 180 degrees
- moved C18 0.72 mm to (65.2, 107.4)
- moved C40 0.63 mm to (46.2, 83.8)
- moved C35 0.56 mm to (47.0, 79.0)
- moved C39 0.40 mm to (46.2, 63.0)
- moved J1 0.30 mm to (51.9, 99.5)
- moved L5 0.20 mm to (44.6, 65.8)
- moved C30 0.16 mm to (64.6, 119.8)
- moved U5 0.06 mm to (57.5, 117.2)
- renumbered C12 to C11, C11 to C12, C20 to C22, C21 to C23, C18 to C26, C19 to C27, C24 to C28, C25 to C29, C28 to C32, C29 to C33, C30 to C34, C31 to C35, C32 to C36, C33 to C37, C34 to C38, C35 to C39, C36 to C40, C37 to C41, C38 to C42, C39 to C43, L2 to L4, L3 to L5, L4 to L6, R9 to R10, R10 to R7, R7 to R8, R8 to R9, SW5 to SW4, SW4 to SW5
Connections:
- C18 pad 2: /HalfBridge_GateDriver/vssh -> /HalfBridge_GateDriver/comh
- C24 pad 2: /HalfBridge_GateDriver/vssl -> /HalfBridge_GateDriver/coml
- U4 pad 1: /HalfBridge_GateDriver/vindc+ -> /HalfBridge_GateDriver/vindc+h
- U4 pad 2: /HalfBridge_GateDriver/vindc- -> /HalfBridge_Diff/gnd
- U6 pad 1: /HalfBridge_GateDriver/vindc+ -> /HalfBridge_GateDriver/vindc+l
- U6 pad 2: /HalfBridge_GateDriver/vindc- -> /HalfBridge_Diff/gnd
Routing:
- net /HalfBridge_Diff/vcc: track 241.8 -> 272.0 mm
- net /HalfBridge_Optical/vcca: track 0.00 -> 8.79 mm
- net /HalfBridge_Diff/ina_db: track 5.43 -> 14.0 mm, vias 0 -> 1
- net /HalfBridge_Diff/inen_db: track 5.42 -> 13.8 mm, vias 0 -> 1
- net /HalfBridge_Diff/ina_da: track 5.10 -> 12.6 mm, vias 0 -> 1
- net /HalfBridge_Diff/inen_da: track 5.10 -> 12.5 mm, vias 0 -> 1
- net /HalfBridge_GateDriver/coml: track 0.00 -> 6.72 mm
- net /HalfBridge_Optical/vccen: track 1.80 -> 8.07 mm
- net /HalfBridge_GateDriver/comh: track 2.79 -> 6.67 mm
- net /HalfBridge_GateDriver/vssh: track 30.4 -> 27.6 mm
- net /HalfBridge_GateDriver/vddl: track 28.9 -> 31.5 mm
- net /HalfBridge_GateDriver/vindc+l: track 0.00 -> 2.17 mm
- net /HalfBridge_GateDriver/vindc+h: track 0.00 -> 2.10 mm
- net /HalfBridge_Diff/gnd: track 8.83 -> 10.9 mm
- net /HalfBridge_GateDriver/lringb: track 0.00 -> 1.85 mm
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Other:
- outline, holes or cut-outs redrawn
- board text added: "${TITLE}"
- board text added: "./pcb/${PROJECTNAME}"
- board text added: "Rev: ${REVISION}"
- board text added: "VCC: V VEE: V"

Commit message: 2DPDT switch footprint
Parts:
- R2, R3: value R -> 10 k
- R27, R28, R29, R33, R34, R35: value R -> 0
- R30, R31, R32: value R -> 120
- SW4, SW5: footprint My_Button_Switch_SMD:Nidec_Copal_CAS-D20A1 -> My_Button_Switch_SMD:Nidec_Copal_CAS-D20B1
- moved Link: 7.86 mm to (115.0, 78.8)
- moved D1 1.80 mm to (42.6, 131.0)
- moved R1 1.80 mm to (43.6, 131.0)
- moved SW5 1.36 mm to (43.8, 125.3)
- moved R6 0.88 mm to (43.4, 112.3)
- moved D4 0.87 mm to (44.2, 112.3)
- moved R10 0.82 mm to (47.4, 122.0), turned to -90 degrees
- moved R7 0.63 mm to (42.4, 116.0)
- moved D3 0.49 mm to (44.2, 108.7)
- moved R5 0.49 mm to (43.4, 108.7)
- moved D2 0.40 mm to (44.2, 105.0)
- moved R4 0.40 mm to (43.4, 105.0)
- moved SW4 0.35 mm to (43.8, 117.8)
- moved C36 0.20 mm to (47.4, 68.8)
- moved C13 0.20 mm to (49.4, 118.8)
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Routing:
- net /HalfBridge_Diff/vcc: track 272.0 -> 276.2 mm
- net /HalfBridge_GateDriver/dt: track 10.9 -> 13.8 mm
- net /HalfBridge_GateDriver/dis_i: track 3.52 -> 6.02 mm
- net /HalfBridge_GateDriver/dis: track 16.2 -> 17.6 mm
- net /HalfBridge_GateDriver/anb: track 12.7 -> 14.1 mm
- net /HalfBridge_GateDriver/dis_x: track 58.2 -> 57.5 mm
- net /HalfBridge_GateDriver/vcci: track 27.0 -> 27.7 mm
- net /HalfBridge_GateDriver/rdt: track 1.70 -> 2.24 mm
Other:
- board text added: "${TITLE} ./pcb/${PROJECTNAME} ${COMPANY} Issued: ${ISSUE_DATE}; Rev: ${REVISION}"
- board text removed: "${TITLE}"
- board text removed: "./pcb/${PROJECTNAME}"
