File: pcb/HalfBridge_SiC/HalfBridge_SiC.kicad_pcb (KiCad board)
At the start: 2 copper layers, 100 x 100 mm, 145 parts, among them J1 Conn_01x02, J10 Conn_01x02, J11 Conn_01x02, J12 Conn_01x01, J13 Conn_01x01, J14 Conn_01x01, J15 Conn_01x01, J2 413638-E, J3 AFBR-2624Z, J4 AFBR-2624Z, J5 AFBR-2624Z, J6 Conn_01x02_Shielded, J7 Conn_01x02_Shielded, J8 Conn_01x02_Shielded, J9 Conn_01x02, Q1 C3M0075120K, Q2 C3M0075120K, SW1 SW_Nidec_CAS-120A1, SW2 SW_Nidec_CAS-120A1, SW3 SW_Nidec_CAS-120A1, SW4 CAS-D20X1, SW5 CAS-D20X1, U1 74AHC1G86, U10 MAX3284E, U11 MAX3284E, U2 74AHC1G86, U3 74AHC1G86, U4 RKD-052005D, U5 NCV51563, U6 RKD-052005D, U7 TL432DBZ, U8 TL432DBZ, U9 MAX3284E

Commit message: local lib
Parts:
- J12, J13, J14, J15: footprint My_Connector:WP_SMRA_74663025R -> My_Connector:WP_SMRA_77466303
- moved TP14 17.8 mm to (95.5, 59.5), turned to 90 degrees
- moved TP16 14.5 mm to (95.5, 73.5), turned to 90 degrees
- moved TP15 2.52 mm to (112.5, 59.0), turned to -90 degrees
- moved TP10 0.50 mm to (55.0, 86.5)
- moved TP6 0.50 mm to (55.0, 66.1)
- moved TP8 0.50 mm to (55.0, 76.3)
