File: pcb/HalfBridge_SiC/HalfBridge_SiC.kicad_pcb (KiCad board)
At the start: 2 copper layers, 100 x 100 mm, 145 parts, among them J1 Conn_01x02, J10 Conn_01x02, J11 Conn_01x02, J12 Conn_01x01, J13 Conn_01x01, J14 Conn_01x01, J15 Conn_01x01, J2 413638-E, J3 AFBR-2624Z, J4 AFBR-2624Z, J5 AFBR-2624Z, J6 Conn_01x02_Shielded, J7 Conn_01x02_Shielded, J8 Conn_01x02_Shielded, J9 Conn_01x02, Q1 C3M0075120K, Q2 C3M0075120K, SW1 SW_Nidec_CAS-120A1, SW2 SW_Nidec_CAS-120A1, SW3 SW_Nidec_CAS-120A1, SW4 CAS-D20X1, SW5 CAS-D20X1, U1 74AHC1G86, U10 MAX3284E, U11 MAX3284E, U2 74AHC1G86, U3 74AHC1G86, U4 RKD-052005D, U5 NCV51563, U6 RKD-052005D, U7 TL432DBZ, U8 TL432DBZ, U9 MAX3284E

Commit message: pcb + newlib
Parts:
- added H1: MountingHole, MountingHole:MountingHole_2.2mm_M2_ISO14580, B.Cu at (43.0, 89.5)
- added TP17: TestPoint_Small, TestPoint:TestPoint_Keystone_5015_Micro-Minature, F.Cu at (85.0, 98.0)
- added TP18: TestPoint_Small, TestPoint:TestPoint_Keystone_5015_Micro-Minature, F.Cu at (130.0, 96.0)
- added TP19: TestPoint_Small, TestPoint:TestPoint_Keystone_5015_Micro-Minature, F.Cu at (85.5, 127.0)
- added TP20: TestPoint_Small, TestPoint:TestPoint_Keystone_5015_Micro-Minature, F.Cu at (80.0, 113.0)
- moved C33 5.19 mm to (48.8, 60.9)
- moved J7 5.19 mm to (64.9, 63.9)
- moved C32 5.19 mm to (48.8, 71.0)
- moved C34 5.19 mm to (49.0, 81.4)
- moved C35 5.19 mm to (47.0, 73.8)
- moved C36 5.19 mm to (47.4, 63.6)
- moved C37 5.19 mm to (47.0, 84.0)
- moved C38 5.19 mm to (46.2, 68.4)
- moved C39 5.19 mm to (46.2, 57.8)
- moved C40 5.19 mm to (46.2, 78.6)
- moved C41 5.19 mm to (64.6, 63.3)
- moved C42 5.19 mm to (64.6, 73.6)
- moved C43 5.19 mm to (64.6, 83.6)
- moved C6 5.19 mm to (72.2, 56.0)
- moved C7 5.19 mm to (72.6, 66.2)
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Routing:
- net /HalfBridge_Diff/vcc: track 276.2 -> 283.5 mm
- net /HalfBridge_GateDriver/inga: track 74.2 -> 77.8 mm
- net /HalfBridge_GateDriver/ingb: track 68.4 -> 71.6 mm
- net /HalfBridge_GateDriver/dis_x: track 57.5 -> 60.2 mm
- net /HalfBridge_Diff/gnd: vias 43 -> 47
- added copper zone on F.Cu, net /dcm
- added copper zone on F.Cu, net /ph
Other:
- board text added: "DCm"
- board text added: "Rev: ${REVISION} ${COMMENT1}"
- board text removed: "AHWV 2024"
- board text removed: "DC0"
- board text removed: "Rev: ${REVISION}"

Commit message: backplane + external lib
Parts:
- added H2: MountingHole, MountingHole:MountingHole_2.7mm_M2.5, F.Cu at (81.8, 81.8)
- added H3: MountingHole, MountingHole:MountingHole_2.7mm_M2.5, F.Cu at (43.2, 51.3)
- added H4: MountingHole, MountingHole:MountingHole_2.7mm_M2.5, F.Cu at (43.2, 89.4)
- added TP21: TestPoint, TestPoint:TestPoint_Keystone_5015_Micro-Minature, F.Cu at (75.2, 62.7)
- added TP22: TestPoint, TestPoint:TestPoint_Keystone_5015_Micro-Minature, F.Cu at (75.3, 72.8)
- added TP23: TestPoint, TestPoint:TestPoint_Keystone_5015_Micro-Minature, F.Cu at (75.4, 52.1)
- H1: footprint MountingHole:MountingHole_2.2mm_M2_ISO14580 -> MountingHole:MountingHole_2.7mm_M2.5; moved to F.Cu
- SW5: footprint My_Button_Switch_SMD:Nidec_Copal_CAS-D20B1 -> My_Button_Switch_SMD:SW_SPDTx02_Slide_Copal_CAS-D20B1_W5.6mm_P1.7mm_GullW
- U10, U11, U9: footprint Package_TO_SOT_SMD:SOT-23-6_Handsoldering -> Package_TO_SOT_SMD:SOT-23-6
- U5: footprint Package_SO:SOIC-16W_7.5x10.3mm_P1.27mm -> My_Package_SO:SOIC-16W_7.5x10.3mm_P1.27mm_NoPin_12_13
- moved H1 54.1 mm to (81.3, 51.3), turned to 0 degrees
- moved SW5 7.60 mm to (43.8, 117.7)
- moved SW4 7.58 mm to (43.8, 125.3)
- moved C1 1.91 mm to (106.4, 105.7)
- moved C7 0.40 mm to (72.2, 66.2)
- moved C8 0.40 mm to (72.2, 74.4)
- moved J13 0.40 mm to (136.0, 96.4)
- moved J15 0.40 mm to (136.0, 55.7)
- moved J12 0.40 mm to (136.0, 116.7)
- moved J14 0.40 mm to (136.0, 76.1)
- moved J1 0.32 mm to (51.9, 99.8)
Connections:
- SW4 pad 1: /HalfBridge_GateDriver/dis_i -> /HalfBridge_GateDriver/rdt
- SW4 pad 2: /HalfBridge_GateDriver/dis -> /HalfBridge_GateDriver/dt
- SW4 pad 3: /HalfBridge_GateDriver/dis_x -> /HalfBridge_Diff/vcc
- SW4 pad 5: /HalfBridge_GateDriver/dis_i -> /HalfBridge_GateDriver/anb
- SW5 pad 1: /HalfBridge_GateDriver/rdt -> /HalfBridge_GateDriver/dis_i
- SW5 pad 2: /HalfBridge_GateDriver/dt -> /HalfBridge_GateDriver/dis
- SW5 pad 3: /HalfBridge_Diff/vcc -> /HalfBridge_GateDriver/dis_x
- SW5 pad 5: /HalfBridge_GateDriver/anb -> /HalfBridge_GateDriver/dis_i
Routing:
- net /HalfBridge_Diff/vcc: track 283.5 -> 282.7 mm
- net /HalfBridge_Diff/gnd: vias 47 -> 56
Other:
- outline, holes or cut-outs redrawn
- board text added: "*EN INB INA DIS PWM"

Commit message: backplane
Parts:
- moved H2 1.19 mm to (80.6, 81.8)
- moved H1 0.68 mm to (80.6, 51.3)
- moved H3 0.68 mm to (42.5, 51.3)
- moved H4 0.68 mm to (42.5, 89.4)
Changed lines of the file:
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@@
 	(footprint "MountingHole:MountingHole_2.7mm_M2.5"
 		(layer "F.Cu")
-		(at 81.28 51.308)
+		(at 80.6 51.308)
 		(descr "Mounting Hole 2.7mm, no annular, M2.5")
 		(tags "mounting hole 2.7mm no annular m2.5")
@@
 	(footprint "MountingHole:MountingHole_2.7mm_M2.5"
 		(layer "F.Cu")
-		(at 81.788 81.788)
+		(at 80.6 81.788)
 		(descr "Mounting Hole 2.7mm, no annular, M2.5")
 		(tags "mounting hole 2.7mm no annular m2.5")
@@
 	(footprint "MountingHole:MountingHole_2.7mm_M2.5"
 		(layer "F.Cu")
-		(at 43.18 89.408)
+		(at 42.5 89.408)
 		(descr "Mounting Hole 2.7mm, no annular, M2.5")
 		(tags "mounting hole 2.7mm no annular m2.5")
@@
 	(footprint "MountingHole:MountingHole_2.7mm_M2.5"
 		(layer "F.Cu")
-		(at 43.18 51.308)
+		(at 42.5 51.308)
 		(descr "Mounting Hole 2.7mm, no annular, M2.5")
 		(tags "mounting hole 2.7mm no annular m2.5")
@@
 	)
 	(gr_text "INA/PWM\n\n\n\n\n\n\nINB\n\n\n\n\n\n\nEN/DIS"
-		(at 78 80.5 -0)
+		(at 78 78.5 -0)
 		(layer "B.SilkS" knockout)
 		(effects
@@
 	)
 	(gr_text "INA/PWM\n\n\n\n\n\n\nINB\n\n\n\n\n\n\nEN/DIS"
-		(at 77.5 80.5 0)
+		(at 77.5 78.5 0)
 		(layer "F.SilkS" knockout)
 		(effects
@@
 		)
 		(height -8.496)
-		(gr_text "100.0000 mm"
+		(gr_text "100,0000 mm"
 			(at 89.5 30.854 0)
 			(layer "Dwgs.User")
@@
 		)
 		(height -8.074)
-		(gr_text "100.0000 mm"
+		(gr_text "100,0000 mm"
 			(at 146.424 90.5 90)
 			(layer "Dwgs.User")
@@
 		(height -15.24)
 		(orientation 1)
-		(gr_text "10.8080 mm"
+		(gr_text "10,8080 mm"
 			(at 26.79 45.904 90)
 			(layer "Dwgs.User")
@@
 		(layer "Dwgs.User")
 		(pts
+			(xy 42.5 51.308) (xy 39.5 40.5)
+		)
+		(height -22.308)
+		(orientation 0)
+		(gr_text "3,0000 mm"
+			(at 41 27.9 0)
+			(layer "Dwgs.User")
+			(effects
+				(font
+					(size 1 1)
+					(thickness 0.1)
+				)
+			)
+		)
+		(format
+			(prefix "")
+			(suffix "")
+			(units 2)
+			(units_format 1)
+			(precision 4)
+		)
+		(style
+			(thickness 0.1)
+			(arrow_length 1.27)
+			(text_position_mode 0)
+			(extension_height 0.58642)
+			(extension_offset 0.5) keep_text_aligned)
+	)
+	(dimension
+		(type orthogonal)
+		(layer "Dwgs.User")
+		(pts
 			(xy 136 116.700001) (xy 139.5 140.5)
 		)
@@
 		(layer "Dwgs.User")
 		(pts
-			(xy 43.18 51.308) (xy 81.28 52.578)
+			(xy 42.5 89.408) (xy 80.6 81.788)
 		)
-		(height -16.002)
+		(height -52.908)
 		(orientation 0)
-		(gr_text "1500.0000 mils"
-			(at 62.23 34.156 0)
+		(gr_text "1500,0000 mils"
+			(at 61.55 35.35 0)
 			(layer "Dwgs.User")
 			(effects

Commit message: update lib
Parts:
- added C44: 1n, Capacitor_SMD:C_0603_1608Metric_Pad1.08x0.95mm_HandSolder, F.Cu at (76.4, 107.5)
- added C45: 1n, Capacitor_SMD:C_0603_1608Metric_Pad1.08x0.95mm_HandSolder, F.Cu at (76.4, 124.2)
- added D7: D, Diode_SMD:D_SMB-SMC_Universal_Handsoldering, B.Cu at (60.0, 117.3)
- added R40: R, Resistor_SMD:R_0805_2012Metric_Pad1.20x1.40mm_HandSolder, F.Cu at (60.2, 124.5)
- C10, C9: value C -> 33p
- C11, C32, C33, C34: value C -> 100n
- C12, C28, C29, C35, C36, C37, C38, C39, C40: value C -> 10u
- C13: value 1 u -> 10u
- C16, C17, C18, C19, C24, C25, C30, C31: value 10 u -> 10u
- C20, C21: value 100 n -> 100n
- J12, J13, J14, J15: footprint My_Connector:WP_SMRA_77466303 -> My_Connector:WP_SMRA_7466303
- L1: value L -> 4.7u
- L2, L3: value 4.7 u -> 4.7u
- L4, L5, L6: value L -> 1u
- R1, R4, R5, R6: footprint Resistor_SMD:R_0603_1608Metric -> Resistor_SMD:R_0603_1608Metric_Pad0.98x0.95mm_HandSolder
- R10: footprint Resistor_SMD:R_0603_1608Metric_Pad0.98x0.95mm_HandSolder -> Resistor_SMD:R_0805_2012Metric_Pad1.20x1.40mm_HandSolder
- R2, R3: value 10 k -> 10k
- R36, R37: value R -> 100k; footprint Resistor_THT:R_Axial_DIN0411_L9.9mm_D3.6mm_P25.40mm_Horizontal -> Resistor_THT:R_Axial_DIN0617_L17.0mm_D6.0mm_P30.48mm_Horizontal
- R8, R9: value R -> 51
- SW4: footprint My_Button_Switch_SMD:Nidec_Copal_CAS-D20B1 -> My_Button_Switch_SMD:SW_SPDTx02_Slide_Copal_CAS-D20B1_W5.6mm_P1.7mm_GullW
- TP11, TP12, TP13, TP16: footprint TestPoint:TestPoint_THTPad_D3.0mm_Drill1.5mm -> TestPoint:TestPoint_THTPad_D2.0mm_Drill1.0mm
- TP14, TP15: footprint TestPoint:TestPoint_THTPad_D3.0mm_Drill1.5mm -> TestPoint:TestPoint_Plated_Hole_D3.0mm
- moved R11 10.9 mm to (63.0, 101.9), turned to 0 degrees
- moved TP11 9.15 mm to (123.6, 65.1)
- moved TP13 8.58 mm to (123.6, 129.1)
- moved R3 7.47 mm to (84.1, 124.2)
- moved R2 7.26 mm to (84.1, 107.2)
- moved TP19 6.82 mm to (85.3, 120.2)
- moved J8 6.26 mm to (70.9, 82.9)
- moved J6 6.23 mm to (70.9, 72.8)
- moved J7 6.10 mm to (70.9, 62.6)
- moved TP16 4.84 mm to (91.2, 75.7)
- moved R36 4.55 mm to (120.3, 65.1)
- moved TP12 3.31 mm to (123.3, 96.8)
- moved C2 2.02 mm to (93.0, 116.9)
- moved C3 2.02 mm to (99.0, 116.9)
- moved C4 2.02 mm to (105.0, 116.9)
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Routing:
- net /HalfBridge_GateDriver/vddh: track 17.1 -> 28.0 mm, vias 2 -> 4
- net /HalfBridge_GateDriver/comh: track 6.67 -> 13.8 mm
- net /HalfBridge_Diff/inen_da: track 12.5 -> 18.9 mm
- net /HalfBridge_Diff/inb_da: track 12.7 -> 18.9 mm
- net /HalfBridge_Diff/ina_da: track 12.6 -> 18.8 mm
- net /HalfBridge_Diff/inen_db: track 13.8 -> 20.0 mm
- net /HalfBridge_Diff/ina_db: track 14.0 -> 20.1 mm
- net /HalfBridge_Diff/inb_db: track 14.2 -> 20.3 mm
- net /HalfBridge_GateDriver/inga: track 77.9 -> 82.5 mm
- net /HalfBridge_GateDriver/kh: track 3.46 -> 7.84 mm, vias 23 -> 22
- net /HalfBridge_GateDriver/kl: track 7.23 -> 11.4 mm
- net /HalfBridge_Power/gh: track 11.2 -> 15.3 mm
- net /HalfBridge_Power/gl: track 12.5 -> 16.6 mm
- net /HalfBridge_GateDriver/ingb: track 71.6 -> 75.5 mm
- net /HalfBridge_GateDriver/vddl: track 31.5 -> 35.3 mm, vias 2 -> 4
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- added copper zone on B.Cu, net /HalfBridge_GateDriver/bootR
- added copper zone on B.Cu, net /HalfBridge_GateDriver/vddh
Other:
- outline, holes or cut-outs redrawn
- board text added: "GND"
- board text added: "SW5 A B 1 D/ext 1 D/int VCC 0 D/int 0 D/int GND SW4 A B 1 DT 1 INA=PWM 0 No-DT 0 INA + INB"
- board text removed: "EN INB INA DIS PWM"

Commit message: filter + sim + assembly3d
Parts:
- R1, R4, R5, R6: value R -> 330
- SW1, SW2, SW3: value SW_Nidec_CAS-120A1 -> CAS-120X1; footprint Button_Switch_SMD:Nidec_Copal_CAS-120A -> My_Button_Switch_SMD:Nidec_Copal_CAS-120B1
- moved C6 3.88 mm to (76.1, 54.9), turned to 0 degrees
- moved C7 3.78 mm to (76.0, 65.1), turned to 0 degrees
- moved C8 3.56 mm to (75.8, 75.2), turned to 0 degrees
- moved H1 2.54 mm to (83.1, 50.0)
- moved H2 2.54 mm to (83.1, 80.5)
- moved U1 0.87 mm to (73.9, 57.5)
- moved U2 0.87 mm to (73.9, 67.6)
- moved U3 0.87 mm to (73.9, 77.8)
- moved SW1 0.55 mm to (68.7, 57.4)
- moved SW2 0.55 mm to (68.7, 67.6)
- moved SW3 0.38 mm to (68.7, 78.0)
- moved TP21 0.37 mm to (75.6, 61.5)
- moved TP22 0.27 mm to (75.6, 71.6)
- moved R40 0.12 mm to (60.1, 124.5)
Routing:
- net /HalfBridge_Diff/vcc: track 282.3 -> 288.2 mm
- net /HalfBridge_GateDriver/inga: track 82.5 -> 84.5 mm
- net /HalfBridge_GateDriver/ingb: track 75.5 -> 77.1 mm
- net /HalfBridge_Diff/inb_d: track 24.3 -> 25.2 mm
- net /HalfBridge_Diff/inen_d: track 23.1 -> 24.0 mm
- net /HalfBridge_Diff/ina_d: track 23.4 -> 24.3 mm
- net /HalfBridge_GateDriver/xorinb: track 2.29 -> 1.79 mm
- net /HalfBridge_GateDriver/xorina: track 2.29 -> 1.79 mm
- net /HalfBridge_Diff/gnd: vias 80 -> 89
Other:
- outline, holes or cut-outs redrawn

Commit message: designator + part n°
Parts:
- removed Q1, Q2: C3M0075120K, Package_TO_SOT_THT:TO-247-4_Vertical
- added Q3: C3M0040120K, Package_TO_SOT_THT:TO-247-4_Vertical, B.Cu at (80.0, 98.3)
- added Q4: C3M0040120K, Package_TO_SOT_THT:TO-247-4_Vertical, B.Cu at (80.0, 115.3)
- C1: value C -> 10 u
- C2, C3, C4, C5: value C -> 100 n
