File: pcb/HalfBridge_SiC/HalfBridge_Power.kicad_sch (KiCad schematic)
At the start: 9 parts, among them Q1 C3M0075120K, Q2 C3M0075120K

Commit message: cap
Parts:
- added C35, C36: C_Polarized, Capacitor_THT:CP_Radial_D10.0mm_P7.50mm, symbol Device:C_Polarized
Connections:
- net dcm: now also C35.2, C36.1
- net dcn: now also C36.2
- net dcp: now also C35.1

Commit message: sch
Parts:
- removed C35, C36: C_Polarized, Capacitor_THT:CP_Radial_D10.0mm_P7.50mm, symbol Device:C_Polarized
- C34: footprint My_Capacitor_THT:C4AQNBU4550M1EJ -> My_Capacitor_THT:C_Rect_L42.0mm_W33.0mm_PW37.50mm_PL20.30mm_2port_C4AU

Commit message: vgatereg + route + hsink
Parts:
- added C5: C, Capacitor_SMD:C_2220_5750Metric_Pad1.97x5.40mm_HandSolder, symbol Device:C
- HS1: footprint My_Heatsink:Heatsink_Fischer_SK125_50 -> My_Heatsink:Heatsink_Fischer_SK687_50; Part Number (none) -> SK 687 50 SA
- renumbered C34 to C1, C1 to C2, C2 to C3, C3 to C4
Connections:
- net dcn: now also C5.2
- net dcp: now also C5.1
Other:
- moved on the sheet: C1, C2, C3, C4

Commit message: comment + gdriver + logo
Parts:
- R2, R3: value R -> 10 k
Other:
- title: (none) -> Power stage (Half Bridge)
- moved on the sheet: C1, C2, C3, C4, C5, HS1

Commit message: part number
Parts:
- HS1: Manufacturer Part Number (none) -> SK 687 50 SA; Part Number SK 687 50 SA -> (none)
Changed lines of the file:
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@@
 			)
 		)
-		(property "Part Number" "SK 687 50 SA"
+		(property "Manufacturer Part Number" "SK 687 50 SA"
 			(at 256.54 39.37 0)
 			(effects
