File: pcb/HalfBridge_SiC/HalfBridge_Power.kicad_sch (KiCad schematic)
At the start: 10 parts, among them Q1 C3M0075120K, Q2 C3M0075120K

Commit message: backplane
Parts:
- added R36, R37: R, Resistor_THT:R_Axial_DIN0411_L9.9mm_D3.6mm_P25.40mm_Horizontal, symbol Device:R
- C1: footprint My_Capacitor_THT:C_Rect_L42.0mm_W33.0mm_PW37.50mm_PL20.30mm_2port_C4AU -> My_Capacitor_THT:C_Rect_L42.0mm_W20.0mm_PW37.50mm_PL10.2mm_C4AU; Manufacturer Part Number (none) -> C4AUNBW5100M3FJ
Connections:
- net dcm: now also R36.2, R37.1
- net dcn: now also R37.2
- net dcp: now also R36.1
Other:
- moved on the sheet: HS1, Q2, R2, R3
