File: pcb/HalfBridge_SiC/HalfBridge_Power.kicad_sch (KiCad schematic)
At the start: 12 parts, among them Q1 C3M0075120K, Q2 C3M0075120K

Commit message: local lib
Parts:
- C1, C2, C3, C4, C5: symbol Device:C -> HalfBridge_SiC:C
- HS1: symbol Mechanical:Heatsink_Pad_2Pin -> HalfBridge_SiC:Heatsink_Pad_2Pin
- Q1, Q2: symbol Transistor_FET:C3M0075120K -> HalfBridge_SiC:C3M0075120K
- R2, R3, R36, R37: symbol Device:R -> HalfBridge_SiC:R
Changed lines of the file:
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@@
+		)
+	)
+	(text_box "Bleeding resistors"
+		(exclude_from_sim no)
+		(at 102.87 25.4 0)
+		(size 21.59 6.35)
+		(stroke
+			(width 0)
+			(type default)
+		)
+		(fill
+			(type none)
+		)
+		(effects
+			(font
+				(size 1.27 1.27)
+			)
+			(justify left top)
 		)
 	)
@@
 	)
 	(symbol
-		(lib_id "Transistor_FET:C3M0075120K")
+		(lib_id "HalfBridge_SiC:C3M0075120K")
 		(at 227.33 59.69 0)
 		(unit 1)
@@
 	)
 	(symbol
-		(lib_id "Mechanical:Heatsink_Pad_2Pin")
+		(lib_id "HalfBridge_SiC:Heatsink_Pad_2Pin")
 		(at 255.27 35.56 0)
 		(unit 1)
@@
 	)
 	(symbol
-		(lib_id "Device:C")
+		(lib_id "HalfBridge_SiC:C")
 		(at 176.53 50.8 0)
 		(unit 1)
@@
 	)
 	(symbol
-		(lib_id "Device:R")
+		(lib_id "HalfBridge_SiC:R")
 		(at 224.79 73.66 0)
 		(unit 1)
@@
 	)
 	(symbol
-		(lib_id "Device:R")
+		(lib_id "HalfBridge_SiC:R")
 		(at 212.09 73.66 0)
 		(unit 1)
@@
 	)
 	(symbol
-		(lib_id "Transistor_FET:C3M0075120K")
+		(lib_id "HalfBridge_SiC:C3M0075120K")
 		(at 227.33 43.18 0)
 		(unit 1)
@@
 	)
 	(symbol
-		(lib_id "Device:C")
+		(lib_id "HalfBridge_SiC:C")
 		(at 189.23 50.8 0)
 		(unit 1)
@@
 	)
 	(symbol
-		(lib_id "Device:C")
+		(lib_id "HalfBridge_SiC:C")
 		(at 165.1 50.8 0)
 		(unit 1)
@@
 	)
 	(symbol
-		(lib_id "Device:C")
+		(lib_id "HalfBridge_SiC:C")
 		(at 138.43 50.8 0)
 		(unit 1)
@@
 	)
 	(symbol
-		(lib_id "Device:R")
+		(lib_id "HalfBridge_SiC:R")
 		(at 110.49 60.96 0)
 		(unit 1)
@@
 	)
 	(symbol
-		(lib_id "Device:C")
+		(lib_id "HalfBridge_SiC:C")
 		(at 201.93 50.8 0)
 		(unit 1)
@@
 	)
 	(symbol
-		(lib_id "Device:R")
+		(lib_id "HalfBridge_SiC:R")
 		(at 110.49 41.91 0)
 		(unit 1)

Commit message: pcb + newlib
Other:
- company: (none) -> Dr.-Ing. Alan H. Wilson Veas
Changed lines of the file:
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@@
 		(title "Power stage (Half Bridge)")
 		(rev "1")
+		(company "Dr.-Ing. Alan H. Wilson Veas")
+		(comment 1 "AHWV")
 	)
 	(junction

Commit message: backplane + external lib
Parts:
- C1: footprint My_Capacitor_THT:C_Rect_L42.0mm_W20.0mm_PW37.50mm_PL10.2mm_C4AU -> (none); Manufacturer Part Number C4AUNBW5100M3FJ -> (none)
- C2, C3, C4, C5: footprint Capacitor_SMD:C_2220_5750Metric_Pad1.97x5.40mm_HandSolder -> (none)
- HS1: footprint My_Heatsink:Heatsink_Fischer_SK687_50 -> (none); Manufacturer Part Number SK 687 50 SA -> (none); Part # (none) -> SK 687 50 SA
- R2, R3: footprint Resistor_SMD:R_0805_2012Metric_Pad1.20x1.40mm_HandSolder -> (none)
- R36, R37: footprint Resistor_THT:R_Axial_DIN0411_L9.9mm_D3.6mm_P25.40mm_Horizontal -> (none)
Changed lines of the file:
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@@
 			)
 		)
-		(property "Footprint" "My_Heatsink:Heatsink_Fischer_SK687_50"
+		(property "Footprint" ""
 			(at 255.5748 36.83 0)
 			(effects
@@
 			)
 		)
-		(property "Manufacturer Part Number" "SK 687 50 SA"
-			(at 256.54 39.37 0)
+		(property "Part #" "SK 687 50 SA"
+			(at 255.27 35.56 0)
 			(effects
 				(font
@@
 			)
 		)
-		(property "Footprint" "Capacitor_SMD:C_2220_5750Metric_Pad1.97x5.40mm_HandSolder"
+		(property "Footprint" ""
 			(at 177.4952 54.61 0)
 			(effects
@@
 			)
 		)
-		(property "Footprint" "Resistor_SMD:R_0805_2012Metric_Pad1.20x1.40mm_HandSolder"
+		(property "Footprint" ""
 			(at 223.012 73.66 90)
 			(effects
@@
 			)
 		)
-		(property "Footprint" "Resistor_SMD:R_0805_2012Metric_Pad1.20x1.40mm_HandSolder"
+		(property "Footprint" ""
 			(at 210.312 73.66 90)
 			(effects
@@
 			)
 		)
-		(property "Footprint" "Capacitor_SMD:C_2220_5750Metric_Pad1.97x5.40mm_HandSolder"
+		(property "Footprint" ""
 			(at 190.1952 54.61 0)
 			(effects
@@
 			)
 		)
-		(property "Footprint" "Capacitor_SMD:C_2220_5750Metric_Pad1.97x5.40mm_HandSolder"
+		(property "Footprint" ""
 			(at 166.0652 54.61 0)
 			(effects
@@
 			)
 		)
-		(property "Footprint" "My_Capacitor_THT:C_Rect_L42.0mm_W20.0mm_PW37.50mm_PL10.2mm_C4AU"
+		(property "Footprint" ""
 			(at 139.3952 54.61 0)
 			(effects
@@
 			)
 		)
-		(property "Manufacturer Part Number" "C4AUNBW5100M3FJ"
-			(at 138.43 50.8 0)
-			(effects
-				(font
-					(size 1.27 1.27)
-				)
-				(hide yes)
-			)
-		)
 		(pin "2"
 		)
@@
 			)
 		)
-		(property "Footprint" "Resistor_THT:R_Axial_DIN0411_L9.9mm_D3.6mm_P25.40mm_Horizontal"
+		(property "Footprint" ""
 			(at 108.712 60.96 90)
 			(effects
@@
 			)
 		)
-		(property "Footprint" "Capacitor_SMD:C_2220_5750Metric_Pad1.97x5.40mm_HandSolder"
+		(property "Footprint" ""
 			(at 202.8952 54.61 0)
 			(effects
@@
 			)
 		)
-		(property "Footprint" "Resistor_THT:R_Axial_DIN0411_L9.9mm_D3.6mm_P25.40mm_Horizontal"
+		(property "Footprint" ""
 			(at 108.712 41.91 90)
 			(effects

Commit message: update lib
Parts:
- C1: footprint (none) -> My_Capacitor_THT:C_Rect_L42.0mm_W20.0mm_PW37.50mm_PL10.2mm_C4AU
- C2, C3, C4, C5: footprint (none) -> Capacitor_SMD:C_2220_5750Metric_Pad1.97x5.40mm_HandSolder
- HS1: footprint (none) -> My_Heatsink:Heatsink_Fischer_SK687_50
- R2, R3: value 10 k -> 10k; footprint (none) -> Resistor_SMD:R_0805_2012Metric_Pad1.20x1.40mm_HandSolder
- R36, R37: value R -> 100k; footprint (none) -> Resistor_THT:R_Axial_DIN0617_L17.0mm_D6.0mm_P30.48mm_Horizontal; Part # (none) -> RR03J100KTB
Changed lines of the file:
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@@
 			)
 		)
-		(property "Footprint" ""
+		(property "Footprint" "My_Heatsink:Heatsink_Fischer_SK687_50"
 			(at 255.5748 36.83 0)
 			(effects
@@
 			)
 		)
-		(property "Footprint" ""
+		(property "Footprint" "Capacitor_SMD:C_2220_5750Metric_Pad1.97x5.40mm_HandSolder"
 			(at 177.4952 54.61 0)
 			(effects
@@
 			)
 		)
-		(property "Value" "10 k"
+		(property "Value" "10k"
 			(at 227.33 74.9299 0)
 			(effects
@@
 			)
 		)
-		(property "Footprint" ""
+		(property "Footprint" "Resistor_SMD:R_0805_2012Metric_Pad1.20x1.40mm_HandSolder"
 			(at 223.012 73.66 90)
 			(effects
@@
 			)
 		)
-		(property "Value" "10 k"
+		(property "Value" "10k"
 			(at 214.63 74.9299 0)
 			(effects
@@
 			)
 		)
-		(property "Footprint" ""
+		(property "Footprint" "Resistor_SMD:R_0805_2012Metric_Pad1.20x1.40mm_HandSolder"
 			(at 210.312 73.66 90)
 			(effects
@@
 			)
 		)
-		(property "Footprint" ""
+		(property "Footprint" "Capacitor_SMD:C_2220_5750Metric_Pad1.97x5.40mm_HandSolder"
 			(at 190.1952 54.61 0)
 			(effects
@@
 			)
 		)
-		(property "Footprint" ""
+		(property "Footprint" "Capacitor_SMD:C_2220_5750Metric_Pad1.97x5.40mm_HandSolder"
 			(at 166.0652 54.61 0)
 			(effects
@@
 			)
 		)
-		(property "Footprint" ""
+		(property "Footprint" "My_Capacitor_THT:C_Rect_L42.0mm_W20.0mm_PW37.50mm_PL10.2mm_C4AU"
 			(at 139.3952 54.61 0)
 			(effects
@@
 			)
 		)
-		(property "Value" "R"
+		(property "Value" "100k"
 			(at 113.03 62.2299 0)
 			(effects
@@
 			)
 		)
-		(property "Footprint" ""
+		(property "Footprint" "Resistor_THT:R_Axial_DIN0617_L17.0mm_D6.0mm_P30.48mm_Horizontal"
 			(at 108.712 60.96 90)
 			(effects
@@
 			)
 		)
+		(property "Part #" "RR03J100KTB"
+			(at 110.49 60.96 0)
+			(effects
+				(font
+					(size 1.27 1.27)
+				)
+				(hide yes)
+			)
+		)
 		(pin "2"
 		)
@@
 			)
 		)
-		(property "Footprint" ""
+		(property "Footprint" "Capacitor_SMD:C_2220_5750Metric_Pad1.97x5.40mm_HandSolder"
 			(at 202.8952 54.61 0)
 			(effects
@@
 			)
 		)
-		(property "Value" "R"
+		(property "Value" "100k"
 			(at 113.03 43.1799 0)
 			(effects
@@
 			)
 		)
-		(property "Footprint" ""
+		(property "Footprint" "Resistor_THT:R_Axial_DIN0617_L17.0mm_D6.0mm_P30.48mm_Horizontal"
 			(at 108.712 41.91 90)
 			(effects
@@
 			(at 110.49 41.91 0)
 			(effects
+				(font
+					(size 1.27 1.27)
+				)
+				(hide yes)
+			)
+		)
+		(property "Part #" "RR03J100KTB"
+			(at 110.49 41.91 0)
+			(effects

Commit message: designator + part n°
Parts:
- removed Q1, Q2: C3M0075120K, Package_TO_SOT_THT:TO-247-4_Vertical, symbol HalfBridge_SiC:C3M0075120K
- added Q1, Q2: C3M0040120K, Package_TO_SOT_THT:TO-247-4_Vertical, symbol My_Transistor_FET:C3M0040120K
- C1: value C -> 10u; Part # (none) -> C4AUNBW5100M3FJ
- C2, C3, C4, C5: value C -> 100n; Part # (none) -> C2220C104KDRACTU
- renumbered R36 to R2, R37 to R3, R2 to R4, R3 to R5
Connections:
- net dcn: now also Q2.2 (S)
- net dcp: now also Q1.1 (D)
- net gh: now also Q1.4 (G)
- net gl: now also Q2.4 (G)
- net kh: now also Q1.3 (DS)
- net kl: now also Q2.3 (DS)
- net ph: now also Q1.2 (S), Q2.1 (D)
Other:
- moved on the sheet: C2

Commit message: titles
Parts:
- Q1, Q2: Part # (none) -> C3M0040120K
Changed lines of the file:
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@@
+			)
+		)
+		(property "Part #" "C3M0040120K"
+			(at 227.33 43.18 0)
+			(effects
+				(font
+					(size 1.27 1.27)
+				)
+				(hide yes)
 			)
 		)
@@
 			(at 227.33 59.69 0)
 			(effects
+				(font
+					(size 1.27 1.27)
+				)
+				(hide yes)
+			)
+		)
+		(property "Part #" "C3M0040120K"
+			(at 227.33 59.69 0)
+			(effects
