File: pcb/HalfBridge_SiC/HalfBridge_SiC.kicad_sch (KiCad schematic)
At the start: 3 parts, among them J1 Screw_Terminal_01x02

Commit message: cap
Parts:
- added J2: 413638-E, My_Connector:TEConnectivity_413638E, symbol My_Connector:413638-E
Changed lines of the file:
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@@
 	(wire
 		(pts
-			(xy 59.69 60.96) (xy 54.61 60.96)
+			(xy 59.69 72.39) (xy 54.61 72.39)
 		)
 		(stroke
@@
 	(wire
 		(pts
-			(xy 54.61 60.96) (xy 54.61 91.44)
+			(xy 54.61 72.39) (xy 54.61 91.44)
 		)
 		(stroke
@@
 	(wire
 		(pts
-			(xy 53.34 58.42) (xy 53.34 88.9)
-		)
-		(stroke
-			(width 0)
-			(type default)
-		)
-	)
-	(wire
-		(pts
-			(xy 93.98 97.79) (xy 102.87 97.79)
+			(xy 53.34 69.85) (xy 53.34 88.9)
+		)
+		(stroke
+			(width 0)
+			(type default)
+		)
+	)
+	(wire
+		(pts
+			(xy 92.71 97.79) (xy 102.87 97.79)
 		)
 		(stroke
@@
 	(wire
 		(pts
-			(xy 59.69 58.42) (xy 53.34 58.42)
-		)
-		(stroke
-			(width 0)
-			(type default)
-		)
-	)
-	(wire
-		(pts
-			(xy 99.06 95.25) (xy 102.87 95.25)
-		)
-		(stroke
-			(width 0)
-			(type default)
-		)
-	)
-	(wire
-		(pts
-			(xy 99.06 85.09) (xy 99.06 95.25)
-		)
-		(stroke
-			(width 0)
-			(type default)
-		)
-	)
-	(wire
-		(pts
-			(xy 86.36 63.5) (xy 91.44 63.5)
+			(xy 59.69 69.85) (xy 53.34 69.85)
+		)
+		(stroke
+			(width 0)
+			(type default)
+		)
+	)
+	(wire
+		(pts
+			(xy 93.98 95.25) (xy 102.87 95.25)
+		)
+		(stroke
+			(width 0)
+			(type default)
+		)
+	)
+	(wire
+		(pts
+			(xy 93.98 85.09) (xy 93.98 95.25)
+		)
+		(stroke
+			(width 0)
+			(type default)
+		)
+	)
+	(wire
+		(pts
+			(xy 86.36 74.93) (xy 91.44 74.93)
 		)
 		(stroke
@@
 	(wire
 		(pts
-			(xy 91.44 63.5) (xy 91.44 90.17)
-		)
-		(stroke
-			(width 0)
-			(type default)
-		)
-	)
-	(wire
-		(pts
-			(xy 93.98 85.09) (xy 99.06 85.09)
+			(xy 91.44 74.93) (xy 91.44 90.17)
 		)
 		(stroke
@@
 	(wire
 		(pts
-			(xy 86.36 60.96) (xy 92.71 60.96)
-		)
-		(stroke
-			(width 0)
-			(type default)
-		)
-	)
-	(wire
-		(pts
-			(xy 86.36 58.42) (xy 93.98 58.42)
+			(xy 86.36 72.39) (xy 92.71 72.39)
+		)
+		(stroke
+			(width 0)
+			(type default)
+		)
+	)
+	(wire
+		(pts
+			(xy 86.36 69.85) (xy 93.98 69.85)
 		)
 		(stroke
@@
 	(wire
 		(pts
-			(xy 93.98 87.63) (xy 93.98 97.79)
+			(xy 92.71 87.63) (xy 92.71 97.79)
 		)
 		(stroke
@@
 	(wire
 		(pts
-			(xy 92.71 60.96) (xy 92.71 87.63)
-		)
-		(stroke
-			(width 0)
-			(type default)
-		)
-	)
-	(wire
-		(pts
-			(xy 92.71 87.63) (xy 93.98 87.63)
-		)
-		(stroke
-			(width 0)
-			(type default)
-		)
-	)
-	(wire
-		(pts
-			(xy 93.98 58.42) (xy 93.98 85.09)
+			(xy 92.71 72.39) (xy 92.71 87.63)
+		)
+		(stroke
+			(width 0)
+			(type default)
+		)
+	)
+	(wire
+		(pts
+			(xy 93.98 69.85) (xy 93.98 85.09)
 		)
 		(stroke
@@
 		)
 	)
+	(symbol
+		(lib_id "My_Connector:413638-E")
+		(at 228.6 96.52 0)
+		(unit 1)
+		(exclude_from_sim no)
+		(in_bom yes)
+		(on_board yes)
+		(dnp no)
+		(fields_autoplaced yes)
+		(property "Reference" "J2"
+			(at 228.6 78.74 0)
+			(effects
+				(font
+					(size 1.27 1.27)
+				)
+			)
+		)
+		(property "Value" "413638-E"
+			(at 228.6 81.28 0)
+			(effects
+				(font
+					(size 1.27 1.27)
+				)
+			)
+		)
+		(property "Footprint" "My_Connector:TEConnectivity_413638E"
+			(at 250.19 191.44 0)
+			(effects
+				(font
+					(size 1.27 1.27)
+				)
+				(justify left top)
+				(hide yes)
+			)
+		)
+		(property "Datasheet" "https://www.erni.com/fileadmin/import/products/assets/DC0002089.PDF"
+			(at 250.19 291.44 0)
+			(effects
+				(font
+					(size 1.27 1.27)
+				)
+				(justify left top)
+				(hide yes)
+			)
+		)
+		(property "Description" "15 Position Header, Male Blades Connector Solder 0.300\" (7.62mm) Through Hole, Right Angle"
+			(at 228.6 96.52 0)
+			(effects
+				(font
+					(size 1.27 1.27)
+				)
+				(hide yes)
+			)
+		)
+		(property "Height" "13"
+			(at 250.19 491.44 0)
+			(effects
+				(font
+					(size 1.27 1.27)
+				)
+				(justify left top)
+				(hide yes)
+			)
+		)
+		(property "Manufacturer_Name" "TE Connectivity"
+			(at 250.19 591.44 0)
+			(effects
+				(font
+					(size 1.27 1.27)
+				)
+				(justify left top)
+				(hide yes)
+			)
+		)
+		(property "Manufacturer_Part_Number" "413638-E"
+			(at 250.19 691.44 0)
+			(effects
+				(font
+					(size 1.27 1.27)
+				)
+				(justify left top)
+				(hide yes)
+			)
+		)
+		(property "Mouser Part Number" ""
+			(at 250.19 791.44 0)
+			(effects
+				(font
+					(size 1.27 1.27)
+				)
+				(justify left top)
+				(hide yes)
+			)
+		)
+		(property "Mouser Price/Stock" ""
+			(at 250.19 891.44 0)
+			(effects
+				(font
+					(size 1.27 1.27)
+				)
+				(justify left top)
+				(hide yes)
+			)
+		)
+		(property "Arrow Part Number" ""
+			(at 250.19 991.44 0)
+			(effects
+				(font
+					(size 1.27 1.27)
+				)
+				(justify left top)
+				(hide yes)
+			)
+		)
+		(property "Arrow Price/Stock" ""
+			(at 250.19 1091.44 0)
+			(effects
+				(font
+					(size 1.27 1.27)
+				)
+				(justify left top)
+				(hide yes)
+			)
+		)
+		(pin "D22"
+		)
+		(pin "Z16"
+		)
+		(pin "Z24"
+		)
+		(pin "MH1"
+		)
+		(pin "Z4"
+		)
+		(pin "D10"
+		)
+		(pin "D18"
+		)
+		(pin "Z32"
+		)
+		(pin "D30"
+		)
+		(pin "MH2"
+		)
+		(pin "D26"
+		)
+		(pin "D14"
+		)
+		(pin "Z28"
+		)
+		(pin "Z8"
+		)
+		(pin "Z20"
+		)
+		(pin "D6"
+		)
+		(pin "Z12"
+		)
+		(instances
+			(project ""
+				(path "/3c187ffa-7f66-4861-b077-b6965c821fc2"
+					(reference "J2")
+					(unit 1)
+				)
+			)
+		)
+	)
 	(sheet
-		(at 59.69 54.61)
+		(at 59.69 66.04)
 		(size 26.67 10.16)
 		(fields_autoplaced yes)
@@
 		)
 		(property "Sheetname" "HalfBridge_Diff"
-			(at 59.69 53.8984 0)
+			(at 59.69 65.3284 0)
 			(effects
 				(font
@@
 		)
 		(property "Sheetfile" "HalfBridge_Diff.kicad_sch"
-			(at 59.69 65.3546 0)
+			(at 59.69 76.7846 0)
 			(effects
 				(font
@@
 		)
 		(pin "vcc" input
-			(at 59.69 58.42 180)
+			(at 59.69 69.85 180)
 			(effects
 				(font
@@
 		)
 		(pin "gnd" input
-			(at 59.69 60.96 180)
+			(at 59.69 72.39 180)
 			(effects
 				(font
@@
 		)
 		(pin "inb_d" output
-			(at 86.36 60.96 0)
+			(at 86.36 72.39 0)
 			(effects
 				(font
@@
 		)
 		(pin "ina_d" output
-			(at 86.36 58.42 0)
+			(at 86.36 69.85 0)
 			(effects
 				(font
@@
 		)
 		(pin "inen_d" output
-			(at 86.36 63.5 0)
-			(effects
-				(font
+			(at 86.36 74.93 0)
+			(effects
+				(font

Commit message: pcb + horizontal of
Connections:
- net dcn: now reaches J2.D10
- net dcn: now also J2.D6, J2.Z4, J2.Z8
- net dcp: now reaches J2.D14
- net dcp: now also J2.D18, J2.Z12, J2.Z16
- net ph: now reaches J2.D22
- net ph: now also J2.D26, J2.Z20, J2.Z24
Other:
- moved on the sheet: J2
Changed lines of the file:
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@@
 	(wire
 		(pts
-			(xy 142.24 102.87) (xy 154.94 102.87)
+			(xy 142.24 102.87) (xy 148.59 102.87)
 		)
 		(stroke
@@
 	(wire
 		(pts
+			(xy 181.61 102.87) (xy 190.5 102.87)
+		)
+		(stroke
+			(width 0)
+			(type default)
+		)
+	)
+	(wire
+		(pts
 			(xy 54.61 72.39) (xy 54.61 91.44)
 		)
@@
 	(wire
 		(pts
-			(xy 142.24 97.79) (xy 154.94 97.79)
+			(xy 142.24 97.79) (xy 148.59 97.79)
 		)
 		(stroke
@@
 	(wire
 		(pts
-			(xy 142.24 100.33) (xy 154.94 100.33)
+			(xy 142.24 100.33) (xy 148.59 100.33)
 		)
 		(stroke
@@
 	(wire
 		(pts
-			(xy 142.24 95.25) (xy 154.94 95.25)
+			(xy 142.24 95.25) (xy 148.59 95.25)
 		)
 		(stroke
@@
 	(wire
 		(pts
+			(xy 181.61 99.06) (xy 190.5 99.06)
+		)
+		(stroke
+			(width 0)
+			(type default)
+		)
+	)
+	(wire
+		(pts
 			(xy 92.71 72.39) (xy 92.71 87.63)
 		)
@@
 	(wire
 		(pts
+			(xy 181.61 95.25) (xy 190.5 95.25)
+		)
+		(stroke
+			(width 0)
+			(type default)
+		)
+	)
+	(wire
+		(pts
 			(xy 44.45 119.38) (xy 54.61 119.38)
 		)
@@
 			(width 0)
 			(type default)
+		)
+	)
+	(label "dcn"
+		(at 241.3 102.87 0)
+		(fields_autoplaced yes)
+		(effects
+			(font
+				(size 1.27 1.27)
+			)
+			(justify left bottom)
+		)
+	)
+	(label "dcp"
+		(at 215.9 95.25 180)
+		(fields_autoplaced yes)
+		(effects
+			(font
+				(size 1.27 1.27)
+			)
+			(justify right bottom)
+		)
+	)
+	(label "dcp"
+		(at 241.3 97.79 0)
+		(fields_autoplaced yes)
+		(effects
+			(font
+				(size 1.27 1.27)
+			)
+			(justify left bottom)
+		)
+	)
+	(label "ph"
+		(at 241.3 92.71 0)
+		(fields_autoplaced yes)
+		(effects
+			(font
+				(size 1.27 1.27)
+			)
+			(justify left bottom)
+		)
+	)
+	(label "dcn"
+		(at 241.3 105.41 0)
+		(fields_autoplaced yes)
+		(effects
+			(font
+				(size 1.27 1.27)
+			)
+			(justify left bottom)
+		)
+	)
+	(label "dcp"
+		(at 182.88 99.06 0)
+		(fields_autoplaced yes)
+		(effects
+			(font
+				(size 1.27 1.27)
+			)
+			(justify left bottom)
+		)
+	)
+	(label "ph"
+		(at 215.9 92.71 180)
+		(fields_autoplaced yes)
+		(effects
+			(font
+				(size 1.27 1.27)
+			)
+			(justify right bottom)
+		)
+	)
+	(label "dcn"
+		(at 215.9 102.87 180)
+		(fields_autoplaced yes)
+		(effects
+			(font
+				(size 1.27 1.27)
+			)
+			(justify right bottom)
+		)
+	)
+	(label "ph"
+		(at 215.9 90.17 180)
+		(fields_autoplaced yes)
+		(effects
+			(font
+				(size 1.27 1.27)
+			)
+			(justify right bottom)
+		)
+	)
+	(label "dcp"
+		(at 241.3 100.33 0)
+		(fields_autoplaced yes)
+		(effects
+			(font
+				(size 1.27 1.27)
+			)
+			(justify left bottom)
+		)
+	)
+	(label "dcp"
+		(at 215.9 97.79 180)
+		(fields_autoplaced yes)
+		(effects
+			(font
+				(size 1.27 1.27)
+			)
+			(justify right bottom)
+		)
+	)
+	(label "ph"
+		(at 182.88 95.25 0)
+		(fields_autoplaced yes)
+		(effects
+			(font
+				(size 1.27 1.27)
+			)
+			(justify left bottom)
+		)
+	)
+	(label "dcn"
+		(at 182.88 102.87 0)
+		(fields_autoplaced yes)
+		(effects
+			(font
+				(size 1.27 1.27)
+			)
+			(justify left bottom)
+		)
+	)
+	(label "dcn"
+		(at 215.9 100.33 180)
+		(fields_autoplaced yes)
+		(effects
+			(font
+				(size 1.27 1.27)
+			)
+			(justify right bottom)
+		)
+	)
+	(label "ph"
+		(at 241.3 95.25 0)
+		(fields_autoplaced yes)
+		(effects
+			(font
+				(size 1.27 1.27)
+			)
+			(justify left bottom)
 		)
 	)
@@
 	(symbol
 		(lib_id "My_Connector:413638-E")
-		(at 228.6 96.52 0)
+		(at 228.6 95.25 0)
+		(mirror x)
 		(unit 1)
 		(exclude_from_sim no)
@@
 		(on_board yes)
 		(dnp no)
-		(fields_autoplaced yes)
 		(property "Reference" "J2"
-			(at 228.6 78.74 0)
+			(at 228.6 113.03 0)
 			(effects
 				(font
@@
 		)
 		(property "Value" "413638-E"
-			(at 228.6 81.28 0)
+			(at 228.6 110.49 0)
 			(effects
 				(font
@@
 		)
 		(property "Footprint" "My_Connector:TEConnectivity_413638E"
-			(at 250.19 191.44 0)
+			(at 250.19 0.33 0)
 			(effects
 				(font
@@
 		)
 		(property "Datasheet" "https://www.erni.com/fileadmin/import/products/assets/DC0002089.PDF"
-			(at 250.19 291.44 0)
+			(at 250.19 -99.67 0)
 			(effects
 				(font
@@
 		)
 		(property "Description" "15 Position Header, Male Blades Connector Solder 0.300\" (7.62mm) Through Hole, Right Angle"
-			(at 228.6 96.52 0)
+			(at 228.6 95.25 0)
 			(effects
 				(font
@@
 		)
 		(property "Height" "13"
-			(at 250.19 491.44 0)
+			(at 250.19 -299.67 0)
 			(effects
 				(font
@@
 		)
 		(property "Manufacturer_Name" "TE Connectivity"
-			(at 250.19 591.44 0)
+			(at 250.19 -399.67 0)
 			(effects
 				(font
@@
 		)
 		(property "Manufacturer_Part_Number" "413638-E"
-			(at 250.19 691.44 0)
+			(at 250.19 -499.67 0)
 			(effects
 				(font
@@
 		)
 		(property "Mouser Part Number" ""
-			(at 250.19 791.44 0)
+			(at 250.19 -599.67 0)
 			(effects
 				(font
@@
 		)
 		(property "Mouser Price/Stock" ""
-			(at 250.19 891.44 0)
+			(at 250.19 -699.67 0)
 			(effects
 				(font
@@
 		)
 		(property "Arrow Part Number" ""
-			(at 250.19 991.44 0)
+			(at 250.19 -799.67 0)
 			(effects
 				(font
@@
 		)
 		(property "Arrow Price/Stock" ""
-			(at 250.19 1091.44 0)
+			(at 250.19 -899.67 0)
 			(effects
 				(font
@@
 	)
 	(sheet
-		(at 154.94 92.71)
+		(at 148.59 92.71)
 		(size 33.02 12.7)
 		(fields_autoplaced yes)
@@
 		)
 		(property "Sheetname" "HalfBridge_Power"
-			(at 154.94 91.9984 0)
+			(at 148.59 91.9984 0)
 			(effects
 				(font
@@
 		)
 		(property "Sheetfile" "HalfBridge_Power.kicad_sch"
-			(at 154.94 105.9946 0)
+			(at 148.59 105.9946 0)
 			(effects
 				(font
@@
 		)
 		(pin "ph" output
-			(at 187.96 95.25 0)
+			(at 181.61 95.25 0)
 			(effects
 				(font
@@
 		)
 		(pin "dcp" input
-			(at 187.96 99.06 0)
+			(at 181.61 99.06 0)
 			(effects
 				(font
@@
 		)
 		(pin "dcn" input
-			(at 187.96 102.87 0)
+			(at 181.61 102.87 0)
 			(effects
 				(font
@@
 		)
 		(pin "gh" input
-			(at 154.94 95.25 180)
+			(at 148.59 95.25 180)
 			(effects
 				(font
@@
 		)
 		(pin "kh" input
-			(at 154.94 97.79 180)
+			(at 148.59 97.79 180)
 			(effects
 				(font
@@
 		)
 		(pin "gl" input
-			(at 154.94 100.33 180)
+			(at 148.59 100.33 180)
 			(effects
 				(font
@@
 		)
 		(pin "kl" input
-			(at 154.94 102.87 180)
-			(effects
-				(font
+			(at 148.59 102.87 180)
+			(effects
+				(font

Commit message: vgatereg + route + hsink
Parts:
- removed J1: Screw_Terminal_01x02, TerminalBlock_Phoenix:TerminalBlock_Phoenix_PT-1,5-2-3.5-H_1x02_P3.50mm_Horizontal, symbol Connector:Screw_Terminal_01x02
- added J1: Conn_01x02, Connector_Phoenix_SPT:PhoenixContact_SPT_1.5_2-H-3.5_1x02_P3.5mm_Horizontal, symbol Connector_Generic:Conn_01x02
Connections:
- net HalfBridge_Diff/gnd: now also J1.2 (Pin_2)
- net HalfBridge_Diff/vcc: now also J1.1 (Pin_1)
- net lvcc: now reaches D1.1 (K), R1.1
Other:
- note added: "Vcc = 5V"
Changed lines of the file:
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@@
+		)
+	)
+	(text "Vcc = 5V"
+		(exclude_from_sim no)
+		(at 39.878 92.202 0)
+		(effects
+			(font
+				(size 1.27 1.27)
+			)
 		)
 	)
@@
 		)
 	)
+	(label "lvcc"
+		(at 44.45 111.76 0)
+		(fields_autoplaced yes)
+		(effects
+			(font
+				(size 1.27 1.27)
+			)
+			(justify left bottom)
+		)
+	)
 	(label "ph"
 		(at 215.9 90.17 180)
@@
 	)
 	(symbol
-		(lib_id "Connector:Screw_Terminal_01x02")
+		(lib_id "Connector_Generic:Conn_01x02")
 		(at 36.83 95.25 0)
 		(mirror y)
@@
 			)
 		)
-		(property "Value" "Screw_Terminal_01x02"
+		(property "Value" "Conn_01x02"
 			(at 34.29 97.7899 0)
 			(effects
@@
 			)
 		)
-		(property "Footprint" "TerminalBlock_Phoenix:TerminalBlock_Phoenix_PT-1,5-2-3.5-H_1x02_P3.50mm_Horizontal"
+		(property "Footprint" "Connector_Phoenix_SPT:PhoenixContact_SPT_1.5_2-H-3.5_1x02_P3.5mm_Horizontal"
 			(at 36.83 95.25 0)
 			(effects
@@
 			)
 		)
-		(property "Description" "Generic screw terminal, single row, 01x02, script generated (kicad-library-utils/schlib/autogen/connector/)"
+		(property "Description" "Generic connector, single row, 01x02, script generated (kicad-library-utils/schlib/autogen/connector/)"
 			(at 36.83 95.25 0)
 			(effects

Commit message: comment + gdriver + logo
Other:
- title: (none) -> Half Bridge converter with SiC-MOSFETs
Changed lines of the file:
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@@
 	(generator_version "8.0")
 	(paper "A4")
+	(title_block
+		(title "Half Bridge converter with SiC-MOSFETs")
+		(rev "1")
+	)
 	(junction
 		(at 44.45 95.25)

Commit message: part number
Parts:
- J2: Manufacturer Part Number (none) -> 413638-E; Manufacturer_Part_Number 413638-E -> (none)
Changed lines of the file:
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@@
 			)
 		)
-		(property "Manufacturer_Part_Number" "413638-E"
+		(property "Manufacturer Part Number" "413638-E"
 			(at 250.19 -499.67 0)
 			(effects
