File: pcb/HalfBridge_SiC/HalfBridge_SiC.kicad_sch (KiCad schematic)
At the start: 4 parts, among them J1 Conn_01x02, J2 413638-E

Commit message: backplane
Parts:
- added J12, J13, J14, J15: Conn_01x01, My_Connector:WP_SMRA_74663025R, symbol Connector_Generic:Conn_01x01
- J2: now not fitted
Connections:
- net dcn: now also J12.1 (Pin_1)
- net dcp: now also J2.D22, J2.D26, J2.Z20, J2.Z24, J14.1 (Pin_1); no longer J2.D14, J2.D18, J2.Z12, J2.Z16
- net ph: no longer J2.D22, J2.D26, J2.Z20, J2.Z24
- net pho: now reaches J2.D30
- net pho: now also J2.Z28, J2.Z32, J15.1 (Pin_1)
- new net dcm: J13.1 (Pin_1), J2.D14, J2.D18, J2.Z12, J2.Z16
Other:
- added sheet HalfBridge_InMeasurement (HalfBridge_InMeasurement.kicad_sch)
- sheet HalfBridge_Power ports: added dcm; removed none
