File: pcb/HalfBridge_SiC/HalfBridge_SiC.kicad_sch (KiCad schematic)
At the start: 8 parts, among them J1 Conn_01x02, J12 Conn_01x01, J13 Conn_01x01, J14 Conn_01x01, J15 Conn_01x01, J2 413638-E

Commit message: local lib
Parts:
- D1: symbol Device:LED -> HalfBridge_SiC:LED
- J1: symbol Connector_Generic:Conn_01x02 -> HalfBridge_SiC:Conn_01x02
- J12, J13, J14, J15: footprint My_Connector:WP_SMRA_74663025R -> My_Connector:WP_SMRA_77466303; symbol Connector_Generic:Conn_01x01 -> HalfBridge_SiC:Conn_01x01
- J2: symbol My_Connector:413638-E -> HalfBridge_SiC:413638-E
- R1: symbol Device:R -> HalfBridge_SiC:R
Other:
- company: (none) -> Dr.-Ing. Alan H. Wilson Veas
- moved on the sheet: J12, J13, J14, J15
Changed lines of the file:
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@@
 		(title "Half Bridge converter with SiC-MOSFETs")
 		(rev "1")
+		(company "Dr.-Ing. Alan H. Wilson Veas")
+		(comment 1 "AHWV")
 	)
 	(junction
@@
 	)
 	(label "dcm"
-		(at 250.19 38.1 180)
+		(at 251.46 62.23 180)
 		(fields_autoplaced yes)
 		(effects
@@
 	)
 	(label "dcp"
-		(at 250.19 44.45 180)
+		(at 251.46 68.58 180)
 		(fields_autoplaced yes)
 		(effects
@@
 	)
 	(label "pho"
-		(at 250.19 50.8 180)
+		(at 251.46 74.93 180)
 		(fields_autoplaced yes)
 		(effects
@@
 	)
 	(label "dcn"
-		(at 250.19 31.75 180)
+		(at 251.46 55.88 180)
 		(fields_autoplaced yes)
 		(effects
@@
 	)
 	(symbol
-		(lib_id "Connector_Generic:Conn_01x02")
+		(lib_id "HalfBridge_SiC:Conn_01x02")
 		(at 36.83 95.25 0)
 		(mirror y)
@@
 	)
 	(symbol
-		(lib_id "Connector_Generic:Conn_01x01")
-		(at 255.27 38.1 0)
+		(lib_id "HalfBridge_SiC:Conn_01x01")
+		(at 256.54 62.23 0)
 		(unit 1)
 		(exclude_from_sim no)
@@
 		(fields_autoplaced yes)
 		(property "Reference" "J13"
-			(at 257.81 36.8299 0)
+			(at 259.08 60.9599 0)
 			(effects
 				(font
@@
 		)
 		(property "Value" "Conn_01x01"
-			(at 257.81 39.3699 0)
+			(at 259.08 63.4999 0)
 			(effects
 				(font
@@
 			)
 		)
-		(property "Footprint" "My_Connector:WP_SMRA_74663025R"
-			(at 255.27 38.1 0)
+		(property "Footprint" "My_Connector:WP_SMRA_77466303"
+			(at 256.54 62.23 0)
 			(effects
 				(font
@@
 		)
 		(property "Datasheet" "~"
-			(at 255.27 38.1 0)
+			(at 256.54 62.23 0)
 			(effects
 				(font
@@
 		)
 		(property "Description" "Generic connector, single row, 01x01, script generated (kicad-library-utils/schlib/autogen/connector/)"
-			(at 255.27 38.1 0)
+			(at 256.54 62.23 0)
 			(effects
 				(font
@@
 	)
 	(symbol
-		(lib_id "Connector_Generic:Conn_01x01")
-		(at 255.27 44.45 0)
+		(lib_id "HalfBridge_SiC:Conn_01x01")
+		(at 256.54 68.58 0)
 		(unit 1)
 		(exclude_from_sim no)
@@
 		(fields_autoplaced yes)
 		(property "Reference" "J14"
-			(at 257.81 43.1799 0)
+			(at 259.08 67.3099 0)
 			(effects
 				(font
@@
 		)
 		(property "Value" "Conn_01x01"
-			(at 257.81 45.7199 0)
+			(at 259.08 69.8499 0)
 			(effects
 				(font
@@
 			)
 		)
-		(property "Footprint" "My_Connector:WP_SMRA_74663025R"
-			(at 255.27 44.45 0)
+		(property "Footprint" "My_Connector:WP_SMRA_77466303"
+			(at 256.54 68.58 0)
 			(effects
 				(font
@@
 		)
 		(property "Datasheet" "~"
-			(at 255.27 44.45 0)
+			(at 256.54 68.58 0)
 			(effects
 				(font
@@
 		)
 		(property "Description" "Generic connector, single row, 01x01, script generated (kicad-library-utils/schlib/autogen/connector/)"
-			(at 255.27 44.45 0)
+			(at 256.54 68.58 0)
 			(effects
 				(font
@@
 	)
 	(symbol
-		(lib_id "Device:R")
+		(lib_id "HalfBridge_SiC:R")
 		(at 44.45 115.57 0)
 		(unit 1)
@@
 	)
 	(symbol
-		(lib_id "Connector_Generic:Conn_01x01")
-		(at 255.27 50.8 0)
+		(lib_id "HalfBridge_SiC:Conn_01x01")
+		(at 256.54 74.93 0)
 		(unit 1)
 		(exclude_from_sim no)
@@
 		(fields_autoplaced yes)
 		(property "Reference" "J15"
-			(at 257.81 49.5299 0)
+			(at 259.08 73.6599 0)
 			(effects
 				(font
@@
 		)
 		(property "Value" "Conn_01x01"
-			(at 257.81 52.0699 0)
+			(at 259.08 76.1999 0)
 			(effects
 				(font
@@
 			)
 		)
-		(property "Footprint" "My_Connector:WP_SMRA_74663025R"
-			(at 255.27 50.8 0)
+		(property "Footprint" "My_Connector:WP_SMRA_77466303"
+			(at 256.54 74.93 0)
 			(effects
 				(font
@@
 		)
 		(property "Datasheet" "~"
-			(at 255.27 50.8 0)
+			(at 256.54 74.93 0)
 			(effects
 				(font
@@
 		)
 		(property "Description" "Generic connector, single row, 01x01, script generated (kicad-library-utils/schlib/autogen/connector/)"
-			(at 255.27 50.8 0)
+			(at 256.54 74.93 0)
 			(effects
 				(font
@@
 	)
 	(symbol
-		(lib_id "Connector_Generic:Conn_01x01")
-		(at 255.27 31.75 0)
+		(lib_id "HalfBridge_SiC:Conn_01x01")
+		(at 256.54 55.88 0)
 		(unit 1)
 		(exclude_from_sim no)
@@
 		(fields_autoplaced yes)
 		(property "Reference" "J12"
-			(at 257.81 30.4799 0)
+			(at 259.08 54.6099 0)
 			(effects
 				(font
@@
 		)
 		(property "Value" "Conn_01x01"
-			(at 257.81 33.0199 0)
+			(at 259.08 57.1499 0)
 			(effects
 				(font
@@
 			)
 		)
-		(property "Footprint" "My_Connector:WP_SMRA_74663025R"
-			(at 255.27 31.75 0)
+		(property "Footprint" "My_Connector:WP_SMRA_77466303"
+			(at 256.54 55.88 0)
 			(effects
 				(font
@@
 		)
 		(property "Datasheet" "~"
-			(at 255.27 31.75 0)
+			(at 256.54 55.88 0)
 			(effects
 				(font
@@
 		)
 		(property "Description" "Generic connector, single row, 01x01, script generated (kicad-library-utils/schlib/autogen/connector/)"
-			(at 255.27 31.75 0)
+			(at 256.54 55.88 0)
 			(effects
 				(font
@@
 	)
 	(symbol
-		(lib_id "Device:LED")
+		(lib_id "HalfBridge_SiC:LED")
 		(at 44.45 105.41 90)
 		(unit 1)
@@
 	)
 	(symbol
-		(lib_id "My_Connector:413638-E")
+		(lib_id "HalfBridge_SiC:413638-E")
 		(at 257.81 95.25 0)
 		(mirror x)

Commit message: backplane + external lib
Parts:
- removed J2: 413638-E, My_Connector:TEConnectivity_413638E, symbol HalfBridge_SiC:413638-E
- added J2: 413638-E, My_Connector:TEConnectivity_413638E, symbol My_Connector:413638-E
- D1: footprint LED_SMD:LED_0603_1608Metric_Pad1.05x0.95mm_HandSolder -> (none)
- J1: footprint Connector_Phoenix_SPT:PhoenixContact_SPT_1.5_2-H-3.5_1x02_P3.5mm_Horizontal -> (none)
- R1: footprint Resistor_SMD:R_0603_1608Metric -> (none)
Connections:
- net dcm: now also J2.D14, J2.D18, J2.Z12, J2.Z16
- net dcn: now also J2.D10, J2.D6, J2.Z4, J2.Z8
- net dcp: now also J2.D22, J2.D26, J2.Z20, J2.Z24
- net pho: now also J2.D30, J2.Z28, J2.Z32
Changed lines of the file:
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@@
 			)
 		)
-		(property "Footprint" "Connector_Phoenix_SPT:PhoenixContact_SPT_1.5_2-H-3.5_1x02_P3.5mm_Horizontal"
+		(property "Footprint" ""
 			(at 36.83 95.25 0)
 			(effects
@@
 			)
 		)
-		(property "Footprint" "Resistor_SMD:R_0603_1608Metric"
+		(property "Footprint" ""
 			(at 42.672 115.57 90)
 			(effects
@@
 			)
 		)
-		(property "Footprint" "LED_SMD:LED_0603_1608Metric_Pad1.05x0.95mm_HandSolder"
+		(property "Footprint" ""
 			(at 44.45 105.41 0)
 			(effects
@@
 	)
 	(symbol
-		(lib_id "HalfBridge_SiC:413638-E")
+		(lib_id "My_Connector:413638-E")
 		(at 257.81 95.25 0)
 		(mirror x)
@@
 			)
 		)
-		(property "Height" "13"
-			(at 279.4 -299.67 0)
-			(effects
-				(font
-					(size 1.27 1.27)
-				)
-				(justify left top)
-				(hide yes)
-			)
-		)
-		(property "Manufacturer_Name" "TE Connectivity"
-			(at 279.4 -399.67 0)
-			(effects
-				(font
-					(size 1.27 1.27)
-				)
-				(justify left top)
-				(hide yes)
-			)
-		)
-		(property "Manufacturer Part Number" "413638-E"
-			(at 250.19 -499.67 0)
-			(effects
-				(font
-					(size 1.27 1.27)
-				)
-				(justify left top)
-				(hide yes)
-			)
-		)
-		(property "Mouser Part Number" ""
-			(at 279.4 -599.67 0)
-			(effects
-				(font
-					(size 1.27 1.27)
-				)
-				(justify left top)
-				(hide yes)
-			)
-		)
-		(property "Mouser Price/Stock" ""
-			(at 279.4 -699.67 0)
-			(effects
-				(font
-					(size 1.27 1.27)
-				)
-				(justify left top)
-				(hide yes)
-			)
-		)
-		(property "Arrow Part Number" ""
-			(at 279.4 -799.67 0)
-			(effects
-				(font
-					(size 1.27 1.27)
-				)
-				(justify left top)
-				(hide yes)
-			)
-		)
-		(property "Arrow Price/Stock" ""
-			(at 279.4 -899.67 0)
-			(effects
-				(font
-					(size 1.27 1.27)
-				)
-				(justify left top)
-				(hide yes)
-			)
+		(property "Part #" "413638-E"
+			(at 257.81 95.25 0)
+			(effects
+				(font
+					(size 1.27 1.27)
+				)
+				(hide yes)
+			)
+		)
+		(pin "D14"
+		)
+		(pin "Z24"
+		)
+		(pin "Z32"
+		)
+		(pin "MH1"
+		)
+		(pin "Z12"
+		)
+		(pin "Z4"
+		)
+		(pin "Z8"
+		)
+		(pin "D10"
+		)
+		(pin "Z28"
+		)
+		(pin "D26"
+		)
+		(pin "D6"
+		)
+		(pin "D18"
+		)
+		(pin "MH2"
+		)
+		(pin "Z16"
+		)
+		(pin "Z20"
 		)
 		(pin "D22"
 		)
-		(pin "Z16"
-		)
-		(pin "Z24"
-		)
-		(pin "MH1"
-		)
-		(pin "Z4"
-		)
-		(pin "D10"
-		)
-		(pin "D18"
-		)
-		(pin "Z32"
-		)
 		(pin "D30"
 		)
-		(pin "MH2"
-		)
-		(pin "D26"
-		)
-		(pin "D14"
-		)
-		(pin "Z28"
-		)
-		(pin "Z8"
-		)
-		(pin "Z20"
-		)
-		(pin "D6"
-		)
-		(pin "Z12"
-		)
-		(instances
-			(project ""
+		(instances
+			(project "HalfBridge_SiC"
 				(path "/3c187ffa-7f66-4861-b077-b6965c821fc2"
 					(reference "J2")

Commit message: update lib
Parts:
- D1: footprint (none) -> LED_SMD:LED_0603_1608Metric_Pad1.05x0.95mm_HandSolder; Part # (none) -> 150060VS75003
- J1: footprint (none) -> Connector_Phoenix_SPT:PhoenixContact_SPT_1.5_2-H-3.5_1x02_P3.5mm_Horizontal
- J12, J13, J14, J15: footprint My_Connector:WP_SMRA_77466303 -> My_Connector:WP_SMRA_7466303
- J2: now left out of the parts list
- R1: value R -> 330; footprint (none) -> Resistor_SMD:R_0603_1608Metric_Pad0.98x0.95mm_HandSolder
Changed lines of the file:
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@@
 			)
 		)
-		(property "Footprint" ""
+		(property "Footprint" "Connector_Phoenix_SPT:PhoenixContact_SPT_1.5_2-H-3.5_1x02_P3.5mm_Horizontal"
 			(at 36.83 95.25 0)
 			(effects
@@
 			)
 		)
-		(property "Footprint" "My_Connector:WP_SMRA_77466303"
+		(property "Footprint" "My_Connector:WP_SMRA_7466303"
 			(at 256.54 62.23 0)
 			(effects
@@
 			)
 		)
-		(property "Footprint" "My_Connector:WP_SMRA_77466303"
+		(property "Footprint" "My_Connector:WP_SMRA_7466303"
 			(at 256.54 68.58 0)
 			(effects
@@
 			)
 		)
-		(property "Value" "R"
+		(property "Value" "330"
 			(at 46.99 116.8399 0)
 			(effects
@@
 			)
 		)
-		(property "Footprint" ""
+		(property "Footprint" "Resistor_SMD:R_0603_1608Metric_Pad0.98x0.95mm_HandSolder"
 			(at 42.672 115.57 90)
 			(effects
@@
 			)
 		)
-		(property "Footprint" "My_Connector:WP_SMRA_77466303"
+		(property "Footprint" "My_Connector:WP_SMRA_7466303"
 			(at 256.54 74.93 0)
 			(effects
@@
 			)
 		)
-		(property "Footprint" "My_Connector:WP_SMRA_77466303"
+		(property "Footprint" "My_Connector:WP_SMRA_7466303"
 			(at 256.54 55.88 0)
 			(effects
@@
 			)
 		)
-		(property "Footprint" ""
+		(property "Footprint" "LED_SMD:LED_0603_1608Metric_Pad1.05x0.95mm_HandSolder"
 			(at 44.45 105.41 0)
 			(effects
@@
 		(property "Description" "Light emitting diode"
 			(at 44.45 105.41 0)
+			(effects
+				(font
+					(size 1.27 1.27)
+				)
+				(hide yes)
+			)
+		)
+		(property "Part #" "150060VS75003"
+			(at 44.45 105.41 90)
 			(effects
 				(font
@@
 		(unit 1)
 		(exclude_from_sim no)
-		(in_bom yes)
+		(in_bom no)
 		(on_board yes)
 		(dnp yes)

Commit message: filter + sim + assembly3d
Parts:
- J12, J13, J14, J15: Part # (none) -> 7466303
Changed lines of the file:
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@@
+			)
+		)
+		(property "Part #" "7466303"
+			(at 256.54 62.23 0)
+			(effects
+				(font
+					(size 1.27 1.27)
+				)
+				(hide yes)
 			)
 		)
@@
 			)
 		)
+		(property "Part #" "7466303"
+			(at 256.54 68.58 0)
+			(effects
+				(font
+					(size 1.27 1.27)
+				)
+				(hide yes)
+			)
+		)
 		(pin "1"
 		)
@@
 			)
 		)
+		(property "Part #" "7466303"
+			(at 256.54 74.93 0)
+			(effects
+				(font
+					(size 1.27 1.27)
+				)
+				(hide yes)
+			)
+		)
 		(pin "1"
 		)
@@
 			(at 256.54 55.88 0)
 			(effects
+				(font
+					(size 1.27 1.27)
+				)
+				(hide yes)
+			)
+		)
+		(property "Part #" "7466303"
+			(at 256.54 55.88 0)
+			(effects

Commit message: designator + part n°
Parts:
- renumbered J12 to J2, J13 to J3, J14 to J4, J15 to J5, J2 to J6
Changed lines of the file:
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@@
 		(dnp no)
 		(fields_autoplaced yes)
-		(property "Reference" "J13"
+		(property "Reference" "J3"
 			(at 259.08 60.9599 0)
 			(effects
@@
 			(project "HalfBridge_SiC"
 				(path "/3c187ffa-7f66-4861-b077-b6965c821fc2"
-					(reference "J13")
+					(reference "J3")
 					(unit 1)
 				)
@@
 		(dnp no)
 		(fields_autoplaced yes)
-		(property "Reference" "J14"
+		(property "Reference" "J4"
 			(at 259.08 67.3099 0)
 			(effects
@@
 			(project "HalfBridge_SiC"
 				(path "/3c187ffa-7f66-4861-b077-b6965c821fc2"
-					(reference "J14")
+					(reference "J4")
 					(unit 1)
 				)
@@
 		(dnp no)
 		(fields_autoplaced yes)
-		(property "Reference" "J15"
+		(property "Reference" "J5"
 			(at 259.08 73.6599 0)
 			(effects
@@
 			(project "HalfBridge_SiC"
 				(path "/3c187ffa-7f66-4861-b077-b6965c821fc2"
-					(reference "J15")
+					(reference "J5")
 					(unit 1)
 				)
@@
 		(dnp no)
 		(fields_autoplaced yes)
-		(property "Reference" "J12"
+		(property "Reference" "J2"
 			(at 259.08 54.6099 0)
 			(effects
@@
 			(project ""
 				(path "/3c187ffa-7f66-4861-b077-b6965c821fc2"
-					(reference "J12")
+					(reference "J2")
 					(unit 1)
 				)
@@
 		(on_board yes)
 		(dnp yes)
-		(property "Reference" "J2"
+		(property "Reference" "J6"
 			(at 257.81 113.03 0)
 			(effects
@@
 			(project "HalfBridge_SiC"
 				(path "/3c187ffa-7f66-4861-b077-b6965c821fc2"
-					(reference "J2")
-					(unit 1)
-				)
+					(reference "J6")
+					(unit 1)
+				)

Commit message: titles
Parts:
- J1: Part # (none) -> M20-9750242
Changed lines of the file:
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@@
+			)
+		)
+		(property "Part #" "M20-9750242"
+			(at 36.83 95.25 0)
+			(effects
+				(font
+					(size 1.27 1.27)
+				)
+				(hide yes)
 			)
 		)
