File: pcb/HalfBridge_SiC/HalfBridge_GateDriver.kicad_sch (KiCad schematic)
At the start: 47 parts, among them SW1 CAS-D20X1, SW2 CAS-D20X1, U1 74AHC1G86, U2 74AHC1G86, U3 74AHC1G86, U4 RKD-052005D, U5 NCD57252, U6 RKD-052005D

Commit message: vgatereg + route + hsink
Parts:
- added C16, C17: 1 u, Capacitor_SMD:C_0805_2012Metric_Pad1.18x1.45mm_HandSolder, symbol Device:C
- added C18, C19: 100n, Capacitor_SMD:C_0603_1608Metric_Pad1.08x0.95mm_HandSolder, symbol Device:C
- added R11, R12: 0, Resistor_SMD:R_0805_2012Metric_Pad1.20x1.40mm_HandSolder, symbol Device:R
- added R13, R14, R15, R16, R17, R18: R, Resistor_SMD:R_0603_1608Metric_Pad0.98x0.95mm_HandSolder, symbol Device:R
- added SW1, SW2, SW3: SW_Nidec_CAS-120A1, Button_Switch_SMD:Nidec_Copal_CAS-120A, symbol Switch:SW_Nidec_CAS-120A1
- added TP1, TP2, TP3, TP4: TestPoint, TestPoint:TestPoint_Keystone_5015_Micro-Minature, symbol Connector:TestPoint
- added U7, U8: TL432DBZ, Package_TO_SOT_SMD:SOT-23, symbol Reference_Voltage:TL432DBZ
- renumbered C8 to C10, C9 to C11, C13 to C12, C10 to C13, C11 to C14, C12 to C15, C16 to C20, C17 to C21, C14 to C22, C15 to C23, C20 to C24, C21 to C25, C18 to C26, C19 to C27, C4 to C6, C5 to C7, C6 to C8, C7 to C9, R9 to R10, R11 to R19, R12 to R20, R13 to R21, R14 to R22, R15 to R23, R16 to R24, R17 to R25, R18 to R26, R10 to R9, SW1 to SW4, SW2 to SW5
Connections:
- net gnd: now also SW1.1 (C), SW2.1 (C), SW3.1 (C)
- net gonh: now also TP1.1
- net gonl: now also TP2.1
- net kh: now also C18.1, R11.2, R13.1, R14.2, TP3.1, U7.2 (K)
- net kl: now also C19.1, R12.2, R16.1, R17.2, TP4.1, U8.2 (K)
- net vcc: now also SW1.3 (A), SW2.3 (A), SW3.3 (A)
- net vddh: now also C16.1, R13.2
- net vddl: now also C17.1, R16.2
- net vssh: now also C16.2, C18.2, R15.1, U7.3 (A)
- net vssl: now also C17.2, C19.2, R18.1, U8.3 (A)
- net xorina: now reaches U1.2
- net xorina: now also SW1.2 (B)
- net lringa: now reaches D2.1 (K), R4.1
- net lringb: now reaches D3.1 (K), R5.1
- net lrdis: now reaches D4.1 (K), R6.1
- net vindc+: now reaches U6.1 (VIN+)
- net vindc+: now also U4.1 (VIN+)
- net vindc-: now reaches U6.2 (VIN-)
- net vindc-: now also U4.2 (VIN-)
- net coml: now reaches U6.6 (COM)
- net coml: now also R12.1
- net xorinen: now reaches U3.2
- net xorinen: now also SW3.2 (B)
- net comh: now reaches U4.6 (COM)
- net comh: now also R11.1
- net xorinb: now reaches U2.2
- net xorinb: now also SW2.2 (B)
- new net adjh: R14.1, R15.2, U7.1 (REF)
- new net adjl: R17.1, R18.2, U8.1 (REF)
Other:
- moved on the sheet: C10, C11, C12, C13, C14, C15, C20, C21, C22, C23, C24, C25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

Commit message: comment + gdriver + logo
Parts:
- removed U5: NCD57252, Package_SO:SOIC-16W_7.5x10.3mm_P1.27mm, symbol My_Driver_FET:NCD57252
- added C16, C17, C19, C25: 10 u, Capacitor_SMD:C_0805_2012Metric_Pad1.18x1.45mm_HandSolder, symbol Device:C
- added L2, L3: 4.7 u, Inductor_SMD:L_0603_1608Metric_Pad1.05x0.95mm_HandSolder, symbol Device:L
- added U5: NCV51563, Package_SO:SOIC-16W_7.5x10.3mm_P1.27mm, symbol My_Driver_FET:NCV51563
- C18: renamed from C16; value 1 u -> 10 u
- C20: renamed from C22; value C -> 100 n
- C21: renamed from C23; value C -> 100 n
- C24: renamed from C17; value 1 u -> 10 u
- C30: renamed from C26; value C -> 10 u
- C31: renamed from C27; value C -> 10 u
- renumbered C12 to C11, C11 to C12, C20 to C22, C21 to C23, C18 to C26, C19 to C27, C24 to C28, C25 to C29, R9 to R10, R10 to R7, R7 to R8, R8 to R9, SW5 to SW4, SW4 to SW5
Connections:
- net vindc- is gone; now on net gnd: U4.2 (VIN-), U6.2 (VIN-)
- net anb: now also U5.7 (ANB)
- net comh: now also C18.2, C19.1
- net coml: now also C24.2, C25.1
- net dis: now also U5.5 (DIS)
- net dt: now also U5.6 (DT)
- net gnd: now also C16.2, C17.2, U5.4 (GND)
- net gonh: now also U5.15 (OUTA)
- net gonl: now also U5.10 (OUTB)
- net inaf: now also U5.1 (INA)
- net inbf: now also U5.2 (INB)
- net vcc: now also C16.1, C17.1, L2.1, L3.1
- net vcci: now also U5.3 (VCCI), U5.8 (VCCI)
- net vddh: now also U5.16 (VDDA)
- net vddl: now also U5.11 (VDDB)
- net vssh: now also C19.2, U5.14 (VSSA); no longer C18.2
- net vssl: now also C25.2, U5.9 (VSSB); no longer C24.2
- net vindc+ renamed vindc+h
- net vindc+h: now also L2.2; no longer U6.1 (VIN+)
- new net vindc+l: L3.2, U6.1 (VIN+)
Other:
- title: (none) -> Dual Gate Diver
- moved on the sheet: C10, C11, C12, C13, C14, C15, C18, C20, C21, C22, C23, C24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

Commit message: 2DPDT switch footprint
Parts:
- C13: value C -> 1 u
- SW4, SW5: footprint My_Button_Switch_SMD:Nidec_Copal_CAS-D20A1 -> My_Button_Switch_SMD:Nidec_Copal_CAS-D20B1
Other:
- moved on the sheet: C12, C13, L1
Changed lines of the file:
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@@
 	(wire
 		(pts
-			(xy 139.7 62.23) (xy 142.24 62.23)
+			(xy 127 80.01) (xy 129.54 80.01)
 		)
 		(stroke
@@
 	(wire
 		(pts
-			(xy 127 62.23) (xy 132.08 62.23)
+			(xy 114.3 80.01) (xy 119.38 80.01)
 		)
 		(stroke
@@
 	)
 	(label "vcc"
-		(at 127 62.23 0)
+		(at 114.3 80.01 0)
 		(fields_autoplaced yes)
 		(effects
@@
 	)
 	(label "gnd"
-		(at 127 69.85 0)
+		(at 114.3 87.63 0)
 		(fields_autoplaced yes)
 		(effects
@@
 	)
 	(label "gnd"
-		(at 142.24 69.85 0)
+		(at 129.54 87.63 0)
 		(fields_autoplaced yes)
 		(effects
@@
 	)
 	(label "vcci"
-		(at 142.24 62.23 0)
+		(at 129.54 80.01 0)
 		(fields_autoplaced yes)
 		(effects
@@
 			)
 		)
-		(property "Footprint" "My_Button_Switch_SMD:Nidec_Copal_CAS-D20A1"
+		(property "Footprint" "My_Button_Switch_SMD:Nidec_Copal_CAS-D20B1"
 			(at 69.85 166.37 0)
 			(effects
@@
 	(symbol
 		(lib_id "Device:C")
-		(at 127 66.04 0)
+		(at 114.3 83.82 0)
 		(unit 1)
 		(exclude_from_sim no)
@@
 		(fields_autoplaced yes)
 		(property "Reference" "C12"
-			(at 130.81 64.7699 0)
+			(at 118.11 82.5499 0)
 			(effects
 				(font
@@
 		)
 		(property "Value" "C"
-			(at 130.81 67.3099 0)
+			(at 118.11 85.0899 0)
 			(effects
 				(font
@@
 		)
 		(property "Footprint" "Capacitor_SMD:C_0805_2012Metric_Pad1.18x1.45mm_HandSolder"
-			(at 127.9652 69.85 0)
+			(at 115.2652 87.63 0)
 			(effects
 				(font
@@
 		)
 		(property "Datasheet" "~"
-			(at 127 66.04 0)
+			(at 114.3 83.82 0)
 			(effects
 				(font
@@
 		)
 		(property "Description" "Unpolarized capacitor"
-			(at 127 66.04 0)
+			(at 114.3 83.82 0)
 			(effects
 				(font
@@
 	)
 	(symbol
-		(lib_name "My_Converter_DCDC:RKZ-052005D")
 		(lib_id "My_Converter_DCDC:RKZ-052005D")
 		(at 173.99 137.16 0)
@@
 	(symbol
 		(lib_id "Device:L")
-		(at 135.89 62.23 90)
+		(at 123.19 80.01 90)
 		(unit 1)
 		(exclude_from_sim no)
@@
 		(fields_autoplaced yes)
 		(property "Reference" "L1"
-			(at 135.89 57.15 90)
+			(at 123.19 74.93 90)
 			(effects
 				(font
@@
 		)
 		(property "Value" "L"
-			(at 135.89 59.69 90)
+			(at 123.19 77.47 90)
 			(effects
 				(font
@@
 		)
 		(property "Footprint" "Inductor_SMD:L_0603_1608Metric_Pad1.05x0.95mm_HandSolder"
-			(at 135.89 62.23 0)
+			(at 123.19 80.01 0)
 			(effects
 				(font
@@
 		)
 		(property "Datasheet" "~"
-			(at 135.89 62.23 0)
+			(at 123.19 80.01 0)
 			(effects
 				(font
@@
 		)
 		(property "Description" "Inductor"
-			(at 135.89 62.23 0)
+			(at 123.19 80.01 0)
 			(effects
 				(font
@@
 			)
 		)
-		(property "Footprint" "My_Button_Switch_SMD:Nidec_Copal_CAS-D20A1"
+		(property "Footprint" "My_Button_Switch_SMD:Nidec_Copal_CAS-D20B1"
 			(at 69.85 181.61 0)
 			(effects
@@
 			)
 		)
-		(property "Footprint" "My_Button_Switch_SMD:Nidec_Copal_CAS-D20A1"
+		(property "Footprint" "My_Button_Switch_SMD:Nidec_Copal_CAS-D20B1"
 			(at 125.73 190.5 0)
 			(effects
@@
 	)
 	(symbol
-		(lib_name "My_Converter_DCDC:RKZ-052005D")
 		(lib_id "My_Converter_DCDC:RKZ-052005D")
 		(at 172.72 38.1 0)
@@
 			)
 		)
-		(property "Footprint" "My_Button_Switch_SMD:Nidec_Copal_CAS-D20A1"
+		(property "Footprint" "My_Button_Switch_SMD:Nidec_Copal_CAS-D20B1"
 			(at 134.62 167.64 0)
 			(effects
@@
 	(symbol
 		(lib_id "Device:C")
-		(at 142.24 66.04 0)
+		(at 129.54 83.82 0)
 		(unit 1)
 		(exclude_from_sim no)
@@
 		(fields_autoplaced yes)
 		(property "Reference" "C13"
-			(at 146.05 64.7699 0)
+			(at 133.35 82.5499 0)
 			(effects
 				(font
@@
 			)
 		)
-		(property "Value" "C"
-			(at 146.05 67.3099 0)
+		(property "Value" "1 u"
+			(at 133.35 85.0899 0)
 			(effects
 				(font
@@
 		)
 		(property "Footprint" "Capacitor_SMD:C_0805_2012Metric_Pad1.18x1.45mm_HandSolder"
-			(at 143.2052 69.85 0)
+			(at 130.5052 87.63 0)
 			(effects
 				(font
@@
 		)
 		(property "Datasheet" "~"
-			(at 142.24 66.04 0)
+			(at 129.54 83.82 0)
 			(effects
 				(font
@@
 		)
 		(property "Description" "Unpolarized capacitor"
-			(at 142.24 66.04 0)
+			(at 129.54 83.82 0)
 			(effects
 				(font

Commit message: local lib
Parts:
- C10, C11, C12, C13, C14, C15, C16, C17, C18, C19, C20, C21, C22, C23, C24, C25, C26, C27, C28, C29, C30, C31, C6, C7, C8, C9: symbol Device:C -> HalfBridge_SiC:C
- D2, D3, D4: symbol Device:LED -> HalfBridge_SiC:LED
- D5, D6: symbol Device:D_Schottky -> HalfBridge_SiC:D_Schottky
- L1, L2, L3: symbol Device:L -> HalfBridge_SiC:L
- R10, R11, R12, R13, R14, R15, R16, R17, R18, R19, R20, R21, R22, R23, R24, R25, R26, R4, R5, R6, R7, R8, R9: symbol Device:R -> HalfBridge_SiC:R
- SW1, SW2, SW3: symbol Switch:SW_Nidec_CAS-120A1 -> HalfBridge_SiC:SW_Nidec_CAS-120A1
- SW4, SW5: symbol My_Switch:CAS-D20X1 -> HalfBridge_SiC:CAS-D20X1
- TP1, TP2, TP3, TP4: symbol Connector:TestPoint -> HalfBridge_SiC:TestPoint
- U1, U2, U3: symbol 74xGxx:74AHC1G86 -> HalfBridge_SiC:74AHC1G86
- U4: symbol My_Converter_DCDC:RKZ-052005D -> HalfBridge_SiC:RKZ-052005D_1
- U5: symbol My_Driver_FET:NCV51563 -> HalfBridge_SiC:NCV51563
- U6: symbol My_Converter_DCDC:RKZ-052005D -> HalfBridge_SiC:RKZ-052005D
- U7, U8: symbol Reference_Voltage:TL432DBZ -> HalfBridge_SiC:TL432DBZ
Other:
- moved on the sheet: D4, R6, R7, SW4A, SW4B
