File: pcb/HalfBridge_SiC/HalfBridge_GateDriver.kicad_sch (KiCad schematic)
At the start: 74 parts, among them SW1 SW_Nidec_CAS-120A1, SW2 SW_Nidec_CAS-120A1, SW3 SW_Nidec_CAS-120A1, SW4 CAS-D20X1, SW5 CAS-D20X1, U1 74AHC1G86, U2 74AHC1G86, U3 74AHC1G86, U4 RKD-052005D, U5 NCV51563, U6 RKD-052005D, U7 TL432DBZ, U8 TL432DBZ

Commit message: pcb + newlib
Other:
- company: (none) -> Dr.-Ing. Alan H. Wilson Veas
Changed lines of the file:
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@@
 		(date "2024-10-30")
 		(rev "1")
+		(company "Dr.-Ing. Alan H. Wilson Veas")
+		(comment 1 "AHWV")
 	)
 	(junction

Commit message: backplane + external lib
Parts:
- removed SW4, SW5: CAS-D20X1, My_Button_Switch_SMD:Nidec_Copal_CAS-D20B1, symbol HalfBridge_SiC:CAS-D20X1
- removed U5: NCV51563, Package_SO:SOIC-16W_7.5x10.3mm_P1.27mm, symbol HalfBridge_SiC:NCV51563
- added SW4, SW5: CAS-D20X1, symbol My_Switch:CAS-D20X1
- added TP21, TP22, TP23: TestPoint, symbol HalfBridge_SiC:TestPoint
- added U5: NCV51563, My_Package_SO:SOIC-16W_7.5x10.3mm_P1.27mm_NoPin_12_13, symbol My_Driver_FET:NCV51563
- C10, C11, C14, C15, C20, C21, C22, C23, C26, C27, C6, C7, C8, C9: footprint Capacitor_SMD:C_0603_1608Metric_Pad1.08x0.95mm_HandSolder -> (none)
- C12, C13, C16, C17, C18, C19, C24, C25, C28, C29, C30, C31: footprint Capacitor_SMD:C_0805_2012Metric_Pad1.18x1.45mm_HandSolder -> (none)
- D2, D3, D4: footprint LED_SMD:LED_0603_1608Metric_Pad1.05x0.95mm_HandSolder -> (none)
- D5, D6: footprint Diode_SMD:D_SOD-123 -> (none)
- L1, L2, L3: footprint Inductor_SMD:L_0603_1608Metric_Pad1.05x0.95mm_HandSolder -> (none)
- R10, R13, R14, R15, R16, R17, R18, R7, R8, R9: footprint Resistor_SMD:R_0603_1608Metric_Pad0.98x0.95mm_HandSolder -> (none)
- R11, R12, R19, R20, R21, R22, R23, R24, R25, R26: footprint Resistor_SMD:R_0805_2012Metric_Pad1.20x1.40mm_HandSolder -> (none)
- R4, R5, R6: footprint Resistor_SMD:R_0603_1608Metric -> (none)
- TP1, TP2, TP3, TP4: footprint TestPoint:TestPoint_Keystone_5015_Micro-Minature -> (none)
- U1, U2, U3: footprint Package_TO_SOT_SMD:SOT-23-5_HandSoldering -> (none)
Connections:
- net anb: now also SW4.5 (B), U5.7 (ANB)
- net dis: now also SW5.2 (B), U5.5 (DIS)
- net dis_i: now also SW5.1 (A), SW5.5 (B)
- net dis_x: now also SW5.3 (C)
- net dt: now also SW4.2 (B), U5.6 (DT)
- net gnd: now also SW4.4 (A), SW5.4 (A), TP23.1, U5.4 (GND)
- net gonh: now also U5.15 (OUTA)
- net gonl: now also U5.10 (OUTB)
- net inaf: now also U5.1 (INA)
- net inbf: now also U5.2 (INB)
- net inga: now also TP21.1
- net ingb: now also TP22.1
- net rdt: now also SW4.1 (A)
- net vcc: now also SW4.3 (C), SW4.6 (C), SW5.6 (C)
- net vcci: now also U5.3 (VCCI), U5.8 (VCCI)
- net vddh: now also U5.16 (VDDA)
- net vddl: now also U5.11 (VDDB)
- net vssh: now also U5.14 (VSSA)
- net vssl: now also U5.9 (VSSB)

Commit message: update lib
Parts:
- added C44, C45: 1n, Capacitor_SMD:C_0603_1608Metric_Pad1.08x0.95mm_HandSolder, symbol HalfBridge_SiC:C
- added D7: D, Diode_SMD:D_SMB-SMC_Universal_Handsoldering, symbol Device:D
- added R40: R, Resistor_SMD:R_0805_2012Metric_Pad1.20x1.40mm_HandSolder, symbol HalfBridge_SiC:R
- C10, C9: value C -> 33p; footprint (none) -> Capacitor_SMD:C_0603_1608Metric_Pad1.08x0.95mm_HandSolder
- C11: value C -> 100n; footprint (none) -> Capacitor_SMD:C_0603_1608Metric_Pad1.08x0.95mm_HandSolder
- C12, C28, C29: value C -> 10u; footprint (none) -> Capacitor_SMD:C_0805_2012Metric_Pad1.18x1.45mm_HandSolder
- C13: value 1 u -> 10u; footprint (none) -> Capacitor_SMD:C_0805_2012Metric_Pad1.18x1.45mm_HandSolder
- C14, C15, C22, C23, C26, C27, C6, C7, C8: footprint (none) -> Capacitor_SMD:C_0603_1608Metric_Pad1.08x0.95mm_HandSolder
- C16, C17, C18, C19, C24, C25, C30, C31: value 10 u -> 10u; footprint (none) -> Capacitor_SMD:C_0805_2012Metric_Pad1.18x1.45mm_HandSolder
- C20, C21: value 100 n -> 100n; footprint (none) -> Capacitor_SMD:C_0603_1608Metric_Pad1.08x0.95mm_HandSolder
- D2, D3, D4: footprint (none) -> LED_SMD:LED_0603_1608Metric_Pad1.05x0.95mm_HandSolder; Part # (none) -> 150060YS75020
- D5, D6: footprint (none) -> Diode_SMD:D_SOD-123
- L1: value L -> 4.7u; footprint (none) -> Inductor_SMD:L_0603_1608Metric_Pad1.05x0.95mm_HandSolder
- L2, L3: value 4.7 u -> 4.7u; footprint (none) -> Inductor_SMD:L_0603_1608Metric_Pad1.05x0.95mm_HandSolder
- R10, R11, R12, R19, R20, R21, R22, R23, R24, R25, R26: footprint (none) -> Resistor_SMD:R_0805_2012Metric_Pad1.20x1.40mm_HandSolder
- R13, R14, R15, R16, R17, R18, R7: footprint (none) -> Resistor_SMD:R_0603_1608Metric_Pad0.98x0.95mm_HandSolder
- R4, R5, R6: value R -> 330; footprint (none) -> Resistor_SMD:R_0603_1608Metric_Pad0.98x0.95mm_HandSolder
- R8, R9: value R -> 51; footprint (none) -> Resistor_SMD:R_0603_1608Metric_Pad0.98x0.95mm_HandSolder
- SW4, SW5: footprint (none) -> My_Button_Switch_SMD:SW_SPDTx02_Slide_Copal_CAS-D20B1_W5.6mm_P1.7mm_GullW
- TP1, TP2, TP21, TP22, TP23, TP3, TP4: footprint (none) -> TestPoint:TestPoint_Keystone_5015_Micro-Minature
- U1, U2, U3: footprint (none) -> Package_TO_SOT_SMD:SOT-23-5_HandSoldering
Connections:
- net gh: now also C44.1
- net gl: now also C45.1
- net kh: now also C44.2
- net kl: now also C45.2
- net vddh: now also D7.1 (K)
- net vddl: now also R40.2
- new net bootR: D7.2 (A), R40.1
Other:
- moved on the sheet: C20, C21, C22, C23, C28, C29, C30, C31, D3, D5, D6, R19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

Commit message: filter + sim + assembly3d
Parts:
- removed SW1, SW2, SW3: SW_Nidec_CAS-120A1, Button_Switch_SMD:Nidec_Copal_CAS-120A, symbol HalfBridge_SiC:SW_Nidec_CAS-120A1
- added SW1, SW2, SW3: CAS-120X1, My_Button_Switch_SMD:Nidec_Copal_CAS-120B1, symbol My_Switch:CAS-120X1
Connections:
- net gnd: now also SW1.1 (A), SW2.1 (A), SW3.1 (A)
- net vcc: now also SW1.3 (C), SW2.3 (C), SW3.3 (C)
- net xorina: now also SW1.2 (B)
- net xorinb: now also SW2.2 (B)
- net xorinen: now also SW3.2 (B)
Changed lines of the file:
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@@
+	)
+	(symbol
+		(lib_id "My_Switch:CAS-120X1")
+		(at 34.29 142.24 180)
+		(unit 1)
+		(exclude_from_sim no)
+		(in_bom yes)
+		(on_board yes)
+		(dnp no)
+		(fields_autoplaced yes)
+		(property "Reference" "SW2"
+			(at 34.29 133.35 0)
+			(effects
+				(font
+					(size 1.27 1.27)
+				)
+			)
+		)
+		(property "Value" "CAS-120X1"
+			(at 34.29 135.89 0)
+			(effects
+				(font
+					(size 1.27 1.27)
+				)
+			)
+		)
+		(property "Footprint" "My_Button_Switch_SMD:Nidec_Copal_CAS-120B1"
+			(at 34.29 142.24 0)
+			(effects
+				(font
+					(size 1.27 1.27)
+				)
+				(hide yes)
+			)
+		)
+		(property "Datasheet" "https://www.nidec-components.com/e/catalog/switch/cas.pdf"
+			(at 34.29 142.24 0)
+			(effects
+				(font
+					(size 1.27 1.27)
+				)
+				(hide yes)
+			)
+		)
+		(property "Description" "Slide Switches SPDT, slide, SMD terminals, 100mA @ 6V DC, bulk packaging, non-washable without seal tape"
+			(at 34.29 142.24 0)
+			(effects
+				(font
+					(size 1.27 1.27)
+				)
+				(hide yes)
+			)
+		)
+		(pin "2"
+		)
+		(pin "3"
+		)
+		(pin "1"
+		)
+		(instances
+			(project "HalfBridge_SiC"
+				(path "/3c187ffa-7f66-4861-b077-b6965c821fc2/8af60660-0838-42a2-a499-fc014bb54766"
+					(reference "SW2")
+					(unit 1)
+				)
+			)
+		)
 	)
 	(symbol
@@
 	)
 	(symbol
+		(lib_id "My_Switch:CAS-120X1")
+		(at 34.29 172.72 180)
+		(unit 1)
+		(exclude_from_sim no)
+		(in_bom yes)
+		(on_board yes)
+		(dnp no)
+		(fields_autoplaced yes)
+		(property "Reference" "SW3"
+			(at 34.29 163.83 0)
+			(effects
+				(font
+					(size 1.27 1.27)
+				)
+			)
+		)
+		(property "Value" "CAS-120X1"
+			(at 34.29 166.37 0)
+			(effects
+				(font
+					(size 1.27 1.27)
+				)
+			)
+		)
+		(property "Footprint" "My_Button_Switch_SMD:Nidec_Copal_CAS-120B1"
+			(at 34.29 172.72 0)
+			(effects
+				(font
+					(size 1.27 1.27)
+				)
+				(hide yes)
+			)
+		)
+		(property "Datasheet" "https://www.nidec-components.com/e/catalog/switch/cas.pdf"
+			(at 34.29 172.72 0)
+			(effects
+				(font
+					(size 1.27 1.27)
+				)
+				(hide yes)
+			)
+		)
+		(property "Description" "Slide Switches SPDT, slide, SMD terminals, 100mA @ 6V DC, bulk packaging, non-washable without seal tape"
+			(at 34.29 172.72 0)
+			(effects
+				(font
+					(size 1.27 1.27)
+				)
+				(hide yes)
+			)
+		)
+		(pin "2"
+		)
+		(pin "3"
+		)
+		(pin "1"
+		)
+		(instances
+			(project "HalfBridge_SiC"
+				(path "/3c187ffa-7f66-4861-b077-b6965c821fc2/8af60660-0838-42a2-a499-fc014bb54766"
+					(reference "SW3")
+					(unit 1)
+				)
+			)
+		)
+	)
+	(symbol
 		(lib_id "HalfBridge_SiC:RKZ-052005D")
 		(at 173.99 137.16 0)
@@
 				(path "/3c187ffa-7f66-4861-b077-b6965c821fc2/8af60660-0838-42a2-a499-fc014bb54766"
 					(reference "C15")
-					(unit 1)
-				)
-			)
-		)
-	)
-	(symbol
-		(lib_id "HalfBridge_SiC:SW_Nidec_CAS-120A1")
-		(at 34.29 111.76 0)
-		(mirror y)
-		(unit 1)
-		(exclude_from_sim no)
-		(in_bom yes)
-		(on_board yes)
-		(dnp no)
-		(property "Reference" "SW1"
-			(at 34.29 102.87 0)
-			(effects
-				(font
-					(size 1.27 1.27)
-				)
-			)
-		)
-		(property "Value" "SW_Nidec_CAS-120A1"
-			(at 34.29 105.41 0)
-			(effects
-				(font
-					(size 1.27 1.27)
-				)
-			)
-		)
-		(property "Footprint" "Button_Switch_SMD:Nidec_Copal_CAS-120A"
-			(at 34.29 121.92 0)
-			(effects
-				(font
-					(size 1.27 1.27)
-				)
-				(hide yes)
-			)
-		)
-		(property "Datasheet" "https://www.nidec-components.com/e/catalog/switch/cas.pdf"
-			(at 34.29 119.38 0)
-			(effects
-				(font
-					(size 1.27 1.27)
-				)
-				(hide yes)
-			)
-		)
-		(property "Description" "Switch, single pole double throw"
-			(at 34.29 111.76 0)
-			(effects
-				(font
-					(size 1.27 1.27)
-				)
-				(hide yes)
-			)
-		)
-		(pin "3"
-		)
-		(pin "1"
-		)
-		(pin "2"
-		)
-		(instances
-			(project ""
-				(path "/3c187ffa-7f66-4861-b077-b6965c821fc2/8af60660-0838-42a2-a499-fc014bb54766"
-					(reference "SW1")
 					(unit 1)
 				)
@@
 	)
 	(symbol
-		(lib_id "HalfBridge_SiC:SW_Nidec_CAS-120A1")
-		(at 34.29 172.72 0)
-		(mirror y)
-		(unit 1)
-		(exclude_from_sim no)
-		(in_bom yes)
-		(on_board yes)
-		(dnp no)
-		(property "Reference" "SW3"
-			(at 34.29 163.83 0)
-			(effects
-				(font
-					(size 1.27 1.27)
-				)
-			)
-		)
-		(property "Value" "SW_Nidec_CAS-120A1"
-			(at 34.29 166.37 0)
-			(effects
-				(font
-					(size 1.27 1.27)
-				)
-			)
-		)
-		(property "Footprint" "Button_Switch_SMD:Nidec_Copal_CAS-120A"
-			(at 34.29 182.88 0)
-			(effects
-				(font
-					(size 1.27 1.27)
-				)
-				(hide yes)
-			)
-		)
-		(property "Datasheet" "https://www.nidec-components.com/e/catalog/switch/cas.pdf"
-			(at 34.29 180.34 0)
-			(effects
-				(font
-					(size 1.27 1.27)
-				)
-				(hide yes)
-			)
-		)
-		(property "Description" "Switch, single pole double throw"
-			(at 34.29 172.72 0)
-			(effects
-				(font
-					(size 1.27 1.27)
-				)
-				(hide yes)
-			)
-		)
-		(pin "3"
-		)
-		(pin "1"
-		)
-		(pin "2"
-		)
-		(instances
-			(project "HalfBridge_SiC"
-				(path "/3c187ffa-7f66-4861-b077-b6965c821fc2/8af60660-0838-42a2-a499-fc014bb54766"
-					(reference "SW3")
-					(unit 1)
-				)
-			)
-		)
-	)
-	(symbol
 		(lib_id "HalfBridge_SiC:LED")
 		(at 74.93 101.6 90)
@@
 	)
 	(symbol
+		(lib_id "My_Switch:CAS-120X1")
+		(at 34.29 111.76 180)
+		(unit 1)
+		(exclude_from_sim no)
+		(in_bom yes)
+		(on_board yes)
+		(dnp no)
+		(fields_autoplaced yes)
+		(property "Reference" "SW1"
+			(at 34.29 102.87 0)
+			(effects
+				(font
+					(size 1.27 1.27)
+				)
+			)
+		)
+		(property "Value" "CAS-120X1"
+			(at 34.29 105.41 0)
+			(effects
+				(font
+					(size 1.27 1.27)
+				)
+			)
+		)
+		(property "Footprint" "My_Button_Switch_SMD:Nidec_Copal_CAS-120B1"
+			(at 34.29 111.76 0)
+			(effects
+				(font
+					(size 1.27 1.27)
+				)
+				(hide yes)
+			)
+		)
+		(property "Datasheet" "https://www.nidec-components.com/e/catalog/switch/cas.pdf"
+			(at 34.29 111.76 0)
+			(effects
+				(font
+					(size 1.27 1.27)
+				)
+				(hide yes)
+			)
+		)
+		(property "Description" "Slide Switches SPDT, slide, SMD terminals, 100mA @ 6V DC, bulk packaging, non-washable without seal tape"
+			(at 34.29 111.76 0)
+			(effects
+				(font
+					(size 1.27 1.27)
+				)
+				(hide yes)
+			)
+		)
+		(pin "2"
+		)
+		(pin "3"
+		)
+		(pin "1"
+		)
+		(instances
+			(project ""
+				(path "/3c187ffa-7f66-4861-b077-b6965c821fc2/8af60660-0838-42a2-a499-fc014bb54766"
+					(reference "SW1")
+					(unit 1)
+				)
+			)
+		)
+	)
+	(symbol
 		(lib_id "HalfBridge_SiC:C")
 		(at 142.24 83.82 0)
@@
 					(unit 1)
 				)
-			)
-		)
-	)
-	(symbol
-		(lib_id "HalfBridge_SiC:SW_Nidec_CAS-120A1")
-		(at 34.29 142.24 0)
-		(mirror y)
-		(unit 1)
-		(exclude_from_sim no)
-		(in_bom yes)
-		(on_board yes)
-		(dnp no)
-		(property "Reference" "SW2"
-			(at 34.29 133.35 0)
-			(effects
-				(font
-					(size 1.27 1.27)
-				)
-			)
-		)
-		(property "Value" "SW_Nidec_CAS-120A1"
-			(at 34.29 135.89 0)
-			(effects
-				(font
-					(size 1.27 1.27)
-				)
-			)
-		)
-		(property "Footprint" "Button_Switch_SMD:Nidec_Copal_CAS-120A"
-			(at 34.29 152.4 0)
-			(effects
-				(font
-					(size 1.27 1.27)
-				)
-				(hide yes)
-			)
-		)
-		(property "Datasheet" "https://www.nidec-components.com/e/catalog/switch/cas.pdf"
-			(at 34.29 149.86 0)
-			(effects
-				(font
-					(size 1.27 1.27)
-				)
-				(hide yes)
-			)
-		)
-		(property "Description" "Switch, single pole double throw"
-			(at 34.29 142.24 0)
-			(effects
-				(font
-					(size 1.27 1.27)
-				)
-				(hide yes)
-			)
-		)
-		(pin "3"
-		)
-		(pin "1"
-		)
-		(pin "2"
-		)
-		(instances
-			(project "HalfBridge_SiC"
-				(path "/3c187ffa-7f66-4861-b077-b6965c821fc2/8af60660-0838-42a2-a499-fc014bb54766"
-					(reference "SW2")
-					(unit 1)
-				)

Commit message: designator + part n°
Parts:
- R11: renamed from R7; value R -> 10k
- R12: renamed from R10; value R -> 10k
- R16: renamed from R13; value R -> 14 k
- R17: renamed from R14; value R -> 30 k
- R18: renamed from R15; value R -> 14 k
- R19: renamed from R16; value R -> 14k
- R20: renamed from R17; value R -> 30k
- R21: renamed from R18; value R -> 14k
- R22: renamed from R19; value R -> 10
- R23: renamed from R20; value R -> 10
- R24: renamed from R21; value R -> 10
- R25: renamed from R22; value R -> 10
- R26: renamed from R23; value R -> 10
- R27: renamed from R24; value R -> 10
- R28: renamed from R25; value R -> 10
- R29: renamed from R26; value R -> 10
- U1, U2, U3: Part # (none) -> SN74LVC1G86DBVR
- renumbered C12 to C11, C11 to C12, C22 to C20, C23 to C21, C20 to C22, C21 to C23, C44 to C32, C45 to C33, D7 to D5, D5 to D6, D6 to D7, R6 to R10, R40 to R13, R11 to R14, R12 to R15, R4 to R6, R5 to R7, SW5 to SW4, SW4 to SW5, TP21 to TP1, TP22 to TP2, TP23 to TP3, TP1 to TP4, TP2 to TP5, TP3 to TP6, TP4 to TP7

Commit message: titles
Parts:
- C10, C9: Part # (none) -> 06035A330F4T2A
- C11, C13, C16, C17, C18, C19, C24, C25, C28, C29, C30, C31: Part # (none) -> GRM21BR61H106KE43L
- C12, C14, C15, C20, C21, C22, C23, C26, C27, C6, C7, C8: Part # (none) -> UMK107BJ104KAHT
- D6, D7: Part # (none) -> PMEG60T30ELR
- SW1, SW2, SW3: Part # (none) -> CAS-120B1
- SW4, SW5: Part # (none) -> CAS-D20B1
- TP1, TP2, TP3, TP4, TP5, TP6, TP7: Part # (none) -> 5015
- U4, U6: Part # (none) -> RKD-052005D
- U7, U8: Part # (none) -> TL432ASA-7
