File: pcb/HalfBridge_SiC/HalfBridge_Optical.kicad_sch (KiCad schematic)
At the start: 18 parts, among them J3 AFBR-2624Z, J4 AFBR-2624Z, J5 AFBR-2624Z

Commit message: pcb + horizontal of
Parts:
- J3, J4, J5: footprint OptoDevice:Broadcom_AFBR-16xxZ_Vertical -> OptoDevice:Broadcom_AFBR-16xxZ_Horizontal
Changed lines of the file:
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@@
 			)
 		)
-		(property "Footprint" "OptoDevice:Broadcom_AFBR-16xxZ_Vertical"
+		(property "Footprint" "OptoDevice:Broadcom_AFBR-16xxZ_Horizontal"
 			(at 55.88 121.92 0)
 			(effects
@@
 			)
 		)
-		(property "Footprint" "OptoDevice:Broadcom_AFBR-16xxZ_Vertical"
+		(property "Footprint" "OptoDevice:Broadcom_AFBR-16xxZ_Horizontal"
 			(at 55.88 160.02 0)
 			(effects
@@
 			)
 		)
-		(property "Footprint" "OptoDevice:Broadcom_AFBR-16xxZ_Vertical"
+		(property "Footprint" "OptoDevice:Broadcom_AFBR-16xxZ_Horizontal"
 			(at 55.88 86.36 0)
 			(effects

Commit message: vgatereg + route + hsink
Parts:
- renumbered C22 to C28, C23 to C29, C24 to C30, C25 to C31, C26 to C32, C27 to C33, C28 to C34, C29 to C35, C30 to C36, R19 to R27, R20 to R28, R21 to R29
Changed lines of the file:
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@@
 		(dnp no)
 		(fields_autoplaced yes)
-		(property "Reference" "C26"
+		(property "Reference" "C32"
 			(at 90.17 95.2499 0)
 			(effects
@@
 			(project "HalfBridge_SiC"
 				(path "/3c187ffa-7f66-4861-b077-b6965c821fc2/6b9f2a3a-4d36-43fe-adee-f56a635b1692"
-					(reference "C26")
+					(reference "C32")
 					(unit 1)
 				)
@@
 		(dnp no)
 		(fields_autoplaced yes)
-		(property "Reference" "C28"
+		(property "Reference" "C34"
 			(at 105.41 55.8799 0)
 			(effects
@@
 			(project "HalfBridge_SiC"
 				(path "/3c187ffa-7f66-4861-b077-b6965c821fc2/6b9f2a3a-4d36-43fe-adee-f56a635b1692"
-					(reference "C28")
+					(reference "C34")
 					(unit 1)
 				)
@@
 		(dnp no)
 		(fields_autoplaced yes)
-		(property "Reference" "C30"
+		(property "Reference" "C36"
 			(at 105.41 133.3499 0)
 			(effects
@@
 			(project "HalfBridge_SiC"
 				(path "/3c187ffa-7f66-4861-b077-b6965c821fc2/6b9f2a3a-4d36-43fe-adee-f56a635b1692"
-					(reference "C30")
+					(reference "C36")
 					(unit 1)
 				)
@@
 		(dnp no)
 		(fields_autoplaced yes)
-		(property "Reference" "C25"
+		(property "Reference" "C31"
 			(at 90.17 55.8799 0)
 			(effects
@@
 			(project "HalfBridge_SiC"
 				(path "/3c187ffa-7f66-4861-b077-b6965c821fc2/6b9f2a3a-4d36-43fe-adee-f56a635b1692"
-					(reference "C25")
+					(reference "C31")
 					(unit 1)
 				)
@@
 		(on_board yes)
 		(dnp no)
-		(property "Reference" "R19"
+		(property "Reference" "R27"
 			(at 77.47 67.31 90)
 			(effects
@@
 			(project "HalfBridge_SiC"
 				(path "/3c187ffa-7f66-4861-b077-b6965c821fc2/6b9f2a3a-4d36-43fe-adee-f56a635b1692"
-					(reference "R19")
+					(reference "R27")
 					(unit 1)
 				)
@@
 		(on_board yes)
 		(dnp no)
-		(property "Reference" "R20"
+		(property "Reference" "R28"
 			(at 77.47 102.87 90)
 			(effects
@@
 			(project ""
 				(path "/3c187ffa-7f66-4861-b077-b6965c821fc2/6b9f2a3a-4d36-43fe-adee-f56a635b1692"
-					(reference "R20")
+					(reference "R28")
 					(unit 1)
 				)
@@
 		(on_board yes)
 		(dnp no)
-		(property "Reference" "R21"
+		(property "Reference" "R29"
 			(at 77.47 140.97 90)
 			(effects
@@
 			(project "HalfBridge_SiC"
 				(path "/3c187ffa-7f66-4861-b077-b6965c821fc2/6b9f2a3a-4d36-43fe-adee-f56a635b1692"
-					(reference "R21")
+					(reference "R29")
 					(unit 1)
 				)
@@
 		(dnp no)
 		(fields_autoplaced yes)
-		(property "Reference" "C24"
+		(property "Reference" "C30"
 			(at 80.01 133.3499 0)
 			(effects
@@
 			(project "HalfBridge_SiC"
 				(path "/3c187ffa-7f66-4861-b077-b6965c821fc2/6b9f2a3a-4d36-43fe-adee-f56a635b1692"
-					(reference "C24")
+					(reference "C30")
 					(unit 1)
 				)
@@
 		(dnp no)
 		(fields_autoplaced yes)
-		(property "Reference" "C22"
+		(property "Reference" "C28"
 			(at 80.01 55.8799 0)
 			(effects
@@
 			(project "HalfBridge_SiC"
 				(path "/3c187ffa-7f66-4861-b077-b6965c821fc2/6b9f2a3a-4d36-43fe-adee-f56a635b1692"
-					(reference "C22")
+					(reference "C28")
 					(unit 1)
 				)
@@
 		(dnp no)
 		(fields_autoplaced yes)
-		(property "Reference" "C29"
+		(property "Reference" "C35"
 			(at 105.41 95.2499 0)
 			(effects
@@
 			(project "HalfBridge_SiC"
 				(path "/3c187ffa-7f66-4861-b077-b6965c821fc2/6b9f2a3a-4d36-43fe-adee-f56a635b1692"
-					(reference "C29")
+					(reference "C35")
 					(unit 1)
 				)
@@
 		(dnp no)
 		(fields_autoplaced yes)
-		(property "Reference" "C27"
+		(property "Reference" "C33"
 			(at 90.17 133.3499 0)
 			(effects
@@
 			(project "HalfBridge_SiC"
 				(path "/3c187ffa-7f66-4861-b077-b6965c821fc2/6b9f2a3a-4d36-43fe-adee-f56a635b1692"
-					(reference "C27")
+					(reference "C33")
 					(unit 1)
 				)
@@
 		(dnp no)
 		(fields_autoplaced yes)
-		(property "Reference" "C23"
+		(property "Reference" "C29"
 			(at 80.01 95.2499 0)
 			(effects
@@
 			(project "HalfBridge_SiC"
 				(path "/3c187ffa-7f66-4861-b077-b6965c821fc2/6b9f2a3a-4d36-43fe-adee-f56a635b1692"
-					(reference "C23")
-					(unit 1)
-				)
+					(reference "C29")
+					(unit 1)
+				)

Commit message: comment + gdriver + logo
Parts:
- R27, R28, R29: value R -> 0
- renumbered C28 to C32, C29 to C33, C30 to C34, C31 to C35, C32 to C36, C33 to C37, C34 to C38, C35 to C39, C36 to C40, L2 to L4, L3 to L5, L4 to L6
Other:
- title: (none) -> Optical receptors x3
Changed lines of the file:
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@@
 	(generator_version "8.0")
 	(paper "A4")
+	(title_block
+		(title "Optical receptors x3")
+		(rev "1")
+	)
 	(junction
 		(at 76.2 130.81)
@@
 	(wire
 		(pts
-			(xy 81.28 73.66) (xy 123.19 73.66)
+			(xy 81.28 73.66) (xy 125.73 73.66)
 		)
 		(stroke
@@
 			(width 0)
 			(type default)
+		)
+	)
+	(text_box "Jump R=0 when Optical Rx is used.\n\nOtherwise, DNP whole module (at least R jumper)"
+		(exclude_from_sim no)
+		(at 74.93 152.4 0)
+		(size 53.34 7.62)
+		(stroke
+			(width 0)
+			(type default)
+		)
+		(fill
+			(type none)
+		)
+		(effects
+			(font
+				(size 1.27 1.27)
+			)
+			(justify left top)
 		)
 	)
@@
 	(hierarchical_label "inb"
 		(shape output)
-		(at 123.19 73.66 0)
+		(at 125.73 73.66 0)
 		(fields_autoplaced yes)
 		(effects
@@
 		(dnp no)
 		(fields_autoplaced yes)
-		(property "Reference" "C32"
+		(property "Reference" "C36"
 			(at 90.17 95.2499 0)
 			(effects
@@
 			(project "HalfBridge_SiC"
 				(path "/3c187ffa-7f66-4861-b077-b6965c821fc2/6b9f2a3a-4d36-43fe-adee-f56a635b1692"
-					(reference "C32")
+					(reference "C36")
 					(unit 1)
 				)
@@
 		(dnp no)
 		(fields_autoplaced yes)
-		(property "Reference" "L2"
+		(property "Reference" "L4"
 			(at 95.25 48.26 90)
 			(effects
@@
 			(project ""
 				(path "/3c187ffa-7f66-4861-b077-b6965c821fc2/6b9f2a3a-4d36-43fe-adee-f56a635b1692"
-					(reference "L2")
+					(reference "L4")
 					(unit 1)
 				)
@@
 		(dnp no)
 		(fields_autoplaced yes)
-		(property "Reference" "C34"
+		(property "Reference" "C38"
 			(at 105.41 55.8799 0)
 			(effects
@@
 			(project "HalfBridge_SiC"
 				(path "/3c187ffa-7f66-4861-b077-b6965c821fc2/6b9f2a3a-4d36-43fe-adee-f56a635b1692"
-					(reference "C34")
+					(reference "C38")
 					(unit 1)
 				)
@@
 		(dnp no)
 		(fields_autoplaced yes)
-		(property "Reference" "C36"
+		(property "Reference" "C40"
 			(at 105.41 133.3499 0)
 			(effects
@@
 			(project "HalfBridge_SiC"
 				(path "/3c187ffa-7f66-4861-b077-b6965c821fc2/6b9f2a3a-4d36-43fe-adee-f56a635b1692"
-					(reference "C36")
+					(reference "C40")
 					(unit 1)
 				)
@@
 		(dnp no)
 		(fields_autoplaced yes)
-		(property "Reference" "C31"
+		(property "Reference" "C35"
 			(at 90.17 55.8799 0)
 			(effects
@@
 			(project "HalfBridge_SiC"
 				(path "/3c187ffa-7f66-4861-b077-b6965c821fc2/6b9f2a3a-4d36-43fe-adee-f56a635b1692"
-					(reference "C31")
+					(reference "C35")
 					(unit 1)
 				)
@@
 			)
 		)
-		(property "Value" "R"
+		(property "Value" "0"
 			(at 77.47 69.85 90)
 			(effects
@@
 			)
 		)
-		(property "Value" "R"
+		(property "Value" "0"
 			(at 77.47 105.41 90)
 			(effects
@@
 			)
 		)
-		(property "Value" "R"
+		(property "Value" "0"
 			(at 77.47 143.51 90)
 			(effects
@@
 		(dnp no)
 		(fields_autoplaced yes)
-		(property "Reference" "C30"
+		(property "Reference" "C34"
 			(at 80.01 133.3499 0)
 			(effects
@@
 			(project "HalfBridge_SiC"
 				(path "/3c187ffa-7f66-4861-b077-b6965c821fc2/6b9f2a3a-4d36-43fe-adee-f56a635b1692"
-					(reference "C30")
+					(reference "C34")
 					(unit 1)
 				)
@@
 		(dnp no)
 		(fields_autoplaced yes)
-		(property "Reference" "C28"
+		(property "Reference" "C32"
 			(at 80.01 55.8799 0)
 			(effects
@@
 			(project "HalfBridge_SiC"
 				(path "/3c187ffa-7f66-4861-b077-b6965c821fc2/6b9f2a3a-4d36-43fe-adee-f56a635b1692"
-					(reference "C28")
+					(reference "C32")
 					(unit 1)
 				)
@@
 		(dnp no)
 		(fields_autoplaced yes)
-		(property "Reference" "C35"
+		(property "Reference" "C39"
 			(at 105.41 95.2499 0)
 			(effects
@@
 			(project "HalfBridge_SiC"
 				(path "/3c187ffa-7f66-4861-b077-b6965c821fc2/6b9f2a3a-4d36-43fe-adee-f56a635b1692"
-					(reference "C35")
+					(reference "C39")
 					(unit 1)
 				)
@@
 		(dnp no)
 		(fields_autoplaced yes)
-		(property "Reference" "C33"
+		(property "Reference" "C37"
 			(at 90.17 133.3499 0)
 			(effects
@@
 			(project "HalfBridge_SiC"
 				(path "/3c187ffa-7f66-4861-b077-b6965c821fc2/6b9f2a3a-4d36-43fe-adee-f56a635b1692"
-					(reference "C33")
+					(reference "C37")
 					(unit 1)
 				)
@@
 		(dnp no)
 		(fields_autoplaced yes)
-		(property "Reference" "L3"
+		(property "Reference" "L5"
 			(at 95.25 87.63 90)
 			(effects
@@
 			(project "HalfBridge_SiC"
 				(path "/3c187ffa-7f66-4861-b077-b6965c821fc2/6b9f2a3a-4d36-43fe-adee-f56a635b1692"
-					(reference "L3")
+					(reference "L5")
 					(unit 1)
 				)
@@
 		(dnp no)
 		(fields_autoplaced yes)
-		(property "Reference" "L4"
+		(property "Reference" "L6"
 			(at 95.25 125.73 90)
 			(effects
@@
 			(project "HalfBridge_SiC"
 				(path "/3c187ffa-7f66-4861-b077-b6965c821fc2/6b9f2a3a-4d36-43fe-adee-f56a635b1692"
-					(reference "L4")
+					(reference "L6")
 					(unit 1)
 				)
@@
 		(dnp no)
 		(fields_autoplaced yes)
-		(property "Reference" "C29"
+		(property "Reference" "C33"
 			(at 80.01 95.2499 0)
 			(effects
@@
 			(project "HalfBridge_SiC"
 				(path "/3c187ffa-7f66-4861-b077-b6965c821fc2/6b9f2a3a-4d36-43fe-adee-f56a635b1692"
-					(reference "C29")
+					(reference "C33")
 					(unit 1)
 				)

Commit message: local lib
Parts:
- C32, C33, C34, C35, C36, C37, C38, C39, C40: symbol Device:C -> HalfBridge_SiC:C
- J3, J4, J5: symbol Fiber_Optic:AFBR-2624Z -> HalfBridge_SiC:AFBR-2624Z
- L4, L5, L6: symbol Device:L -> HalfBridge_SiC:L
- R27, R28, R29: symbol Device:R -> HalfBridge_SiC:R
Changed lines of the file:
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@@
 	)
 	(symbol
-		(lib_id "Device:C")
+		(lib_id "HalfBridge_SiC:C")
 		(at 86.36 96.52 0)
 		(unit 1)
@@
 	)
 	(symbol
-		(lib_id "Device:L")
+		(lib_id "HalfBridge_SiC:L")
 		(at 95.25 53.34 90)
 		(unit 1)
@@
 	)
 	(symbol
-		(lib_id "Device:C")
+		(lib_id "HalfBridge_SiC:C")
 		(at 101.6 57.15 0)
 		(unit 1)
@@
 	)
 	(symbol
-		(lib_id "Device:C")
+		(lib_id "HalfBridge_SiC:C")
 		(at 101.6 134.62 0)
 		(unit 1)
@@
 	)
 	(symbol
-		(lib_id "Device:C")
+		(lib_id "HalfBridge_SiC:C")
 		(at 86.36 57.15 0)
 		(unit 1)
@@
 	)
 	(symbol
-		(lib_id "Device:R")
+		(lib_id "HalfBridge_SiC:R")
 		(at 77.47 73.66 270)
 		(unit 1)
@@
 	)
 	(symbol
-		(lib_id "Device:R")
+		(lib_id "HalfBridge_SiC:R")
 		(at 77.47 109.22 270)
 		(unit 1)
@@
 	)
 	(symbol
-		(lib_id "Device:R")
+		(lib_id "HalfBridge_SiC:R")
 		(at 77.47 147.32 270)
 		(unit 1)
@@
 	)
 	(symbol
-		(lib_id "Device:C")
+		(lib_id "HalfBridge_SiC:C")
 		(at 76.2 134.62 0)
 		(unit 1)
@@
 	)
 	(symbol
-		(lib_id "Device:C")
+		(lib_id "HalfBridge_SiC:C")
 		(at 76.2 57.15 0)
 		(unit 1)
@@
 	)
 	(symbol
-		(lib_id "Device:C")
+		(lib_id "HalfBridge_SiC:C")
 		(at 101.6 96.52 0)
 		(unit 1)
@@
 	)
 	(symbol
-		(lib_id "Device:C")
+		(lib_id "HalfBridge_SiC:C")
 		(at 86.36 134.62 0)
 		(unit 1)
@@
 	)
 	(symbol
-		(lib_id "Fiber_Optic:AFBR-2624Z")
+		(lib_id "HalfBridge_SiC:AFBR-2624Z")
 		(at 58.42 109.22 0)
 		(unit 1)
@@
 	)
 	(symbol
-		(lib_id "Fiber_Optic:AFBR-2624Z")
+		(lib_id "HalfBridge_SiC:AFBR-2624Z")
 		(at 58.42 147.32 0)
 		(unit 1)
@@
 	)
 	(symbol
-		(lib_id "Device:L")
+		(lib_id "HalfBridge_SiC:L")
 		(at 95.25 92.71 90)
 		(unit 1)
@@
 	)
 	(symbol
-		(lib_id "Device:L")
+		(lib_id "HalfBridge_SiC:L")
 		(at 95.25 130.81 90)
 		(unit 1)
@@
 	)
 	(symbol
-		(lib_id "Device:C")
+		(lib_id "HalfBridge_SiC:C")
 		(at 76.2 96.52 0)
 		(unit 1)
@@
 	)
 	(symbol
-		(lib_id "Fiber_Optic:AFBR-2624Z")
+		(lib_id "HalfBridge_SiC:AFBR-2624Z")
 		(at 58.42 73.66 0)
 		(unit 1)

Commit message: pcb + newlib
Other:
- company: (none) -> Dr.-Ing. Alan H. Wilson Veas
Changed lines of the file:
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@@
 		(title "Optical receptors x3")
 		(rev "1")
+		(company "Dr.-Ing. Alan H. Wilson Veas")
+		(comment 1 "AHWV")
 	)
 	(junction

Commit message: backplane + external lib
Parts:
- C32, C33, C34: footprint Capacitor_SMD:C_0603_1608Metric_Pad1.08x0.95mm_HandSolder -> (none)
- C35, C36, C37, C38, C39, C40: footprint Capacitor_SMD:C_0805_2012Metric_Pad1.18x1.45mm_HandSolder -> (none)
- J3, J4, J5: footprint OptoDevice:Broadcom_AFBR-16xxZ_Horizontal -> (none)
- L4, L5, L6: footprint Inductor_SMD:L_0603_1608Metric_Pad1.05x0.95mm_HandSolder -> (none)
- R27, R28, R29: footprint Resistor_SMD:R_0603_1608Metric_Pad0.98x0.95mm_HandSolder -> (none)
Changed lines of the file:
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@@
 			)
 		)
-		(property "Footprint" "Capacitor_SMD:C_0805_2012Metric_Pad1.18x1.45mm_HandSolder"
+		(property "Footprint" ""
 			(at 87.3252 100.33 0)
 			(effects
@@
 			)
 		)
-		(property "Footprint" "Inductor_SMD:L_0603_1608Metric_Pad1.05x0.95mm_HandSolder"
+		(property "Footprint" ""
 			(at 95.25 53.34 0)
 			(effects
@@
 			)
 		)
-		(property "Footprint" "Capacitor_SMD:C_0805_2012Metric_Pad1.18x1.45mm_HandSolder"
+		(property "Footprint" ""
 			(at 102.5652 60.96 0)
 			(effects
@@
 			)
 		)
-		(property "Footprint" "Capacitor_SMD:C_0805_2012Metric_Pad1.18x1.45mm_HandSolder"
+		(property "Footprint" ""
 			(at 102.5652 138.43 0)
 			(effects
@@
 			)
 		)
-		(property "Footprint" "Capacitor_SMD:C_0805_2012Metric_Pad1.18x1.45mm_HandSolder"
+		(property "Footprint" ""
 			(at 87.3252 60.96 0)
 			(effects
@@
 			)
 		)
-		(property "Footprint" "Resistor_SMD:R_0603_1608Metric_Pad0.98x0.95mm_HandSolder"
+		(property "Footprint" ""
 			(at 77.47 71.882 90)
 			(effects
@@
 			)
 		)
-		(property "Footprint" "Resistor_SMD:R_0603_1608Metric_Pad0.98x0.95mm_HandSolder"
+		(property "Footprint" ""
 			(at 77.47 107.442 90)
 			(effects
@@
 			)
 		)
-		(property "Footprint" "Resistor_SMD:R_0603_1608Metric_Pad0.98x0.95mm_HandSolder"
+		(property "Footprint" ""
 			(at 77.47 145.542 90)
 			(effects
@@
 			)
 		)
-		(property "Footprint" "Capacitor_SMD:C_0603_1608Metric_Pad1.08x0.95mm_HandSolder"
+		(property "Footprint" ""
 			(at 77.1652 138.43 0)
 			(effects
@@
 			)
 		)
-		(property "Footprint" "Capacitor_SMD:C_0603_1608Metric_Pad1.08x0.95mm_HandSolder"
+		(property "Footprint" ""
 			(at 77.1652 60.96 0)
 			(effects
@@
 			)
 		)
-		(property "Footprint" "Capacitor_SMD:C_0805_2012Metric_Pad1.18x1.45mm_HandSolder"
+		(property "Footprint" ""
 			(at 102.5652 100.33 0)
 			(effects
@@
 			)
 		)
-		(property "Footprint" "Capacitor_SMD:C_0805_2012Metric_Pad1.18x1.45mm_HandSolder"
+		(property "Footprint" ""
 			(at 87.3252 138.43 0)
 			(effects
@@
 			)
 		)
-		(property "Footprint" "OptoDevice:Broadcom_AFBR-16xxZ_Horizontal"
+		(property "Footprint" ""
 			(at 55.88 121.92 0)
 			(effects
@@
 			)
 		)
-		(property "Footprint" "OptoDevice:Broadcom_AFBR-16xxZ_Horizontal"
+		(property "Footprint" ""
 			(at 55.88 160.02 0)
 			(effects
@@
 			)
 		)
-		(property "Footprint" "Inductor_SMD:L_0603_1608Metric_Pad1.05x0.95mm_HandSolder"
+		(property "Footprint" ""
 			(at 95.25 92.71 0)
 			(effects
@@
 			)
 		)
-		(property "Footprint" "Inductor_SMD:L_0603_1608Metric_Pad1.05x0.95mm_HandSolder"
+		(property "Footprint" ""
 			(at 95.25 130.81 0)
 			(effects
@@
 			)
 		)
-		(property "Footprint" "Capacitor_SMD:C_0603_1608Metric_Pad1.08x0.95mm_HandSolder"
+		(property "Footprint" ""
 			(at 77.1652 100.33 0)
 			(effects
@@
 			)
 		)
-		(property "Footprint" "OptoDevice:Broadcom_AFBR-16xxZ_Horizontal"
+		(property "Footprint" ""
 			(at 55.88 86.36 0)
 			(effects

Commit message: update lib
Parts:
- C32, C33, C34: value C -> 100n; footprint (none) -> Capacitor_SMD:C_0603_1608Metric_Pad1.08x0.95mm_HandSolder
- C35, C36, C37, C38, C39, C40: value C -> 10u; footprint (none) -> Capacitor_SMD:C_0805_2012Metric_Pad1.18x1.45mm_HandSolder
- J3, J4, J5: footprint (none) -> OptoDevice:Broadcom_AFBR-16xxZ_Horizontal
- L4, L5, L6: value L -> 1u; footprint (none) -> Inductor_SMD:L_0603_1608Metric_Pad1.05x0.95mm_HandSolder
- R27, R28, R29: footprint (none) -> Resistor_SMD:R_0603_1608Metric_Pad0.98x0.95mm_HandSolder
Other:
- moved on the sheet: C35, C36, C37, C38, C39, C40, L4, L5, L6

Commit message: designator + part n°
Parts:
- renumbered C32 to C34, C33 to C35, C34 to C36, C35 to C37, C36 to C38, C37 to C39, C38 to C40, C39 to C41, C40 to C42, J3 to J7, J4 to J8, J5 to J9, R27 to R30, R28 to R31, R29 to R32
Other:
- title: Optical receptors x3 -> Optical reciver x3
Changed lines of the file:
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@@
 	(paper "A4")
 	(title_block
-		(title "Optical receptors x3")
+		(title "Optical reciver x3")
 		(rev "1")
 		(company "Dr.-Ing. Alan H. Wilson Veas")
@@
 		(dnp no)
 		(fields_autoplaced yes)
-		(property "Reference" "C36"
+		(property "Reference" "C38"
 			(at 92.71 95.2499 0)
 			(effects
@@
 			(project "HalfBridge_SiC"
 				(path "/3c187ffa-7f66-4861-b077-b6965c821fc2/6b9f2a3a-4d36-43fe-adee-f56a635b1692"
-					(reference "C36")
+					(reference "C38")
 					(unit 1)
 				)
@@
 		(dnp no)
 		(fields_autoplaced yes)
-		(property "Reference" "C38"
+		(property "Reference" "C40"
 			(at 107.95 55.8799 0)
 			(effects
@@
 			(project "HalfBridge_SiC"
 				(path "/3c187ffa-7f66-4861-b077-b6965c821fc2/6b9f2a3a-4d36-43fe-adee-f56a635b1692"
-					(reference "C38")
+					(reference "C40")
 					(unit 1)
 				)
@@
 		(dnp no)
 		(fields_autoplaced yes)
-		(property "Reference" "C40"
+		(property "Reference" "C42"
 			(at 107.95 133.3499 0)
 			(effects
@@
 			(project "HalfBridge_SiC"
 				(path "/3c187ffa-7f66-4861-b077-b6965c821fc2/6b9f2a3a-4d36-43fe-adee-f56a635b1692"
-					(reference "C40")
+					(reference "C42")
 					(unit 1)
 				)
@@
 		(dnp no)
 		(fields_autoplaced yes)
-		(property "Reference" "C35"
+		(property "Reference" "C37"
 			(at 92.71 55.8799 0)
 			(effects
@@
 			(project "HalfBridge_SiC"
 				(path "/3c187ffa-7f66-4861-b077-b6965c821fc2/6b9f2a3a-4d36-43fe-adee-f56a635b1692"
-					(reference "C35")
+					(reference "C37")
 					(unit 1)
 				)
@@
 		(on_board yes)
 		(dnp no)
-		(property "Reference" "R27"
+		(property "Reference" "R30"
 			(at 77.47 67.31 90)
 			(effects
@@
 			(project "HalfBridge_SiC"
 				(path "/3c187ffa-7f66-4861-b077-b6965c821fc2/6b9f2a3a-4d36-43fe-adee-f56a635b1692"
-					(reference "R27")
+					(reference "R30")
 					(unit 1)
 				)
@@
 		(on_board yes)
 		(dnp no)
-		(property "Reference" "R28"
+		(property "Reference" "R31"
 			(at 77.47 102.87 90)
 			(effects
@@
 			(project ""
 				(path "/3c187ffa-7f66-4861-b077-b6965c821fc2/6b9f2a3a-4d36-43fe-adee-f56a635b1692"
-					(reference "R28")
+					(reference "R31")
 					(unit 1)
 				)
@@
 		(on_board yes)
 		(dnp no)
-		(property "Reference" "R29"
+		(property "Reference" "R32"
 			(at 77.47 140.97 90)
 			(effects
@@
 			(project "HalfBridge_SiC"
 				(path "/3c187ffa-7f66-4861-b077-b6965c821fc2/6b9f2a3a-4d36-43fe-adee-f56a635b1692"
-					(reference "R29")
+					(reference "R32")
 					(unit 1)
 				)
@@
 		(dnp no)
 		(fields_autoplaced yes)
-		(property "Reference" "C34"
+		(property "Reference" "C36"
 			(at 80.01 133.3499 0)
 			(effects
@@
 			(project "HalfBridge_SiC"
 				(path "/3c187ffa-7f66-4861-b077-b6965c821fc2/6b9f2a3a-4d36-43fe-adee-f56a635b1692"
-					(reference "C34")
+					(reference "C36")
 					(unit 1)
 				)
@@
 		(dnp no)
 		(fields_autoplaced yes)
-		(property "Reference" "C32"
+		(property "Reference" "C34"
 			(at 80.01 55.8799 0)
 			(effects
@@
 			(project "HalfBridge_SiC"
 				(path "/3c187ffa-7f66-4861-b077-b6965c821fc2/6b9f2a3a-4d36-43fe-adee-f56a635b1692"
-					(reference "C32")
+					(reference "C34")
 					(unit 1)
 				)
@@
 		(dnp no)
 		(fields_autoplaced yes)
-		(property "Reference" "C39"
+		(property "Reference" "C41"
 			(at 107.95 95.2499 0)
 			(effects
@@
 			(project "HalfBridge_SiC"
 				(path "/3c187ffa-7f66-4861-b077-b6965c821fc2/6b9f2a3a-4d36-43fe-adee-f56a635b1692"
-					(reference "C39")
+					(reference "C41")
 					(unit 1)
 				)
@@
 		(on_board yes)
 		(dnp no)
-		(property "Reference" "C37"
+		(property "Reference" "C39"
 			(at 92.71 133.3499 0)
 			(effects
@@
 			(project "HalfBridge_SiC"
 				(path "/3c187ffa-7f66-4861-b077-b6965c821fc2/6b9f2a3a-4d36-43fe-adee-f56a635b1692"
-					(reference "C37")
+					(reference "C39")
 					(unit 1)
 				)
@@
 		(dnp no)
 		(fields_autoplaced yes)
-		(property "Reference" "J4"
+		(property "Reference" "J8"
 			(at 49.53 107.9499 0)
 			(effects
@@
 			(project "HalfBridge_SiC"
 				(path "/3c187ffa-7f66-4861-b077-b6965c821fc2/6b9f2a3a-4d36-43fe-adee-f56a635b1692"
-					(reference "J4")
+					(reference "J8")
 					(unit 1)
 				)
@@
 		(dnp no)
 		(fields_autoplaced yes)
-		(property "Reference" "J5"
+		(property "Reference" "J9"
 			(at 49.53 146.0499 0)
 			(effects
@@
 			(project "HalfBridge_SiC"
 				(path "/3c187ffa-7f66-4861-b077-b6965c821fc2/6b9f2a3a-4d36-43fe-adee-f56a635b1692"
-					(reference "J5")
+					(reference "J9")
 					(unit 1)
 				)
@@
 		(dnp no)
 		(fields_autoplaced yes)
-		(property "Reference" "C33"
+		(property "Reference" "C35"
 			(at 80.01 95.2499 0)
 			(effects
@@
 			(project "HalfBridge_SiC"
 				(path "/3c187ffa-7f66-4861-b077-b6965c821fc2/6b9f2a3a-4d36-43fe-adee-f56a635b1692"
-					(reference "C33")
+					(reference "C35")
 					(unit 1)
 				)
@@
 		(dnp no)
 		(fields_autoplaced yes)
-		(property "Reference" "J3"
+		(property "Reference" "J7"
 			(at 49.53 72.3899 0)
 			(effects
@@
 			(project ""
 				(path "/3c187ffa-7f66-4861-b077-b6965c821fc2/6b9f2a3a-4d36-43fe-adee-f56a635b1692"
-					(reference "J3")
+					(reference "J7")
 					(unit 1)
 				)
