File: pcb/HalfBridge_SiC/HalfBridge_Optical.kicad_sch (KiCad schematic)
At the start: 18 parts, among them J7 AFBR-2624Z, J8 AFBR-2624Z, J9 AFBR-2624Z

Commit message: titles
Parts:
- C34, C35, C36: Part # (none) -> UMK107BJ104KAHT
- C37, C38, C39, C40, C41, C42: Part # (none) -> GRM21BR61H106KE43L
- J7, J8, J9: Part # (none) -> AFBR-2624Z
Changed lines of the file:
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@@
+			)
+		)
+		(property "Part #" "GRM21BR61H106KE43L"
+			(at 88.9 96.52 0)
+			(effects
+				(font
+					(size 1.27 1.27)
+				)
+				(hide yes)
 			)
 		)
@@
 			)
 		)
+		(property "Part #" "GRM21BR61H106KE43L"
+			(at 104.14 57.15 0)
+			(effects
+				(font
+					(size 1.27 1.27)
+				)
+				(hide yes)
+			)
+		)
 		(pin "2"
 		)
@@
 			)
 		)
+		(property "Part #" "GRM21BR61H106KE43L"
+			(at 104.14 134.62 0)
+			(effects
+				(font
+					(size 1.27 1.27)
+				)
+				(hide yes)
+			)
+		)
 		(pin "2"
 		)
@@
 			)
 		)
+		(property "Part #" "GRM21BR61H106KE43L"
+			(at 88.9 57.15 0)
+			(effects
+				(font
+					(size 1.27 1.27)
+				)
+				(hide yes)
+			)
+		)
 		(pin "2"
 		)
@@
 			)
 		)
+		(property "Part #" "UMK107BJ104KAHT"
+			(at 76.2 134.62 0)
+			(effects
+				(font
+					(size 1.27 1.27)
+				)
+				(hide yes)
+			)
+		)
 		(pin "1"
 		)
@@
 			)
 		)
+		(property "Part #" "UMK107BJ104KAHT"
+			(at 76.2 57.15 0)
+			(effects
+				(font
+					(size 1.27 1.27)
+				)
+				(hide yes)
+			)
+		)
 		(pin "1"
 		)
@@
 			)
 		)
+		(property "Part #" "GRM21BR61H106KE43L"
+			(at 104.14 96.52 0)
+			(effects
+				(font
+					(size 1.27 1.27)
+				)
+				(hide yes)
+			)
+		)
 		(pin "2"
 		)
@@
 		)
 		(property "Description" "Unpolarized capacitor"
+			(at 88.9 134.62 0)
+			(effects
+				(font
+					(size 1.27 1.27)
+				)
+				(hide yes)
+			)
+		)
+		(property "Part #" "GRM21BR61H106KE43L"
 			(at 88.9 134.62 0)
 			(effects
@@
 			)
 		)
+		(property "Part #" "AFBR-2624Z"
+			(at 58.42 109.22 0)
+			(effects
+				(font
+					(size 1.27 1.27)
+				)
+				(hide yes)
+			)
+		)
 		(pin "3"
 		)
@@
 			)
 		)
+		(property "Part #" "AFBR-2624Z"
+			(at 58.42 147.32 0)
+			(effects
+				(font
+					(size 1.27 1.27)
+				)
+				(hide yes)
+			)
+		)
 		(pin "3"
 		)
@@
 			)
 		)
+		(property "Part #" "UMK107BJ104KAHT"
+			(at 76.2 96.52 0)
+			(effects
+				(font
+					(size 1.27 1.27)
+				)
+				(hide yes)
+			)
+		)
 		(pin "1"
 		)
@@
 			(at 58.42 73.66 0)
 			(effects
+				(font
+					(size 1.27 1.27)
+				)
+				(hide yes)
+			)
+		)
+		(property "Part #" "AFBR-2624Z"
+			(at 58.42 73.66 0)
+			(effects
