File: pcb/HalfBridge_SiC/HalfBridge_Diff.kicad_sch (KiCad schematic)
At the start: 19 parts, among them J10 Conn_01x02, J11 Conn_01x02, J12 Conn_01x02, J14 Conn_01x02_Shielded, J7 Conn_01x02, J8 Conn_01x02, J9 Conn_01x02, U7 MAX3284E, U8 MAX3284E, U9 MAX3284E

Commit message: vgatereg + route + hsink
Parts:
- removed J10, J12, J7, J8: Conn_01x02, Connector_PinHeader_2.54mm:PinHeader_1x02_P2.54mm_Vertical, symbol Connector_Generic:Conn_01x02
- added J11: Conn_01x02, Connector_PinHeader_2.54mm:PinHeader_1x02_P2.54mm_Horizontal, symbol Connector_Generic:Conn_01x02
- added J7, J8: Conn_01x02_Shielded, My_Connector:SAMTEC_T1M-02-F-SH-L-K, symbol Connector_Generic_Shielded:Conn_01x02_Shielded
- added TP10, TP5, TP6, TP7, TP8, TP9: TestPoint, TestPoint:TestPoint_Keystone_5015_Micro-Minature, symbol Connector:TestPoint
- J10: renamed from J11; footprint Connector_PinHeader_2.54mm:PinHeader_1x02_P2.54mm_Vertical -> Connector_PinHeader_2.54mm:PinHeader_1x02_P2.54mm_Horizontal
- J6: renamed from J14; footprint My_Connector:SAMTEC_T1M-02-F-SV-L-P -> My_Connector:SAMTEC_T1M-02-F-SH-L-K
- J9: footprint Connector_PinHeader_2.54mm:PinHeader_1x02_P2.54mm_Vertical -> Connector_PinHeader_2.54mm:PinHeader_1x02_P2.54mm_Horizontal; now fitted
- R33: renamed from R25; footprint Resistor_SMD:R_0603_1608Metric -> Resistor_SMD:R_0603_1608Metric_Pad0.98x0.95mm_HandSolder
- R34: renamed from R27; footprint Resistor_SMD:R_0603_1608Metric -> Resistor_SMD:R_0603_1608Metric_Pad0.98x0.95mm_HandSolder
- R35: renamed from R26; footprint Resistor_SMD:R_0603_1608Metric -> Resistor_SMD:R_0603_1608Metric_Pad0.98x0.95mm_HandSolder
- renumbered C31 to C37, C32 to C38, C33 to C39, R22 to R30, R23 to R31, R24 to R32, U8 to U10, U9 to U11, U7 to U9
Connections:
- net gnd: now also J9.2 (Pin_2), J11.2 (Pin_2), J7.SH (Shield), J8.SH (Shield)
- net ina_d: now also J9.1 (Pin_1)
- net ina_da: now also J7.1 (Pin_1), TP5.1
- net ina_db: now also J7.2 (Pin_2), TP6.1
- net inb_da: now also TP7.1
- net inb_db: now also TP8.1
- net inen_d: now also J11.1 (Pin_1)
- net inen_da: now also J8.1 (Pin_1), TP9.1; no longer J9.2 (Pin_2)
- net inen_db: now also J8.2 (Pin_2), TP10.1; no longer J9.1 (Pin_1)

Commit message: comment + gdriver + logo
Parts:
- R30, R31, R32: value R -> 120
- R33, R34, R35: value R -> 0
- renumbered C37 to C41, C38 to C42, C39 to C43
Other:
- title: (none) -> Differential receptors x3
- moved on the sheet: J6, J7, J8, R30, R31, R32, TP10, TP5, TP6, TP7, TP8, TP9

Commit message: local lib
Parts:
- C41, C42, C43: symbol Device:C -> HalfBridge_SiC:C
- J10, J11, J9: symbol Connector_Generic:Conn_01x02 -> HalfBridge_SiC:Conn_01x02
- J6, J7, J8: symbol Connector_Generic_Shielded:Conn_01x02_Shielded -> HalfBridge_SiC:Conn_01x02_Shielded
- R30, R31, R32, R33, R34, R35: symbol Device:R -> HalfBridge_SiC:R
- TP10, TP5, TP6, TP7, TP8, TP9: symbol Connector:TestPoint -> HalfBridge_SiC:TestPoint
- U10, U11, U9: symbol Interface_UART:MAX3284E -> HalfBridge_SiC:MAX3284E
Changed lines of the file:
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@@
 	)
 	(symbol
-		(lib_id "Connector_Generic_Shielded:Conn_01x02_Shielded")
+		(lib_id "HalfBridge_SiC:Conn_01x02_Shielded")
 		(at 52.07 105.41 0)
 		(mirror y)
@@
 	)
 	(symbol
-		(lib_id "Connector:TestPoint")
+		(lib_id "HalfBridge_SiC:TestPoint")
 		(at 68.58 137.16 0)
 		(unit 1)
@@
 	)
 	(symbol
-		(lib_id "Device:R")
+		(lib_id "HalfBridge_SiC:R")
 		(at 118.11 105.41 90)
 		(unit 1)
@@
 	)
 	(symbol
-		(lib_id "Device:R")
+		(lib_id "HalfBridge_SiC:R")
 		(at 116.84 140.97 90)
 		(unit 1)
@@
 	)
 	(symbol
-		(lib_id "Device:R")
+		(lib_id "HalfBridge_SiC:R")
 		(at 116.84 67.31 90)
 		(unit 1)
@@
 	)
 	(symbol
-		(lib_id "Device:C")
+		(lib_id "HalfBridge_SiC:C")
 		(at 105.41 91.44 90)
 		(unit 1)
@@
 	)
 	(symbol
-		(lib_id "Connector:TestPoint")
+		(lib_id "HalfBridge_SiC:TestPoint")
 		(at 68.58 144.78 180)
 		(unit 1)
@@
 	)
 	(symbol
-		(lib_id "Connector:TestPoint")
+		(lib_id "HalfBridge_SiC:TestPoint")
 		(at 68.58 71.12 180)
 		(unit 1)
@@
 	)
 	(symbol
-		(lib_id "Connector_Generic:Conn_01x02")
+		(lib_id "HalfBridge_SiC:Conn_01x02")
 		(at 127 111.76 0)
 		(unit 1)
@@
 	)
 	(symbol
-		(lib_id "Device:R")
+		(lib_id "HalfBridge_SiC:R")
 		(at 68.58 140.97 0)
 		(unit 1)
@@
 	)
 	(symbol
-		(lib_id "Connector_Generic_Shielded:Conn_01x02_Shielded")
+		(lib_id "HalfBridge_SiC:Conn_01x02_Shielded")
 		(at 52.07 140.97 0)
 		(mirror y)
@@
 	)
 	(symbol
-		(lib_id "Device:C")
+		(lib_id "HalfBridge_SiC:C")
 		(at 105.41 127 90)
 		(unit 1)
@@
 	)
 	(symbol
-		(lib_id "Connector_Generic:Conn_01x02")
+		(lib_id "HalfBridge_SiC:Conn_01x02")
 		(at 127 147.32 0)
 		(unit 1)
@@
 	)
 	(symbol
-		(lib_id "Connector:TestPoint")
+		(lib_id "HalfBridge_SiC:TestPoint")
 		(at 68.58 109.22 180)
 		(unit 1)
@@
 	)
 	(symbol
-		(lib_id "Device:R")
+		(lib_id "HalfBridge_SiC:R")
 		(at 68.58 67.31 0)
 		(unit 1)
@@
 	)
 	(symbol
-		(lib_id "Connector_Generic:Conn_01x02")
+		(lib_id "HalfBridge_SiC:Conn_01x02")
 		(at 125.73 73.66 0)
 		(unit 1)
@@
 	)
 	(symbol
-		(lib_id "Device:C")
+		(lib_id "HalfBridge_SiC:C")
 		(at 105.41 53.34 90)
 		(unit 1)
@@
 	)
 	(symbol
-		(lib_id "Interface_UART:MAX3284E")
+		(lib_id "HalfBridge_SiC:MAX3284E")
 		(at 97.79 105.41 0)
 		(unit 1)
@@
 	)
 	(symbol
-		(lib_id "Interface_UART:MAX3284E")
+		(lib_id "HalfBridge_SiC:MAX3284E")
 		(at 97.79 67.31 0)
 		(unit 1)
@@
 	)
 	(symbol
-		(lib_id "Connector:TestPoint")
+		(lib_id "HalfBridge_SiC:TestPoint")
 		(at 68.58 63.5 0)
 		(unit 1)
@@
 	)
 	(symbol
-		(lib_id "Interface_UART:MAX3284E")
+		(lib_id "HalfBridge_SiC:MAX3284E")
 		(at 97.79 140.97 0)
 		(unit 1)
@@
 	)
 	(symbol
-		(lib_id "Device:R")
+		(lib_id "HalfBridge_SiC:R")
 		(at 68.58 105.41 0)
 		(unit 1)
@@
 	)
 	(symbol
-		(lib_id "Connector_Generic_Shielded:Conn_01x02_Shielded")
+		(lib_id "HalfBridge_SiC:Conn_01x02_Shielded")
 		(at 53.34 66.04 0)
 		(mirror y)
@@
 	)
 	(symbol
-		(lib_id "Connector:TestPoint")
+		(lib_id "HalfBridge_SiC:TestPoint")
 		(at 68.58 101.6 0)
 		(unit 1)

Commit message: pcb + newlib
Other:
- company: (none) -> Dr.-Ing. Alan H. Wilson Veas
Changed lines of the file:
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@@
 		(title "Differential receptors x3")
 		(rev "1")
+		(company "Dr.-Ing. Alan H. Wilson Veas")
+		(comment 1 "AHWV")
 	)
 	(junction

Commit message: backplane + external lib
Parts:
- C41, C42, C43: footprint Capacitor_SMD:C_0603_1608Metric_Pad1.08x0.95mm_HandSolder -> (none)
- J10, J11, J9: footprint Connector_PinHeader_2.54mm:PinHeader_1x02_P2.54mm_Horizontal -> (none)
- J6, J7, J8: footprint My_Connector:SAMTEC_T1M-02-F-SH-L-K -> (none)
- R30, R31, R32, R33, R34, R35: footprint Resistor_SMD:R_0603_1608Metric_Pad0.98x0.95mm_HandSolder -> (none)
- TP10, TP5, TP6, TP7, TP8, TP9: footprint TestPoint:TestPoint_Keystone_5015_Micro-Minature -> (none)
- U10, U11, U9: footprint Package_TO_SOT_SMD:SOT-23-6_Handsoldering -> Package_TO_SOT_SMD:SOT-23-6
Changed lines of the file:
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@@
 			)
 		)
-		(property "Footprint" "My_Connector:SAMTEC_T1M-02-F-SH-L-K"
+		(property "Footprint" ""
 			(at 52.07 105.41 0)
 			(effects
@@
 			)
 		)
-		(property "Footprint" "TestPoint:TestPoint_Keystone_5015_Micro-Minature"
+		(property "Footprint" ""
 			(at 73.66 137.16 0)
 			(effects
@@
 			)
 		)
-		(property "Footprint" "Resistor_SMD:R_0603_1608Metric_Pad0.98x0.95mm_HandSolder"
+		(property "Footprint" ""
 			(at 118.11 107.188 90)
 			(effects
@@
 			)
 		)
-		(property "Footprint" "Resistor_SMD:R_0603_1608Metric_Pad0.98x0.95mm_HandSolder"
+		(property "Footprint" ""
 			(at 116.84 142.748 90)
 			(effects
@@
 			)
 		)
-		(property "Footprint" "Resistor_SMD:R_0603_1608Metric_Pad0.98x0.95mm_HandSolder"
+		(property "Footprint" ""
 			(at 116.84 69.088 90)
 			(effects
@@
 			)
 		)
-		(property "Footprint" "Capacitor_SMD:C_0603_1608Metric_Pad1.08x0.95mm_HandSolder"
+		(property "Footprint" ""
 			(at 109.22 90.4748 0)
 			(effects
@@
 			)
 		)
-		(property "Footprint" "TestPoint:TestPoint_Keystone_5015_Micro-Minature"
+		(property "Footprint" ""
 			(at 63.5 144.78 0)
 			(effects
@@
 			)
 		)
-		(property "Footprint" "TestPoint:TestPoint_Keystone_5015_Micro-Minature"
+		(property "Footprint" ""
 			(at 63.5 71.12 0)
 			(effects
@@
 			)
 		)
-		(property "Footprint" "Connector_PinHeader_2.54mm:PinHeader_1x02_P2.54mm_Horizontal"
+		(property "Footprint" ""
 			(at 127 111.76 0)
 			(effects
@@
 			)
 		)
-		(property "Footprint" "Resistor_SMD:R_0603_1608Metric_Pad0.98x0.95mm_HandSolder"
+		(property "Footprint" ""
 			(at 66.802 140.97 90)
 			(effects
@@
 			)
 		)
-		(property "Footprint" "My_Connector:SAMTEC_T1M-02-F-SH-L-K"
+		(property "Footprint" ""
 			(at 52.07 140.97 0)
 			(effects
@@
 			)
 		)
-		(property "Footprint" "Capacitor_SMD:C_0603_1608Metric_Pad1.08x0.95mm_HandSolder"
+		(property "Footprint" ""
 			(at 109.22 126.0348 0)
 			(effects
@@
 			)
 		)
-		(property "Footprint" "Connector_PinHeader_2.54mm:PinHeader_1x02_P2.54mm_Horizontal"
+		(property "Footprint" ""
 			(at 127 147.32 0)
 			(effects
@@
 			)
 		)
-		(property "Footprint" "TestPoint:TestPoint_Keystone_5015_Micro-Minature"
+		(property "Footprint" ""
 			(at 63.5 109.22 0)
 			(effects
@@
 			)
 		)
-		(property "Footprint" "Resistor_SMD:R_0603_1608Metric_Pad0.98x0.95mm_HandSolder"
+		(property "Footprint" ""
 			(at 66.802 67.31 90)
 			(effects
@@
 			)
 		)
-		(property "Footprint" "Connector_PinHeader_2.54mm:PinHeader_1x02_P2.54mm_Horizontal"
+		(property "Footprint" ""
 			(at 125.73 73.66 0)
 			(effects
@@
 			)
 		)
-		(property "Footprint" "Capacitor_SMD:C_0603_1608Metric_Pad1.08x0.95mm_HandSolder"
+		(property "Footprint" ""
 			(at 109.22 52.3748 0)
 			(effects
@@
 			)
 		)
-		(property "Footprint" "Package_TO_SOT_SMD:SOT-23-6_Handsoldering"
+		(property "Footprint" "Package_TO_SOT_SMD:SOT-23-6"
 			(at 97.79 123.19 0)
 			(effects
@@
 			)
 		)
-		(property "Footprint" "Package_TO_SOT_SMD:SOT-23-6_Handsoldering"
+		(property "Footprint" "Package_TO_SOT_SMD:SOT-23-6"
 			(at 97.79 85.09 0)
 			(effects
@@
 			)
 		)
-		(property "Footprint" "TestPoint:TestPoint_Keystone_5015_Micro-Minature"
+		(property "Footprint" ""
 			(at 73.66 63.5 0)
 			(effects
@@
 			)
 		)
-		(property "Footprint" "Package_TO_SOT_SMD:SOT-23-6_Handsoldering"
+		(property "Footprint" "Package_TO_SOT_SMD:SOT-23-6"
 			(at 97.79 158.75 0)
 			(effects
@@
 			)
 		)
-		(property "Footprint" "Resistor_SMD:R_0603_1608Metric_Pad0.98x0.95mm_HandSolder"
+		(property "Footprint" ""
 			(at 66.802 105.41 90)
 			(effects
@@
 			)
 		)
-		(property "Footprint" "My_Connector:SAMTEC_T1M-02-F-SH-L-K"
+		(property "Footprint" ""
 			(at 53.34 66.04 0)
 			(effects
@@
 			)
 		)
-		(property "Footprint" "TestPoint:TestPoint_Keystone_5015_Micro-Minature"
+		(property "Footprint" ""
 			(at 73.66 101.6 0)
 			(effects

Commit message: update lib
Parts:
- C41, C42, C43: footprint (none) -> Capacitor_SMD:C_0603_1608Metric_Pad1.08x0.95mm_HandSolder
- J10, J11, J9: footprint (none) -> Connector_PinHeader_2.54mm:PinHeader_1x02_P2.54mm_Horizontal
- J6, J7, J8: footprint (none) -> My_Connector:SAMTEC_T1M-02-F-SH-L-K
- R30, R31, R32, R33, R34, R35: footprint (none) -> Resistor_SMD:R_0603_1608Metric_Pad0.98x0.95mm_HandSolder
- TP10, TP5, TP6, TP7, TP8, TP9: footprint (none) -> TestPoint:TestPoint_Keystone_5015_Micro-Minature
Changed lines of the file:
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@@
 			)
 		)
-		(property "Footprint" ""
+		(property "Footprint" "My_Connector:SAMTEC_T1M-02-F-SH-L-K"
 			(at 52.07 105.41 0)
 			(effects
@@
 			)
 		)
-		(property "Footprint" ""
+		(property "Footprint" "TestPoint:TestPoint_Keystone_5015_Micro-Minature"
 			(at 73.66 137.16 0)
 			(effects
@@
 			)
 		)
-		(property "Footprint" ""
+		(property "Footprint" "Resistor_SMD:R_0603_1608Metric_Pad0.98x0.95mm_HandSolder"
 			(at 118.11 107.188 90)
 			(effects
@@
 			)
 		)
-		(property "Footprint" ""
+		(property "Footprint" "Resistor_SMD:R_0603_1608Metric_Pad0.98x0.95mm_HandSolder"
 			(at 116.84 142.748 90)
 			(effects
@@
 			)
 		)
-		(property "Footprint" ""
+		(property "Footprint" "Resistor_SMD:R_0603_1608Metric_Pad0.98x0.95mm_HandSolder"
 			(at 116.84 69.088 90)
 			(effects
@@
 			)
 		)
-		(property "Footprint" ""
+		(property "Footprint" "Capacitor_SMD:C_0603_1608Metric_Pad1.08x0.95mm_HandSolder"
 			(at 109.22 90.4748 0)
 			(effects
@@
 			)
 		)
-		(property "Footprint" ""
+		(property "Footprint" "TestPoint:TestPoint_Keystone_5015_Micro-Minature"
 			(at 63.5 144.78 0)
 			(effects
@@
 			)
 		)
-		(property "Footprint" ""
+		(property "Footprint" "TestPoint:TestPoint_Keystone_5015_Micro-Minature"
 			(at 63.5 71.12 0)
 			(effects
@@
 			)
 		)
-		(property "Footprint" ""
+		(property "Footprint" "Connector_PinHeader_2.54mm:PinHeader_1x02_P2.54mm_Horizontal"
 			(at 127 111.76 0)
 			(effects
@@
 			)
 		)
-		(property "Footprint" ""
+		(property "Footprint" "Resistor_SMD:R_0603_1608Metric_Pad0.98x0.95mm_HandSolder"
 			(at 66.802 140.97 90)
 			(effects
@@
 			)
 		)
-		(property "Footprint" ""
+		(property "Footprint" "My_Connector:SAMTEC_T1M-02-F-SH-L-K"
 			(at 52.07 140.97 0)
 			(effects
@@
 			)
 		)
-		(property "Footprint" ""
+		(property "Footprint" "Capacitor_SMD:C_0603_1608Metric_Pad1.08x0.95mm_HandSolder"
 			(at 109.22 126.0348 0)
 			(effects
@@
 			)
 		)
-		(property "Footprint" ""
+		(property "Footprint" "Connector_PinHeader_2.54mm:PinHeader_1x02_P2.54mm_Horizontal"
 			(at 127 147.32 0)
 			(effects
@@
 			)
 		)
-		(property "Footprint" ""
+		(property "Footprint" "TestPoint:TestPoint_Keystone_5015_Micro-Minature"
 			(at 63.5 109.22 0)
 			(effects
@@
 			)
 		)
-		(property "Footprint" ""
+		(property "Footprint" "Resistor_SMD:R_0603_1608Metric_Pad0.98x0.95mm_HandSolder"
 			(at 66.802 67.31 90)
 			(effects
@@
 			)
 		)
-		(property "Footprint" ""
+		(property "Footprint" "Connector_PinHeader_2.54mm:PinHeader_1x02_P2.54mm_Horizontal"
 			(at 125.73 73.66 0)
 			(effects
@@
 			)
 		)
-		(property "Footprint" ""
+		(property "Footprint" "Capacitor_SMD:C_0603_1608Metric_Pad1.08x0.95mm_HandSolder"
 			(at 109.22 52.3748 0)
 			(effects
@@
 			)
 		)
-		(property "Footprint" ""
+		(property "Footprint" "TestPoint:TestPoint_Keystone_5015_Micro-Minature"
 			(at 73.66 63.5 0)
 			(effects
@@
 			)
 		)
-		(property "Footprint" ""
+		(property "Footprint" "Resistor_SMD:R_0603_1608Metric_Pad0.98x0.95mm_HandSolder"
 			(at 66.802 105.41 90)
 			(effects
@@
 			)
 		)
-		(property "Footprint" ""
+		(property "Footprint" "My_Connector:SAMTEC_T1M-02-F-SH-L-K"
 			(at 53.34 66.04 0)
 			(effects
@@
 			)
 		)
-		(property "Footprint" ""
+		(property "Footprint" "TestPoint:TestPoint_Keystone_5015_Micro-Minature"
 			(at 73.66 101.6 0)
 			(effects

Commit message: designator + part n°
Parts:
- renumbered C41 to C43, C42 to C44, C43 to C45, J6 to J10, J8 to J11, J7 to J12, J9 to J13, J10 to J14, J11 to J15, R30 to R33, R31 to R34, R32 to R35, R33 to R36, R34 to R37, R35 to R38, TP7 to TP10, TP8 to TP11, TP9 to TP12, TP10 to TP13, TP5 to TP8, TP6 to TP9
Other:
- title: Differential receptors x3 -> Differential receiver x3
Changed lines of the file:
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@@
 	(paper "A4")
 	(title_block
-		(title "Differential receptors x3")
+		(title "Differential receiver x3")
 		(rev "1")
 		(company "Dr.-Ing. Alan H. Wilson Veas")
@@
 		(on_board yes)
 		(dnp no)
-		(property "Reference" "J6"
+		(property "Reference" "J10"
 			(at 49.53 105.4099 0)
 			(effects
@@
 			(project ""
 				(path "/3c187ffa-7f66-4861-b077-b6965c821fc2/2168827a-beb7-4093-81fb-f68e70ab414e"
-					(reference "J6")
+					(reference "J10")
 					(unit 1)
 				)
@@
 		(dnp no)
 		(fields_autoplaced yes)
-		(property "Reference" "TP9"
+		(property "Reference" "TP12"
 			(at 71.12 132.5879 0)
 			(effects
@@
 			(project "HalfBridge_SiC"
 				(path "/3c187ffa-7f66-4861-b077-b6965c821fc2/2168827a-beb7-4093-81fb-f68e70ab414e"
-					(reference "TP9")
+					(reference "TP12")
 					(unit 1)
 				)
@@
 		(dnp no)
 		(fields_autoplaced yes)
-		(property "Reference" "R35"
+		(property "Reference" "R38"
 			(at 118.11 99.06 90)
 			(effects
@@
 			(project "HalfBridge_SiC"
 				(path "/3c187ffa-7f66-4861-b077-b6965c821fc2/2168827a-beb7-4093-81fb-f68e70ab414e"
-					(reference "R35")
+					(reference "R38")
 					(unit 1)
 				)
@@
 		(dnp no)
 		(fields_autoplaced yes)
-		(property "Reference" "R34"
+		(property "Reference" "R37"
 			(at 116.84 134.62 90)
 			(effects
@@
 			(project "HalfBridge_SiC"
 				(path "/3c187ffa-7f66-4861-b077-b6965c821fc2/2168827a-beb7-4093-81fb-f68e70ab414e"
-					(reference "R34")
+					(reference "R37")
 					(unit 1)
 				)
@@
 		(dnp no)
 		(fields_autoplaced yes)
-		(property "Reference" "R33"
+		(property "Reference" "R36"
 			(at 116.84 60.96 90)
 			(effects
@@
 			(project "HalfBridge_SiC"
 				(path "/3c187ffa-7f66-4861-b077-b6965c821fc2/2168827a-beb7-4093-81fb-f68e70ab414e"
-					(reference "R33")
+					(reference "R36")
 					(unit 1)
 				)
@@
 		(dnp no)
 		(fields_autoplaced yes)
-		(property "Reference" "C42"
+		(property "Reference" "C44"
 			(at 105.41 83.82 90)
 			(effects
@@
 			(project "HalfBridge_SiC"
 				(path "/3c187ffa-7f66-4861-b077-b6965c821fc2/2168827a-beb7-4093-81fb-f68e70ab414e"
-					(reference "C42")
+					(reference "C44")
 					(unit 1)
 				)
@@
 		(dnp no)
 		(fields_autoplaced yes)
-		(property "Reference" "TP10"
+		(property "Reference" "TP13"
 			(at 71.12 146.8119 0)
 			(effects
@@
 			(project "HalfBridge_SiC"
 				(path "/3c187ffa-7f66-4861-b077-b6965c821fc2/2168827a-beb7-4093-81fb-f68e70ab414e"
-					(reference "TP10")
+					(reference "TP13")
 					(unit 1)
 				)
@@
 		(dnp no)
 		(fields_autoplaced yes)
-		(property "Reference" "TP6"
+		(property "Reference" "TP9"
 			(at 71.12 73.1519 0)
 			(effects
@@
 			(project "HalfBridge_SiC"
 				(path "/3c187ffa-7f66-4861-b077-b6965c821fc2/2168827a-beb7-4093-81fb-f68e70ab414e"
-					(reference "TP6")
+					(reference "TP9")
 					(unit 1)
 				)
@@
 		(on_board yes)
 		(dnp no)
-		(property "Reference" "J10"
+		(property "Reference" "J14"
 			(at 129.54 111.7599 0)
 			(effects
@@
 			(project "HalfBridge_SiC"
 				(path "/3c187ffa-7f66-4861-b077-b6965c821fc2/2168827a-beb7-4093-81fb-f68e70ab414e"
-					(reference "J10")
+					(reference "J14")
 					(unit 1)
 				)
@@
 		(dnp no)
 		(fields_autoplaced yes)
-		(property "Reference" "R32"
+		(property "Reference" "R35"
 			(at 71.12 139.6999 0)
 			(effects
@@
 			(project "HalfBridge_SiC"
 				(path "/3c187ffa-7f66-4861-b077-b6965c821fc2/2168827a-beb7-4093-81fb-f68e70ab414e"
-					(reference "R32")
+					(reference "R35")
 					(unit 1)
 				)
@@
 		(on_board yes)
 		(dnp no)
-		(property "Reference" "J8"
+		(property "Reference" "J11"
 			(at 49.53 140.9699 0)
 			(effects
@@
 			(project "HalfBridge_SiC"
 				(path "/3c187ffa-7f66-4861-b077-b6965c821fc2/2168827a-beb7-4093-81fb-f68e70ab414e"
-					(reference "J8")
+					(reference "J11")
 					(unit 1)
 				)
@@
 		(dnp no)
 		(fields_autoplaced yes)
-		(property "Reference" "C43"
+		(property "Reference" "C45"
 			(at 105.41 119.38 90)
 			(effects
@@
 			(project "HalfBridge_SiC"
 				(path "/3c187ffa-7f66-4861-b077-b6965c821fc2/2168827a-beb7-4093-81fb-f68e70ab414e"
-					(reference "C43")
+					(reference "C45")
 					(unit 1)
 				)
@@
 		(on_board yes)
 		(dnp no)
-		(property "Reference" "J11"
+		(property "Reference" "J15"
 			(at 129.54 147.3199 0)
 			(effects
@@
 			(project "HalfBridge_SiC"
 				(path "/3c187ffa-7f66-4861-b077-b6965c821fc2/2168827a-beb7-4093-81fb-f68e70ab414e"
-					(reference "J11")
+					(reference "J15")
 					(unit 1)
 				)
@@
 		(dnp no)
 		(fields_autoplaced yes)
-		(property "Reference" "TP8"
+		(property "Reference" "TP11"
 			(at 71.12 111.2519 0)
 			(effects
@@
 			(project "HalfBridge_SiC"
 				(path "/3c187ffa-7f66-4861-b077-b6965c821fc2/2168827a-beb7-4093-81fb-f68e70ab414e"
-					(reference "TP8")
+					(reference "TP11")
 					(unit 1)
 				)
@@
 		(dnp no)
 		(fields_autoplaced yes)
-		(property "Reference" "R30"
+		(property "Reference" "R33"
 			(at 71.12 66.0399 0)
 			(effects
@@
 			(project ""
 				(path "/3c187ffa-7f66-4861-b077-b6965c821fc2/2168827a-beb7-4093-81fb-f68e70ab414e"
-					(reference "R30")
+					(reference "R33")
 					(unit 1)
 				)
@@
 		(on_board yes)
 		(dnp no)
-		(property "Reference" "J9"
+		(property "Reference" "J13"
 			(at 128.27 73.6599 0)
 			(effects
@@
 			(project "HalfBridge_SiC"
 				(path "/3c187ffa-7f66-4861-b077-b6965c821fc2/2168827a-beb7-4093-81fb-f68e70ab414e"
-					(reference "J9")
+					(reference "J13")
 					(unit 1)
 				)
@@
 		(dnp no)
 		(fields_autoplaced yes)
-		(property "Reference" "C41"
+		(property "Reference" "C43"
 			(at 105.41 45.72 90)
 			(effects
@@
 			(project "HalfBridge_SiC"
 				(path "/3c187ffa-7f66-4861-b077-b6965c821fc2/2168827a-beb7-4093-81fb-f68e70ab414e"
-					(reference "C41")
+					(reference "C43")
 					(unit 1)
 				)
@@
 		(dnp no)
 		(fields_autoplaced yes)
-		(property "Reference" "TP5"
+		(property "Reference" "TP8"
 			(at 71.12 58.9279 0)
 			(effects
@@
 			(project "HalfBridge_SiC"
 				(path "/3c187ffa-7f66-4861-b077-b6965c821fc2/2168827a-beb7-4093-81fb-f68e70ab414e"
-					(reference "TP5")
+					(reference "TP8")
 					(unit 1)
 				)
@@
 		(dnp no)
 		(fields_autoplaced yes)
-		(property "Reference" "R31"
+		(property "Reference" "R34"
 			(at 71.12 104.1399 0)
 			(effects
@@
 			(project "HalfBridge_SiC"
 				(path "/3c187ffa-7f66-4861-b077-b6965c821fc2/2168827a-beb7-4093-81fb-f68e70ab414e"
-					(reference "R31")
+					(reference "R34")
 					(unit 1)
 				)
@@
 		(on_board yes)
 		(dnp no)
-		(property "Reference" "J7"
+		(property "Reference" "J12"
 			(at 50.8 66.0399 0)
 			(effects
@@
 			(project "HalfBridge_SiC"
 				(path "/3c187ffa-7f66-4861-b077-b6965c821fc2/2168827a-beb7-4093-81fb-f68e70ab414e"
-					(reference "J7")
+					(reference "J12")
 					(unit 1)
 				)
@@
 		(dnp no)
 		(fields_autoplaced yes)
-		(property "Reference" "TP7"
+		(property "Reference" "TP10"
 			(at 71.12 97.0279 0)
 			(effects
@@
 			(project "HalfBridge_SiC"
 				(path "/3c187ffa-7f66-4861-b077-b6965c821fc2/2168827a-beb7-4093-81fb-f68e70ab414e"
-					(reference "TP7")
+					(reference "TP10")
 					(unit 1)
 				)
