File: pcb/HalfBridge_SiC/HalfBridge_InMeasurement.kicad_sch (KiCad schematic)
At the start: 8 parts

Commit message: local lib
Parts:
- R38, R39: symbol Device:R -> HalfBridge_SiC:R
- TP11, TP12, TP13, TP14, TP15, TP16: symbol Connector:TestPoint -> HalfBridge_SiC:TestPoint
Changed lines of the file:
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@@
 	)
 	(symbol
-		(lib_id "Connector:TestPoint")
+		(lib_id "HalfBridge_SiC:TestPoint")
 		(at 97.79 85.09 270)
 		(unit 1)
@@
 	)
 	(symbol
-		(lib_id "Connector:TestPoint")
+		(lib_id "HalfBridge_SiC:TestPoint")
 		(at 66.04 100.33 0)
 		(unit 1)
@@
 	)
 	(symbol
-		(lib_id "Connector:TestPoint")
+		(lib_id "HalfBridge_SiC:TestPoint")
 		(at 66.04 125.73 0)
 		(unit 1)
@@
 	)
 	(symbol
-		(lib_id "Connector:TestPoint")
+		(lib_id "HalfBridge_SiC:TestPoint")
 		(at 66.04 113.03 0)
 		(unit 1)
@@
 	)
 	(symbol
-		(lib_id "Connector:TestPoint")
+		(lib_id "HalfBridge_SiC:TestPoint")
 		(at 64.77 76.2 0)
 		(unit 1)
@@
 	)
 	(symbol
-		(lib_id "Device:R")
+		(lib_id "HalfBridge_SiC:R")
 		(at 90.17 85.09 90)
 		(unit 1)
@@
 	)
 	(symbol
-		(lib_id "Connector:TestPoint")
+		(lib_id "HalfBridge_SiC:TestPoint")
 		(at 82.55 85.09 90)
 		(unit 1)
@@
 	)
 	(symbol
-		(lib_id "Device:R")
+		(lib_id "HalfBridge_SiC:R")
 		(at 90.17 76.2 90)
 		(unit 1)

Commit message: pcb + newlib
Parts:
- added H1: MountingHole, MountingHole:MountingHole_2.2mm_M2_ISO14580, symbol Mechanical:MountingHole
- added TP17, TP18, TP19, TP20: TestPoint_Small, TestPoint:TestPoint_Keystone_5015_Micro-Minature, symbol Connector:TestPoint_Small
Connections:
- net dcm: now also TP18.1
- net dcn: now also TP19.1
- net dcp: now also TP17.1
- net ph: now also TP20.1
Other:
- company: (none) -> Dr.-Ing. Alan H. Wilson Veas

Commit message: backplane + external lib
Parts:
- added H2, H3, H4: MountingHole, MountingHole:MountingHole_2.7mm_M2.5, symbol Mechanical:MountingHole
- H1: footprint MountingHole:MountingHole_2.2mm_M2_ISO14580 -> MountingHole:MountingHole_2.7mm_M2.5
- R38, R39: footprint Resistor_SMD:R_4020_10251Metric_Pad1.65x5.30mm_HandSolder -> (none)
- TP11, TP12, TP13, TP14, TP15, TP16: footprint TestPoint:TestPoint_THTPad_D3.0mm_Drill1.5mm -> (none)
- TP17, TP18, TP19, TP20: footprint TestPoint:TestPoint_Keystone_5015_Micro-Minature -> (none)
Changed lines of the file:
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@@
 			)
 		)
-		(property "Footprint" "TestPoint:TestPoint_THTPad_D3.0mm_Drill1.5mm"
+		(property "Footprint" ""
 			(at 97.79 90.17 0)
 			(effects
@@
 			)
 		)
-		(property "Footprint" "TestPoint:TestPoint_THTPad_D3.0mm_Drill1.5mm"
+		(property "Footprint" ""
 			(at 71.12 100.33 0)
 			(effects
@@
 			)
 		)
-		(property "Footprint" "TestPoint:TestPoint_THTPad_D3.0mm_Drill1.5mm"
+		(property "Footprint" ""
 			(at 71.12 125.73 0)
 			(effects
@@
 			)
 		)
-		(property "Footprint" "TestPoint:TestPoint_THTPad_D3.0mm_Drill1.5mm"
+		(property "Footprint" ""
 			(at 71.12 113.03 0)
 			(effects
@@
 	)
 	(symbol
+		(lib_id "Mechanical:MountingHole")
+		(at 71.12 38.1 0)
+		(unit 1)
+		(exclude_from_sim yes)
+		(in_bom no)
+		(on_board yes)
+		(dnp no)
+		(fields_autoplaced yes)
+		(property "Reference" "H3"
+			(at 73.66 36.8299 0)
+			(effects
+				(font
+					(size 1.27 1.27)
+				)
+				(justify left)
+			)
+		)
+		(property "Value" "MountingHole"
+			(at 73.66 39.3699 0)
+			(effects
+				(font
+					(size 1.27 1.27)
+				)
+				(justify left)
+			)
+		)
+		(property "Footprint" "MountingHole:MountingHole_2.7mm_M2.5"
+			(at 71.12 38.1 0)
+			(effects
+				(font
+					(size 1.27 1.27)
+				)
+				(hide yes)
+			)
+		)
+		(property "Datasheet" "~"
+			(at 71.12 38.1 0)
+			(effects
+				(font
+					(size 1.27 1.27)
+				)
+				(hide yes)
+			)
+		)
+		(property "Description" "Mounting Hole without connection"
+			(at 71.12 38.1 0)
+			(effects
+				(font
+					(size 1.27 1.27)
+				)
+				(hide yes)
+			)
+		)
+		(instances
+			(project "HalfBridge_SiC"
+				(path "/3c187ffa-7f66-4861-b077-b6965c821fc2/c9be4e5e-b12a-4beb-8fd4-318e3bf3d480"
+					(reference "H3")
+					(unit 1)
+				)
+			)
+		)
+	)
+	(symbol
 		(lib_id "Connector:TestPoint_Small")
 		(at 64.77 86.36 0)
@@
 			)
 		)
-		(property "Footprint" "TestPoint:TestPoint_Keystone_5015_Micro-Minature"
+		(property "Footprint" ""
 			(at 69.85 86.36 0)
 			(effects
@@
 	)
 	(symbol
+		(lib_id "Mechanical:MountingHole")
+		(at 91.44 49.53 0)
+		(unit 1)
+		(exclude_from_sim yes)
+		(in_bom no)
+		(on_board yes)
+		(dnp no)
+		(fields_autoplaced yes)
+		(property "Reference" "H2"
+			(at 93.98 48.2599 0)
+			(effects
+				(font
+					(size 1.27 1.27)
+				)
+				(justify left)
+			)
+		)
+		(property "Value" "MountingHole"
+			(at 93.98 50.7999 0)
+			(effects
+				(font
+					(size 1.27 1.27)
+				)
+				(justify left)
+			)
+		)
+		(property "Footprint" "MountingHole:MountingHole_2.7mm_M2.5"
+			(at 91.44 49.53 0)
+			(effects
+				(font
+					(size 1.27 1.27)
+				)
+				(hide yes)
+			)
+		)
+		(property "Datasheet" "~"
+			(at 91.44 49.53 0)
+			(effects
+				(font
+					(size 1.27 1.27)
+				)
+				(hide yes)
+			)
+		)
+		(property "Description" "Mounting Hole without connection"
+			(at 91.44 49.53 0)
+			(effects
+				(font
+					(size 1.27 1.27)
+				)
+				(hide yes)
+			)
+		)
+		(instances
+			(project "HalfBridge_SiC"
+				(path "/3c187ffa-7f66-4861-b077-b6965c821fc2/c9be4e5e-b12a-4beb-8fd4-318e3bf3d480"
+					(reference "H2")
+					(unit 1)
+				)
+			)
+		)
+	)
+	(symbol
 		(lib_id "Connector:TestPoint_Small")
 		(at 80.01 113.03 0)
@@
 			)
 		)
-		(property "Footprint" "TestPoint:TestPoint_Keystone_5015_Micro-Minature"
+		(property "Footprint" ""
 			(at 85.09 113.03 0)
 			(effects
@@
 			)
 		)
-		(property "Footprint" "TestPoint:TestPoint_THTPad_D3.0mm_Drill1.5mm"
+		(property "Footprint" ""
 			(at 69.85 76.2 0)
 			(effects
@@
 	(symbol
 		(lib_id "Mechanical:MountingHole")
-		(at 67.31 46.99 0)
+		(at 91.44 38.1 0)
 		(unit 1)
 		(exclude_from_sim yes)
@@
 		(dnp no)
 		(fields_autoplaced yes)
-		(property "Reference" "H1"
-			(at 69.85 45.7199 0)
+		(property "Reference" "H4"
+			(at 93.98 36.8299 0)
 			(effects
 				(font
@@
 		)
 		(property "Value" "MountingHole"
-			(at 69.85 48.2599 0)
-			(effects
-				(font
-					(size 1.27 1.27)
-				)
-				(justify left)
-			)
-		)
-		(property "Footprint" "MountingHole:MountingHole_2.2mm_M2_ISO14580"
-			(at 67.31 46.99 0)
-			(effects
-				(font
-					(size 1.27 1.27)
-				)
-				(hide yes)
-			)
-		)
-		(property "Datasheet" "~"
-			(at 67.31 46.99 0)
+			(at 93.98 39.3699 0)
+			(effects
+				(font
+					(size 1.27 1.27)
+				)
+				(justify left)
+			)
+		)
+		(property "Footprint" "MountingHole:MountingHole_2.7mm_M2.5"
+			(at 91.44 38.1 0)
+			(effects
+				(font
+					(size 1.27 1.27)
+				)
+				(hide yes)
+			)
+		)
+		(property "Datasheet" "~"
+			(at 91.44 38.1 0)
 			(effects
 				(font
@@
 		)
 		(property "Description" "Mounting Hole without connection"
-			(at 67.31 46.99 0)
-			(effects
-				(font
-					(size 1.27 1.27)
-				)
-				(hide yes)
-			)
-		)
-		(instances
-			(project ""
-				(path "/3c187ffa-7f66-4861-b077-b6965c821fc2/c9be4e5e-b12a-4beb-8fd4-318e3bf3d480"
-					(reference "H1")
+			(at 91.44 38.1 0)
+			(effects
+				(font
+					(size 1.27 1.27)
+				)
+				(hide yes)
+			)
+		)
+		(instances
+			(project "HalfBridge_SiC"
+				(path "/3c187ffa-7f66-4861-b077-b6965c821fc2/c9be4e5e-b12a-4beb-8fd4-318e3bf3d480"
+					(reference "H4")
 					(unit 1)
 				)
@@
 			)
 		)
-		(property "Footprint" "TestPoint:TestPoint_Keystone_5015_Micro-Minature"
+		(property "Footprint" ""
 			(at 85.09 100.33 0)
 			(effects
@@
 	)
 	(symbol
+		(lib_id "Mechanical:MountingHole")
+		(at 71.12 49.53 0)
+		(unit 1)
+		(exclude_from_sim yes)
+		(in_bom no)
+		(on_board yes)
+		(dnp no)
+		(fields_autoplaced yes)
+		(property "Reference" "H1"
+			(at 73.66 48.2599 0)
+			(effects
+				(font
+					(size 1.27 1.27)
+				)
+				(justify left)
+			)
+		)
+		(property "Value" "MountingHole"
+			(at 73.66 50.7999 0)
+			(effects
+				(font
+					(size 1.27 1.27)
+				)
+				(justify left)
+			)
+		)
+		(property "Footprint" "MountingHole:MountingHole_2.7mm_M2.5"
+			(at 71.12 49.53 0)
+			(effects
+				(font
+					(size 1.27 1.27)
+				)
+				(hide yes)
+			)
+		)
+		(property "Datasheet" "~"
+			(at 71.12 49.53 0)
+			(effects
+				(font
+					(size 1.27 1.27)
+				)
+				(hide yes)
+			)
+		)
+		(property "Description" "Mounting Hole without connection"
+			(at 71.12 49.53 0)
+			(effects
+				(font
+					(size 1.27 1.27)
+				)
+				(hide yes)
+			)
+		)
+		(instances
+			(project ""
+				(path "/3c187ffa-7f66-4861-b077-b6965c821fc2/c9be4e5e-b12a-4beb-8fd4-318e3bf3d480"
+					(reference "H1")
+					(unit 1)
+				)
+			)
+		)
+	)
+	(symbol
 		(lib_id "HalfBridge_SiC:R")
 		(at 90.17 85.09 90)
@@
 			)
 		)
-		(property "Footprint" "Resistor_SMD:R_4020_10251Metric_Pad1.65x5.30mm_HandSolder"
+		(property "Footprint" ""
 			(at 90.17 86.868 90)
 			(effects
@@
 			)
 		)
-		(property "Footprint" "TestPoint:TestPoint_Keystone_5015_Micro-Minature"
+		(property "Footprint" ""
 			(at 85.09 125.73 0)
 			(effects
@@
 			)
 		)
-		(property "Footprint" "TestPoint:TestPoint_THTPad_D3.0mm_Drill1.5mm"
+		(property "Footprint" ""
 			(at 82.55 80.01 0)
 			(effects
@@
 			)
 		)
-		(property "Footprint" "Resistor_SMD:R_4020_10251Metric_Pad1.65x5.30mm_HandSolder"
+		(property "Footprint" ""
 			(at 90.17 77.978 90)
 			(effects

Commit message: update lib
Parts:
- added MS1, MS2, MS3, MS4: ~, symbol My_Standoff:Standoff_M_F
- R38, R39: footprint (none) -> Resistor_SMD:R_4020_10251Metric_Pad1.65x5.30mm_HandSolder
- TP11, TP12, TP13, TP16: footprint (none) -> TestPoint:TestPoint_THTPad_D2.0mm_Drill1.0mm
- TP14, TP15: footprint (none) -> TestPoint:TestPoint_Plated_Hole_D3.0mm
- TP17, TP18, TP19, TP20: footprint (none) -> TestPoint:TestPoint_Keystone_5015_Micro-Minature

Commit message: designator + part n°
Parts:
- renumbered H3 to H1, H1 to H2, H4 to H3, H2 to H4, R38 to R39, R39 to R40, TP16 to TP14, TP20 to TP15, TP11 to TP16, TP12 to TP17, TP13 to TP18, TP17 to TP19, TP18 to TP20, TP19 to TP21, TP14 to TP22, TP15 to TP23
Other:
- title: (none) -> Measurement placer
Changed lines of the file:
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@@
 	(paper "A4")
 	(title_block
+		(title "Measurement placer")
+		(date "2024-12-10")
 		(rev "1")
 		(company "Dr.-Ing. Alan H. Wilson Veas")
@@
 		(dnp no)
 		(fields_autoplaced yes)
-		(property "Reference" "TP15"
+		(property "Reference" "TP23"
 			(at 102.87 83.8199 90)
 			(effects
@@
 			(project "HalfBridge_SiC"
 				(path "/3c187ffa-7f66-4861-b077-b6965c821fc2/c9be4e5e-b12a-4beb-8fd4-318e3bf3d480"
-					(reference "TP15")
+					(reference "TP23")
 					(unit 1)
 				)
@@
 		(dnp no)
 		(fields_autoplaced yes)
-		(property "Reference" "TP11"
+		(property "Reference" "TP16"
 			(at 68.58 95.7579 0)
 			(effects
@@
 			(project "HalfBridge_SiC"
 				(path "/3c187ffa-7f66-4861-b077-b6965c821fc2/c9be4e5e-b12a-4beb-8fd4-318e3bf3d480"
-					(reference "TP11")
+					(reference "TP16")
 					(unit 1)
 				)
@@
 		(dnp no)
 		(fields_autoplaced yes)
-		(property "Reference" "TP13"
+		(property "Reference" "TP18"
 			(at 68.58 121.1579 0)
 			(effects
@@
 			(project "HalfBridge_SiC"
 				(path "/3c187ffa-7f66-4861-b077-b6965c821fc2/c9be4e5e-b12a-4beb-8fd4-318e3bf3d480"
-					(reference "TP13")
+					(reference "TP18")
 					(unit 1)
 				)
@@
 		(dnp no)
 		(fields_autoplaced yes)
-		(property "Reference" "TP12"
+		(property "Reference" "TP17"
 			(at 68.58 108.4579 0)
 			(effects
@@
 			(project "HalfBridge_SiC"
 				(path "/3c187ffa-7f66-4861-b077-b6965c821fc2/c9be4e5e-b12a-4beb-8fd4-318e3bf3d480"
-					(reference "TP12")
+					(reference "TP17")
 					(unit 1)
 				)
@@
 		(dnp no)
 		(fields_autoplaced yes)
-		(property "Reference" "H3"
+		(property "Reference" "H1"
 			(at 73.66 36.8299 0)
 			(effects
@@
 			(project "HalfBridge_SiC"
 				(path "/3c187ffa-7f66-4861-b077-b6965c821fc2/c9be4e5e-b12a-4beb-8fd4-318e3bf3d480"
-					(reference "H3")
+					(reference "H1")
 					(unit 1)
 				)
@@
 		(dnp no)
 		(fields_autoplaced yes)
-		(property "Reference" "TP20"
+		(property "Reference" "TP15"
 			(at 66.04 85.0899 0)
 			(effects
@@
 			(project "HalfBridge_SiC"
 				(path "/3c187ffa-7f66-4861-b077-b6965c821fc2/c9be4e5e-b12a-4beb-8fd4-318e3bf3d480"
-					(reference "TP20")
+					(reference "TP15")
 					(unit 1)
 				)
@@
 		(dnp no)
 		(fields_autoplaced yes)
-		(property "Reference" "H2"
+		(property "Reference" "H4"
 			(at 93.98 48.2599 0)
 			(effects
@@
 			(project "HalfBridge_SiC"
 				(path "/3c187ffa-7f66-4861-b077-b6965c821fc2/c9be4e5e-b12a-4beb-8fd4-318e3bf3d480"
-					(reference "H2")
+					(reference "H4")
 					(unit 1)
 				)
@@
 		(dnp no)
 		(fields_autoplaced yes)
-		(property "Reference" "TP18"
+		(property "Reference" "TP20"
 			(at 81.28 111.7599 0)
 			(effects
@@
 			(project "HalfBridge_SiC"
 				(path "/3c187ffa-7f66-4861-b077-b6965c821fc2/c9be4e5e-b12a-4beb-8fd4-318e3bf3d480"
-					(reference "TP18")
+					(reference "TP20")
 					(unit 1)
 				)
@@
 		(dnp no)
 		(fields_autoplaced yes)
-		(property "Reference" "TP16"
+		(property "Reference" "TP14"
 			(at 67.31 71.6279 0)
 			(effects
@@
 			(project "HalfBridge_SiC"
 				(path "/3c187ffa-7f66-4861-b077-b6965c821fc2/c9be4e5e-b12a-4beb-8fd4-318e3bf3d480"
-					(reference "TP16")
+					(reference "TP14")
 					(unit 1)
 				)
@@
 		(dnp no)
 		(fields_autoplaced yes)
-		(property "Reference" "H4"
+		(property "Reference" "H3"
 			(at 93.98 36.8299 0)
 			(effects
@@
 			(project "HalfBridge_SiC"
 				(path "/3c187ffa-7f66-4861-b077-b6965c821fc2/c9be4e5e-b12a-4beb-8fd4-318e3bf3d480"
-					(reference "H4")
+					(reference "H3")
 					(unit 1)
 				)
@@
 		(dnp no)
 		(fields_autoplaced yes)
-		(property "Reference" "TP17"
+		(property "Reference" "TP19"
 			(at 81.28 99.0599 0)
 			(effects
@@
 			(project "HalfBridge_SiC"
 				(path "/3c187ffa-7f66-4861-b077-b6965c821fc2/c9be4e5e-b12a-4beb-8fd4-318e3bf3d480"
-					(reference "TP17")
+					(reference "TP19")
 					(unit 1)
 				)
@@
 		(dnp no)
 		(fields_autoplaced yes)
-		(property "Reference" "H1"
+		(property "Reference" "H2"
 			(at 73.66 48.2599 0)
 			(effects
@@
 			(project ""
 				(path "/3c187ffa-7f66-4861-b077-b6965c821fc2/c9be4e5e-b12a-4beb-8fd4-318e3bf3d480"
-					(reference "H1")
+					(reference "H2")
 					(unit 1)
 				)
@@
 		(dnp no)
 		(fields_autoplaced yes)
-		(property "Reference" "R39"
+		(property "Reference" "R40"
 			(at 90.17 78.74 90)
 			(effects
@@
 			(project "HalfBridge_SiC"
 				(path "/3c187ffa-7f66-4861-b077-b6965c821fc2/c9be4e5e-b12a-4beb-8fd4-318e3bf3d480"
-					(reference "R39")
+					(reference "R40")
 					(unit 1)
 				)
@@
 		(dnp no)
 		(fields_autoplaced yes)
-		(property "Reference" "TP19"
+		(property "Reference" "TP21"
 			(at 81.28 124.4599 0)
 			(effects
@@
 			(project "HalfBridge_SiC"
 				(path "/3c187ffa-7f66-4861-b077-b6965c821fc2/c9be4e5e-b12a-4beb-8fd4-318e3bf3d480"
-					(reference "TP19")
+					(reference "TP21")
 					(unit 1)
 				)
@@
 		(dnp no)
 		(fields_autoplaced yes)
-		(property "Reference" "TP14"
+		(property "Reference" "TP22"
 			(at 79.248 80.01 90)
 			(effects
@@
 			(project "HalfBridge_SiC"
 				(path "/3c187ffa-7f66-4861-b077-b6965c821fc2/c9be4e5e-b12a-4beb-8fd4-318e3bf3d480"
-					(reference "TP14")
+					(reference "TP22")
 					(unit 1)
 				)
@@
 		(dnp no)
 		(fields_autoplaced yes)
-		(property "Reference" "R38"
+		(property "Reference" "R39"
 			(at 90.17 69.85 90)
 			(effects
@@
 			(project "HalfBridge_SiC"
 				(path "/3c187ffa-7f66-4861-b077-b6965c821fc2/c9be4e5e-b12a-4beb-8fd4-318e3bf3d480"
-					(reference "R38")
-					(unit 1)
-				)
+					(reference "R39")
+					(unit 1)
+				)

Commit message: titles
Parts:
- TP15, TP19, TP20, TP21: Part # (none) -> 5015
Changed lines of the file:
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@@
+			)
+		)
+		(property "Part #" "5015"
+			(at 64.77 86.36 0)
+			(effects
+				(font
+					(size 1.27 1.27)
+				)
+				(hide yes)
 			)
 		)
@@
 			)
 		)
+		(property "Part #" "5015"
+			(at 80.01 113.03 0)
+			(effects
+				(font
+					(size 1.27 1.27)
+				)
+				(hide yes)
+			)
+		)
 		(pin "1"
 		)
@@
 		)
 		(property "Description" "test point"
+			(at 80.01 100.33 0)
+			(effects
+				(font
+					(size 1.27 1.27)
+				)
+				(hide yes)
+			)
+		)
+		(property "Part #" "5015"
 			(at 80.01 100.33 0)
 			(effects
@@
 			(at 80.01 125.73 0)
 			(effects
+				(font
+					(size 1.27 1.27)
+				)
+				(hide yes)
+			)
+		)
+		(property "Part #" "5015"
+			(at 80.01 125.73 0)
+			(effects
