File: pcb/Backplane_DC/Backplane_DC.kicad_pcb (KiCad board)
At the start: 2 copper layers, 100 x 100 mm, 4 parts, among them J1 413638-E, J2 413638-E

Commit message: backplane + external lib
Parts:
- removed J2: 413638-E, My_Connector:TE_594750-E
- added D1: DNA40U2200GU, Diode_THT:Diode_Bridge_IXYS_GUFP, B.Cu at (116.8, 82.0)
- added H1: MountingHole_Pad, MountingHole:MountingHole_4.3mm_M4_DIN965_Pad, B.Cu at (100.8, 55.4)
- added H2: MountingHole_Pad, MountingHole:MountingHole_4.3mm_M4_DIN965_Pad, B.Cu at (50.0, 55.2)
- added H3: MountingHole_Pad, MountingHole:MountingHole_4.3mm_M4_DIN965_Pad, B.Cu at (50.0, 75.6)
- added H4: MountingHole_Pad, MountingHole:MountingHole_4.3mm_M4_DIN965_Pad, B.Cu at (100.8, 75.7)
- added H5: MountingHole_Pad, MountingHole:MountingHole_4.3mm_M4_DIN965_Pad, B.Cu at (50.0, 95.9)
- added H6: MountingHole_Pad, MountingHole:MountingHole_4.3mm_M4_DIN965_Pad, B.Cu at (100.8, 96.0)
- added H7: MountingHole_Pad, MountingHole:MountingHole_4.3mm_M4_DIN965_Pad, B.Cu at (50.0, 116.2)
- added H8: MountingHole_Pad, MountingHole:MountingHole_4.3mm_M4_DIN965_Pad, B.Cu at (100.8, 116.3)
- J1: value 413638-E -> Conn_01x03; footprint My_Connector:TE_594750-E -> Connector_Phoenix_SPT:PhoenixContact_SPT_5_3-H-7.5-ZB_1x03_P7.5mm_Horizontal
- moved J1 76.5 mm to (123.2, 104.6), turned to 90 degrees
- moved C1 4.27 mm to (75.2, 73.6)
- moved C2 3.56 mm to (75.2, 114.3)
Connections:
- C1 pad 1: unconnected-(C1-Pad1) -> /dcp
- C1 pad 2: unconnected-(C1-Pad2) -> /dcm
- C2 pad 1: unconnected-(C2-Pad1) -> /dcm
- C2 pad 2: unconnected-(C2-Pad2) -> /dcn

Commit message: backplane
Parts:
- removed J1: Conn_01x03, Connector_Phoenix_SPT:PhoenixContact_SPT_5_3-H-7.5-ZB_1x03_P7.5mm_Horizontal
- added J2: Conn_01x05, Connector_Phoenix_SPT:PhoenixContact_SPT_5_5-H-7.5-ZB_1x05_P7.5mm_Horizontal, F.Cu at (124.0, 116.5)
- moved D1 4.43 mm to (117.3, 86.4)
Connections:
- D1 pad 2: unconnected-(D1-Pad2) -> /l1
- D1 pad 3: unconnected-(D1-Pad3) -> /l2
- D1 pad 4: unconnected-(D1-Pad4) -> /l3
Routing:
- added copper zone on B.Cu, net /dcm
- added copper zone on F.Cu, net /dcn
- added copper zone on F.Cu, net /dcp

Commit message: update lib
Parts:
- added R1: 100k, Resistor_THT:R_Axial_DIN0411_L9.9mm_D3.6mm_P25.40mm_Horizontal, B.Cu at (107.7, 71.1)
- added R2: 100k, Resistor_THT:R_Axial_DIN0411_L9.9mm_D3.6mm_P25.40mm_Horizontal, B.Cu at (107.7, 99.6)
- C1, C2: footprint Capacitor_THT:CP_Radial_D40.0mm_P10.00mm_SnapIn -> My_Capacitor_THT:CP_Radial_D40.0mm_P22.50mm_SnapIn_4Pin_ALF80
- moved C1 6.90 mm to (75.7, 66.8)
- moved C2 6.32 mm to (75.7, 108.0)
Routing:
- net /l3: track 0.00 -> 19.9 mm
- net /l1: track 0.00 -> 19.9 mm
- net /l2: track 0.00 -> 6.70 mm

Commit message: filter + sim + assembly3d
Parts:
- removed C1, C2: C_Polarized, My_Capacitor_THT:CP_Radial_D40.0mm_P22.50mm_SnapIn_4Pin_ALF80
- removed D1: DNA40U2200GU, Diode_THT:Diode_Bridge_IXYS_GUFP
- removed J2: Conn_01x05, Connector_Phoenix_SPT:PhoenixContact_SPT_5_5-H-7.5-ZB_1x05_P7.5mm_Horizontal
- removed R1, R2: 100k, Resistor_THT:R_Axial_DIN0411_L9.9mm_D3.6mm_P25.40mm_Horizontal
- added H10: MountingHole_Pad, MountingHole:MountingHole_4.3mm_M4_DIN965_Pad, B.Cu at (128.0, 45.1)
- added H11: MountingHole_Pad, MountingHole:MountingHole_4.3mm_M4_DIN965_Pad, B.Cu at (44.2, 75.6)
- added H12: MountingHole_Pad, MountingHole:MountingHole_4.3mm_M4_DIN965_Pad, B.Cu at (44.2, 95.9)
- added H13: MountingHole_Pad, MountingHole:MountingHole_4.3mm_M4_DIN965_Pad, B.Cu at (44.2, 116.2)
- added H9: MountingHole_Pad, MountingHole:MountingHole_4.3mm_M4_DIN965_Pad, B.Cu at (67.1, 45.1)
- added J1: Conn_01x02, Connector_Phoenix_SPT:PhoenixContact_SPT_1.5_2-H-3.5_1x02_P3.5mm_Horizontal, F.Cu at (128.2, 138.1)
- added U1: IRM-05-5, My_Converter_ACDC:IRM-05-5, F.Cu at (101.8, 125.3)
- moved H1 34.9 mm to (135.7, 55.2)
- moved H4 34.9 mm to (135.7, 75.6)
- moved H6 34.9 mm to (135.7, 95.9)
- moved H8 34.9 mm to (135.7, 116.2)
- moved H2 24.7 mm to (74.7, 55.2)
- moved H3 24.7 mm to (74.7, 75.6)
- moved H5 24.7 mm to (74.7, 95.9)
- moved H7 24.7 mm to (74.7, 116.2)
Routing:
- net /dcm: track 0.00 -> 60.1 mm
- net /l3: track 19.9 -> 0.00 mm
- net /l1: track 19.9 -> 0.00 mm
- net /5v: track 0.00 -> 18.0 mm
- net /gnd: track 0.00 -> 16.1 mm
- net /dcn: track 0.00 -> 12.5 mm
- net /l2: track 6.70 -> 0.00 mm
- added copper zone on B.Cu, net /pha
- added copper zone on F.Cu, net /pha
- added copper zone on B.Cu, net /phb
- added copper zone on F.Cu, net /phb

Commit message: filter + backplane
Parts:
- moved H10 2.54 mm to (128.0, 47.6)
- moved H9 2.54 mm to (67.1, 47.6)
- moved J1 0.14 mm to (128.1, 138.0)
Changed lines of the file:
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@@
 	(footprint "Connector_Phoenix_SPT:PhoenixContact_SPT_1.5_2-H-3.5_1x02_P3.5mm_Horizontal"
 		(layer "F.Cu")
-		(at 128.2 138.1 90)
+		(at 128.1 138 90)
 		(descr "Connector Phoenix Contact, SPT 1.5/2-H-3.5 Terminal Block, 1990737 (https://www.phoenixcontact.com/online/portal/gb/?uri=pxc-oc-itemdetail:pid=1990737), generated with kicad-footprint-generator")
 		(tags "Connector Phoenix Contact SPT 1.5/2-H-3.5 1990737")
@@
 	(footprint "MountingHole:MountingHole_4.3mm_M4_DIN965_Pad"
 		(layer "B.Cu")
-		(at 128.037999 45.079999 180)
+		(at 128.037999 47.619999 180)
 		(descr "Mounting Hole 4.3mm, M4, DIN965")
 		(tags "mounting hole 4.3mm m4 din965")
@@
 	(footprint "MountingHole:MountingHole_4.3mm_M4_DIN965_Pad"
 		(layer "B.Cu")
-		(at 67.077999 45.079999 180)
+		(at 67.077999 47.619999 180)
 		(descr "Mounting Hole 4.3mm, M4, DIN965")
 		(tags "mounting hole 4.3mm m4 din965")
@@
 		(layer "Dwgs.User")
 		(pts
-			(xy 80 55.239999) (xy 116.119999 45.079999)
-		)
-		(height -42)
+			(xy 74.697999 55.239999) (xy 128.037999 47.619999)
+		)
+		(height -37.997999)
 		(orientation 1)
-		(gr_text "400.0000 mils"
-			(at 36.85 50.159999 90)
+		(gr_text "300.0000 mils"
+			(at 35.55 51.429999 90)
 			(layer "Dwgs.User")
 			(effects

Commit message: titles
Parts:
- added H14: MountingHole, MountingHole:MountingHole_2.7mm_M2.5, F.Cu at (44.0, 136.0)
- added H15: MountingHole, MountingHole:MountingHole_2.7mm_M2.5, F.Cu at (44.0, 44.0)
- added H16: MountingHole, MountingHole:MountingHole_2.7mm_M2.5, F.Cu at (136.0, 126.0)
- added H17: MountingHole, MountingHole:MountingHole_2.7mm_M2.5, F.Cu at (136.0, 65.0)
Other:
- board text added: "${TITLE} ./pcb/${PROJECTNAME} ${COMPANY} Issued: ${ISSUE_DATE} Rev: ${REVISION} ${COMMENT1}"
- board text added: "Rev: ${REVISION} ${COMMENT1}"
