File: pcb/Backplane_DC/Backplane_DC.kicad_sch (KiCad schematic)
At the start: 4 parts, among them J1 413638-E, J2 413638-E

Commit message: backplane + external lib
Parts:
- removed J1, J2: 413638-E, My_Connector:TE_594750-E, symbol My_Connector:594750-E
- added D1: DNA40U2200GU, Diode_THT:Diode_Bridge_IXYS_GUFP, symbol Diode_Bridge:DNA40U2200GU
- added H1, H2, H3, H4, H5, H6, H7, H8: MountingHole_Pad, MountingHole:MountingHole_4.3mm_M4_DIN965_Pad, symbol Mechanical:MountingHole_Pad
- added J1: Conn_01x03, Connector_Phoenix_SPT:PhoenixContact_SPT_5_3-H-7.5-ZB_1x03_P7.5mm_Horizontal, symbol Connector_Generic:Conn_01x03
Connections:
- net dcp: now reaches C1.1
- net dcp: now also D1.1 (+), H3.1, H4.1
- net dcm: now reaches C1.2
- net dcm: now also C2.1, H5.1, H6.1
- net dcn: now reaches C2.2
- net dcn: now also D1.5 (-), H7.1, H8.1
- new net pha: H2.1
- new net phb: H1.1
Other:
- moved on the sheet: C1, C2

Commit message: backplane
Parts:
- removed J1: Conn_01x03, Connector_Phoenix_SPT:PhoenixContact_SPT_5_3-H-7.5-ZB_1x03_P7.5mm_Horizontal, symbol Connector_Generic:Conn_01x03
- added J2: Conn_01x05, Connector_Phoenix_SPT:PhoenixContact_SPT_5_5-H-7.5-ZB_1x05_P7.5mm_Horizontal, symbol Connector_Generic:Conn_01x05
Connections:
- net dcn: now also J2.1 (Pin_1)
- net dcp: now also J2.5 (Pin_5)
- net l1: now reaches D1.2
- net l1: now also J2.4 (Pin_4)
- net l2: now reaches D1.3
- net l2: now also J2.3 (Pin_3)
- net l3: now reaches D1.4
- net l3: now also J2.2 (Pin_2)
Other:
- moved on the sheet: C1, C2, D1
Changed lines of the file:
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@@
 	(wire
 		(pts
-			(xy 148.59 119.38) (xy 148.59 121.92)
+			(xy 124.46 90.17) (xy 124.46 92.71)
 		)
 		(stroke
@@
 		)
 	)
+	(label "l1"
+		(at 82.55 88.9 180)
+		(fields_autoplaced yes)
+		(effects
+			(font
+				(size 1.27 1.27)
+			)
+			(justify right bottom)
+		)
+	)
+	(label "dcn"
+		(at 58.42 86.36 0)
+		(fields_autoplaced yes)
+		(effects
+			(font
+				(size 1.27 1.27)
+			)
+			(justify left bottom)
+		)
+	)
 	(label "dcp"
-		(at 124.46 110.49 0)
-		(fields_autoplaced yes)
-		(effects
-			(font
-				(size 1.27 1.27)
-			)
-			(justify left bottom)
+		(at 100.33 81.28 0)
+		(fields_autoplaced yes)
+		(effects
+			(font
+				(size 1.27 1.27)
+			)
+			(justify left bottom)
+		)
+	)
+	(label "l3"
+		(at 82.55 93.98 180)
+		(fields_autoplaced yes)
+		(effects
+			(font
+				(size 1.27 1.27)
+			)
+			(justify right bottom)
 		)
 	)
@@
 		)
 	)
+	(label "dcp"
+		(at 58.42 96.52 0)
+		(fields_autoplaced yes)
+		(effects
+			(font
+				(size 1.27 1.27)
+			)
+			(justify left bottom)
+		)
+	)
 	(label "pha"
 		(at 67.31 44.45 0)
@@
 		)
 	)
+	(label "l1"
+		(at 58.42 93.98 0)
+		(fields_autoplaced yes)
+		(effects
+			(font
+				(size 1.27 1.27)
+			)
+			(justify left bottom)
+		)
+	)
+	(label "l2"
+		(at 82.55 91.44 180)
+		(fields_autoplaced yes)
+		(effects
+			(font
+				(size 1.27 1.27)
+			)
+			(justify right bottom)
+		)
+	)
+	(label "l2"
+		(at 58.42 91.44 0)
+		(fields_autoplaced yes)
+		(effects
+			(font
+				(size 1.27 1.27)
+			)
+			(justify left bottom)
+		)
+	)
 	(label "dcn"
-		(at 124.46 130.81 0)
+		(at 100.33 101.6 0)
+		(fields_autoplaced yes)
+		(effects
+			(font
+				(size 1.27 1.27)
+			)
+			(justify left bottom)
+		)
+	)
+	(label "l3"
+		(at 58.42 88.9 0)
 		(fields_autoplaced yes)
 		(effects
@@
 	)
 	(label "dcm"
-		(at 148.59 120.65 0)
+		(at 124.46 91.44 0)
 		(fields_autoplaced yes)
 		(effects
@@
 	)
 	(label "dcn"
-		(at 148.59 129.54 0)
+		(at 124.46 100.33 0)
 		(fields_autoplaced yes)
 		(effects
@@
 	)
 	(label "dcp"
-		(at 148.59 111.76 0)
+		(at 124.46 82.55 0)
 		(fields_autoplaced yes)
 		(effects
@@
 	)
 	(symbol
-		(lib_id "Connector_Generic:Conn_01x03")
-		(at 60.96 116.84 0)
+		(lib_id "Connector_Generic:Conn_01x05")
+		(at 53.34 91.44 0)
 		(mirror y)
 		(unit 1)
@@
 		(on_board yes)
 		(dnp no)
-		(property "Reference" "J1"
-			(at 58.42 115.5699 0)
-			(effects
-				(font
-					(size 1.27 1.27)
-				)
-				(justify left)
-			)
-		)
-		(property "Value" "Conn_01x03"
-			(at 58.42 118.1099 0)
-			(effects
-				(font
-					(size 1.27 1.27)
-				)
-				(justify left)
-			)
-		)
-		(property "Footprint" "Connector_Phoenix_SPT:PhoenixContact_SPT_5_3-H-7.5-ZB_1x03_P7.5mm_Horizontal"
-			(at 60.96 116.84 0)
+		(property "Reference" "J2"
+			(at 50.8 90.1699 0)
+			(effects
+				(font
+					(size 1.27 1.27)
+				)
+				(justify left)
+			)
+		)
+		(property "Value" "Conn_01x05"
+			(at 50.8 92.7099 0)
+			(effects
+				(font
+					(size 1.27 1.27)
+				)
+				(justify left)
+			)
+		)
+		(property "Footprint" "Connector_Phoenix_SPT:PhoenixContact_SPT_5_5-H-7.5-ZB_1x05_P7.5mm_Horizontal"
+			(at 53.34 91.44 0)
 			(effects
 				(font
@@
 		)
 		(property "Datasheet" "~"
-			(at 60.96 116.84 0)
-			(effects
-				(font
-					(size 1.27 1.27)
-				)
-				(hide yes)
-			)
-		)
-		(property "Description" "Generic connector, single row, 01x03, script generated (kicad-library-utils/schlib/autogen/connector/)"
-			(at 60.96 116.84 0)
-			(effects
-				(font
-					(size 1.27 1.27)
-				)
-				(hide yes)
-			)
+			(at 53.34 91.44 0)
+			(effects
+				(font
+					(size 1.27 1.27)
+				)
+				(hide yes)
+			)
+		)
+		(property "Description" "Generic connector, single row, 01x05, script generated (kicad-library-utils/schlib/autogen/connector/)"
+			(at 53.34 91.44 0)
+			(effects
+				(font
+					(size 1.27 1.27)
+				)
+				(hide yes)
+			)
+		)
+		(pin "1"
 		)
 		(pin "2"
 		)
-		(pin "1"
+		(pin "4"
 		)
 		(pin "3"
+		)
+		(pin "5"
 		)
 		(instances
 			(project ""
 				(path "/1d08233b-efae-4958-9b81-9924f8f7b590"
-					(reference "J1")
+					(reference "J2")
 					(unit 1)
 				)
@@
 	(symbol
 		(lib_id "Diode_Bridge:DNA40U2200GU")
-		(at 116.84 120.65 0)
+		(at 92.71 91.44 0)
 		(unit 1)
 		(exclude_from_sim no)
@@
 		(fields_autoplaced yes)
 		(property "Reference" "D1"
-			(at 116.2685 105.41 0)
+			(at 92.1385 76.2 0)
 			(effects
 				(font
@@
 		)
 		(property "Value" "DNA40U2200GU"
-			(at 116.2685 107.95 0)
+			(at 92.1385 78.74 0)
 			(effects
 				(font
@@
 		)
 		(property "Footprint" "Diode_THT:Diode_Bridge_IXYS_GUFP"
-			(at 116.84 135.89 0)
+			(at 92.71 106.68 0)
 			(effects
 				(font
@@
 		)
 		(property "Datasheet" "https://ixapps.ixys.com/Datasheet/DNA40U2200GU.pdf"
-			(at 116.84 102.87 0)
+			(at 92.71 73.66 0)
 			(effects
 				(font
@@
 		)
 		(property "Description" "690V Vrms, 40A If, GUFP(X025B)"
-			(at 116.84 120.65 0)
+			(at 92.71 91.44 0)
 			(effects
 				(font
@@
 	(symbol
 		(lib_id "Device:C_Polarized")
-		(at 148.59 115.57 0)
+		(at 124.46 86.36 0)
 		(unit 1)
 		(exclude_from_sim no)
@@
 		(fields_autoplaced yes)
 		(property "Reference" "C1"
-			(at 152.4 113.4109 0)
+			(at 128.27 84.2009 0)
 			(effects
 				(font
@@
 		)
 		(property "Value" "C_Polarized"
-			(at 152.4 115.9509 0)
+			(at 128.27 86.7409 0)
 			(effects
 				(font
@@
 		)
 		(property "Footprint" "Capacitor_THT:CP_Radial_D40.0mm_P10.00mm_SnapIn"
-			(at 149.5552 119.38 0)
+			(at 125.4252 90.17 0)
 			(effects
 				(font
@@
 		)
 		(property "Datasheet" "~"
-			(at 148.59 115.57 0)
+			(at 124.46 86.36 0)
 			(effects
 				(font
@@
 		)
 		(property "Description" "Polarized capacitor"
-			(at 148.59 115.57 0)
+			(at 124.46 86.36 0)
 			(effects
 				(font
@@
 	(symbol
 		(lib_id "Device:C_Polarized")
-		(at 148.59 125.73 0)
+		(at 124.46 96.52 0)
 		(unit 1)
 		(exclude_from_sim no)
@@
 		(fields_autoplaced yes)
 		(property "Reference" "C2"
-			(at 152.4 123.5709 0)
+			(at 128.27 94.3609 0)
 			(effects
 				(font
@@
 		)
 		(property "Value" "C_Polarized"
-			(at 152.4 126.1109 0)
+			(at 128.27 96.9009 0)
 			(effects
 				(font
@@
 		)
 		(property "Footprint" "Capacitor_THT:CP_Radial_D40.0mm_P10.00mm_SnapIn"
-			(at 149.5552 129.54 0)
+			(at 125.4252 100.33 0)
 			(effects
 				(font
@@
 		)
 		(property "Datasheet" "~"
-			(at 148.59 125.73 0)
+			(at 124.46 96.52 0)
 			(effects
 				(font
@@
 		)
 		(property "Description" "Polarized capacitor"
-			(at 148.59 125.73 0)
-			(effects
-				(font
+			(at 124.46 96.52 0)
+			(effects
+				(font

Commit message: update lib
Parts:
- added R1, R2: 100k, Resistor_THT:R_Axial_DIN0411_L9.9mm_D3.6mm_P25.40mm_Horizontal, symbol HalfBridge_SiC:R
- C1, C2: footprint Capacitor_THT:CP_Radial_D40.0mm_P10.00mm_SnapIn -> My_Capacitor_THT:CP_Radial_D40.0mm_P22.50mm_SnapIn_4Pin_ALF80
Connections:
- net dcm: now also R1.2, R2.1
- net dcn: now also R2.2
- net dcp: now also R1.1
Changed lines of the file:
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@@
 	(generator_version "8.0")
 	(paper "A4")
+	(junction
+		(at 144.78 90.17)
+		(diameter 0)
+		(color 0 0 0 0)
+	)
+	(wire
+		(pts
+			(xy 144.78 90.17) (xy 144.78 91.44)
+		)
+		(stroke
+			(width 0)
+			(type default)
+		)
+	)
 	(wire
 		(pts
@@
 		)
 	)
+	(wire
+		(pts
+			(xy 144.78 100.33) (xy 146.05 100.33)
+		)
+		(stroke
+			(width 0)
+			(type default)
+		)
+	)
+	(wire
+		(pts
+			(xy 144.78 90.17) (xy 146.05 90.17)
+		)
+		(stroke
+			(width 0)
+			(type default)
+		)
+	)
+	(wire
+		(pts
+			(xy 144.78 99.06) (xy 144.78 100.33)
+		)
+		(stroke
+			(width 0)
+			(type default)
+		)
+	)
 	(label "l1"
 		(at 82.55 88.9 180)
@@
 	)
 	(label "dcn"
+		(at 146.05 100.33 0)
+		(fields_autoplaced yes)
+		(effects
+			(font
+				(size 1.27 1.27)
+			)
+			(justify left bottom)
+		)
+	)
+	(label "dcn"
 		(at 58.42 86.36 0)
 		(fields_autoplaced yes)
@@
 		)
 	)
+	(label "dcp"
+		(at 144.78 82.55 0)
+		(fields_autoplaced yes)
+		(effects
+			(font
+				(size 1.27 1.27)
+			)
+			(justify left bottom)
+		)
+	)
 	(label "l1"
 		(at 58.42 93.98 0)
@@
 	(label "dcn"
 		(at 92.71 67.31 0)
+		(fields_autoplaced yes)
+		(effects
+			(font
+				(size 1.27 1.27)
+			)
+			(justify left bottom)
+		)
+	)
+	(label "dcm"
+		(at 146.05 90.17 0)
 		(fields_autoplaced yes)
 		(effects
@@
 	)
 	(symbol
+		(lib_id "HalfBridge_SiC:R")
+		(at 144.78 95.25 0)
+		(unit 1)
+		(exclude_from_sim no)
+		(in_bom yes)
+		(on_board yes)
+		(dnp no)
+		(fields_autoplaced yes)
+		(property "Reference" "R2"
+			(at 147.32 93.9799 0)
+			(effects
+				(font
+					(size 1.27 1.27)
+				)
+				(justify left)
+			)
+		)
+		(property "Value" "100k"
+			(at 147.32 96.5199 0)
+			(effects
+				(font
+					(size 1.27 1.27)
+				)
+				(justify left)
+			)
+		)
+		(property "Footprint" "Resistor_THT:R_Axial_DIN0411_L9.9mm_D3.6mm_P25.40mm_Horizontal"
+			(at 143.002 95.25 90)
+			(effects
+				(font
+					(size 1.27 1.27)
+				)
+				(hide yes)
+			)
+		)
+		(property "Datasheet" "~"
+			(at 144.78 95.25 0)
+			(effects
+				(font
+					(size 1.27 1.27)
+				)
+				(hide yes)
+			)
+		)
+		(property "Description" "Resistor"
+			(at 144.78 95.25 0)
+			(effects
+				(font
+					(size 1.27 1.27)
+				)
+				(hide yes)
+			)
+		)
+		(pin "2"
+		)
+		(pin "1"
+		)
+		(instances
+			(project "Backplane_DC"
+				(path "/1d08233b-efae-4958-9b81-9924f8f7b590"
+					(reference "R2")
+					(unit 1)
+				)
+			)
+		)
+	)
+	(symbol
 		(lib_id "Mechanical:MountingHole_Pad")
 		(at 67.31 64.77 0)
@@
 	)
 	(symbol
+		(lib_id "HalfBridge_SiC:R")
+		(at 144.78 86.36 0)
+		(unit 1)
+		(exclude_from_sim no)
+		(in_bom yes)
+		(on_board yes)
+		(dnp no)
+		(fields_autoplaced yes)
+		(property "Reference" "R1"
+			(at 147.32 85.0899 0)
+			(effects
+				(font
+					(size 1.27 1.27)
+				)
+				(justify left)
+			)
+		)
+		(property "Value" "100k"
+			(at 147.32 87.6299 0)
+			(effects
+				(font
+					(size 1.27 1.27)
+				)
+				(justify left)
+			)
+		)
+		(property "Footprint" "Resistor_THT:R_Axial_DIN0411_L9.9mm_D3.6mm_P25.40mm_Horizontal"
+			(at 143.002 86.36 90)
+			(effects
+				(font
+					(size 1.27 1.27)
+				)
+				(hide yes)
+			)
+		)
+		(property "Datasheet" "~"
+			(at 144.78 86.36 0)
+			(effects
+				(font
+					(size 1.27 1.27)
+				)
+				(hide yes)
+			)
+		)
+		(property "Description" "Resistor"
+			(at 144.78 86.36 0)
+			(effects
+				(font
+					(size 1.27 1.27)
+				)
+				(hide yes)
+			)
+		)
+		(pin "2"
+		)
+		(pin "1"
+		)
+		(instances
+			(project "Backplane_DC"
+				(path "/1d08233b-efae-4958-9b81-9924f8f7b590"
+					(reference "R1")
+					(unit 1)
+				)
+			)
+		)
+	)
+	(symbol
 		(lib_id "Mechanical:MountingHole_Pad")
 		(at 92.71 49.53 0)
@@
 			)
 		)
-		(property "Footprint" "Capacitor_THT:CP_Radial_D40.0mm_P10.00mm_SnapIn"
+		(property "Footprint" "My_Capacitor_THT:CP_Radial_D40.0mm_P22.50mm_SnapIn_4Pin_ALF80"
 			(at 125.4252 90.17 0)
 			(effects
@@
 			)
 		)
-		(property "Footprint" "Capacitor_THT:CP_Radial_D40.0mm_P10.00mm_SnapIn"
+		(property "Footprint" "My_Capacitor_THT:CP_Radial_D40.0mm_P22.50mm_SnapIn_4Pin_ALF80"
 			(at 125.4252 100.33 0)
 			(effects

Commit message: filter + sim + assembly3d
Parts:
- removed C1, C2: C_Polarized, My_Capacitor_THT:CP_Radial_D40.0mm_P22.50mm_SnapIn_4Pin_ALF80, symbol Device:C_Polarized
- removed D1: DNA40U2200GU, Diode_THT:Diode_Bridge_IXYS_GUFP, symbol Diode_Bridge:DNA40U2200GU
- removed J2: Conn_01x05, Connector_Phoenix_SPT:PhoenixContact_SPT_5_5-H-7.5-ZB_1x05_P7.5mm_Horizontal, symbol Connector_Generic:Conn_01x05
- removed R1, R2: 100k, Resistor_THT:R_Axial_DIN0411_L9.9mm_D3.6mm_P25.40mm_Horizontal, symbol HalfBridge_SiC:R
- added H10, H11, H12, H13, H9: MountingHole_Pad, MountingHole:MountingHole_4.3mm_M4_DIN965_Pad, symbol Mechanical:MountingHole_Pad
- added J1: Conn_01x02, Connector_Phoenix_SPT:PhoenixContact_SPT_1.5_2-H-3.5_1x02_P3.5mm_Horizontal, symbol Connector_Generic:Conn_01x02
- added U1: IRM-05-5, My_Converter_ACDC:IRM-05-5, symbol My_Converter_ACDC:IRM-05-5
Connections:
- net dcm: now also H12.1, U1.2 (AC/L)
- net dcn: now also H13.1, U1.1 (AC/N)
- net dcp: now also H11.1
- net pha: now also H9.1
- net phb: now also H10.1
- new net 5v: J1.2 (Pin_2), U1.5 (+Vo)
- new net gnd: J1.1 (Pin_1), U1.4 (-Vo)

Commit message: designator + part n°
Changed lines of the file:
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@@
+		)
+	)
+	(text_box "AC/DC-DC converter to 5V"
+		(exclude_from_sim no)
+		(at 127 24.638 0)
+		(size 30.988 8.636)
+		(stroke
+			(width 0)
+			(type default)
+		)
+		(fill
+			(type none)
+		)
+		(effects
+			(font
+				(size 1.27 1.27)
+			)
+			(justify left top)
 		)
 	)

Commit message: titles
Parts:
- added H14, H15, H16, H17: MountingHole, MountingHole:MountingHole_2.7mm_M2.5, symbol Mechanical:MountingHole
Other:
- company: (none) -> Dr.-Ing. Alan H. Wilson Veas
- title: (none) -> Backplane DC-link
