File: pcb/Filter/Filter.kicad_sch (KiCad schematic)
At the start: 8 parts, among them J1 Conn_01x01, J2 Conn_01x01, J3 Conn_01x02

Commit message: titles
Parts:
- added H1, H2, H3, H4: MountingHole, MountingHole:MountingHole_2.7mm_M2.5, symbol Mechanical:MountingHole
Other:
- company: (none) -> Dr.-Ing. Alan H. Wilson V
- title: (none) -> Output LC filter
