File: pcb/Rectifier/Rectifier.kicad_pcb (KiCad board)
At the start: 2 copper layers, 100 x 100 mm, 11 parts, among them J2 Conn_01x01, J3 Conn_01x01, J4 Conn_01x01, J5 Conn_01x06

Commit message: titles
Parts:
- added H1: MountingHole, MountingHole:MountingHole_2.7mm_M2.5, F.Cu at (57.7, 33.2)
- added H2: MountingHole, MountingHole:MountingHole_2.7mm_M2.5, F.Cu at (149.7, 33.2)
- added H3: MountingHole, MountingHole:MountingHole_2.7mm_M2.5, F.Cu at (57.7, 125.2)
- added H4: MountingHole, MountingHole:MountingHole_2.7mm_M2.5, F.Cu at (149.7, 125.2)
- C1, C2, C3, C4: value C_Polarized -> 1200 uF
Other:
- board text added: "${TITLE} ./pcb/${PROJECTNAME} ${COMPANY} Issued: ${ISSUE_DATE} Rev: ${REVISION} ${COMMENT1}"
- board text added: "H"
- board text added: "Rev: ${REVISION} ${COMMENT1}"
