File: pcb/Rectifier/Rectifier.kicad_sch (KiCad schematic)
At the start: 11 parts, among them J2 Conn_01x01, J3 Conn_01x01, J4 Conn_01x01, J5 Conn_01x06

Commit message: designator + part n°
Parts:
- C1, C2, C3, C4: value C_Polarized -> 1200 uF; Part # (none) -> MAL229956122E3
Changed lines of the file:
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@@
 			)
 		)
-		(property "Value" "C_Polarized"
+		(property "Value" "1200 uF"
 			(at 149.86 95.6309 0)
 			(effects
@@
 		)
 		(property "Description" "Polarized capacitor"
+			(at 146.05 95.25 0)
+			(effects
+				(font
+					(size 1.27 1.27)
+				)
+				(hide yes)
+			)
+		)
+		(property "Part #" "MAL229956122E3"
 			(at 146.05 95.25 0)
 			(effects
@@
 			)
 		)
-		(property "Value" "C_Polarized"
+		(property "Value" "1200 uF"
 			(at 149.86 105.7909 0)
 			(effects
@@
 		)
 		(property "Description" "Polarized capacitor"
+			(at 146.05 105.41 0)
+			(effects
+				(font
+					(size 1.27 1.27)
+				)
+				(hide yes)
+			)
+		)
+		(property "Part #" "MAL229956122E3"
 			(at 146.05 105.41 0)
 			(effects
@@
 			)
 		)
-		(property "Value" "C_Polarized"
+		(property "Value" "1200 uF"
 			(at 129.54 105.7909 0)
 			(effects
@@
 		)
 		(property "Description" "Polarized capacitor"
+			(at 125.73 105.41 0)
+			(effects
+				(font
+					(size 1.27 1.27)
+				)
+				(hide yes)
+			)
+		)
+		(property "Part #" "MAL229956122E3"
 			(at 125.73 105.41 0)
 			(effects
@@
 			)
 		)
-		(property "Value" "C_Polarized"
+		(property "Value" "1200 uF"
 			(at 129.54 95.6309 0)
 			(effects
@@
 			(at 125.73 95.25 0)
 			(effects
+				(font
+					(size 1.27 1.27)
+				)
+				(hide yes)
+			)
+		)
+		(property "Part #" "MAL229956122E3"
+			(at 125.73 95.25 0)
+			(effects

Commit message: titles
Parts:
- added H1, H2, H3, H4: MountingHole, MountingHole:MountingHole_2.7mm_M2.5, symbol Mechanical:MountingHole
Other:
- company: (none) -> Dr.-Ing. Alan H. Wilson Veas
- title: (none) -> Diode-front-end rectifier
